File: pcb/qca7000.kicad_pcb (KiCad board)
At the start: 4 copper layers, 41.6 x 28.2 mm, 111 parts, among them J1 Conn_01x20, J2 JTAG, J3 FLASH, U1 25Q16, Y1 25MHz

Commit message: schematic improvements and board draft
Parts:
- removed C1: 100nF, Capacitor_SMD:C_0603_1608Metric
- removed D11, D12, D13, D14: 19-217/GHC-YR1S2/3T, LED_SMD:LED_0603_1608Metric
- removed J3: FLASH, Connector_PinSocket_2.00mm:PinSocket_1x06_P2.00mm_Vertical
- removed R10, R11, R12, R13, R14, R18, R21: 3.3K, Resistor_SMD:R_0603_1608Metric
- removed R15, R17, R20, R22, R4: 10k, Resistor_SMD:R_0603_1608Metric
- removed TP1, TP3, TP4: TestPoint, TestPoint:TestPoint_Pad_D1.0mm
- added TP6: FL_CS, TestPoint:TestPoint_THTPad_D1.0mm_Drill0.5mm, F.Cu at (156.8, 51.5)
- added TP7: FL_CLK, TestPoint:TestPoint_THTPad_D1.0mm_Drill0.5mm, F.Cu at (157.5, 59.0)
- added TP8: FL_MOSI, TestPoint:TestPoint_THTPad_D1.0mm_Drill0.5mm, F.Cu at (162.9, 59.3)
- added TP9: FL_MISO, TestPoint:TestPoint_THTPad_D1.0mm_Drill0.5mm, F.Cu at (154.9, 54.5)
- C10, C17, C18, C19, C20, C21, C22, C23, C29, C30, C34, C38, C39, C43, C44, C45, C46, C47, C48, C5, C51, C6, C9: footprint Capacitor_SMD:C_0603_1608Metric -> Capacitor_SMD:C_1206_3216Metric_Pad1.33x1.80mm_HandSolder
- C11, C16, C25, C26, C27, C28, C31, C33, C40, C50: footprint Capacitor_SMD:C_0603_1608Metric -> Capacitor_SMD:C_1206_3216Metric_Pad1.33x1.80mm_HandSolder; moved to B.Cu
- C12, C35, C36, C41, C42, C52, C53, C55, C56: value 10uF 25V -> 10uF 10V; footprint Capacitor_SMD:C_0603_1608Metric -> Capacitor_SMD:C_1210_3225Metric_Pad1.33x2.70mm_HandSolder
- C13, C14, C15, C2, C24, C3, C32, C4, C49, C7, C8: footprint Capacitor_SMD:C_0603_1608Metric -> Capacitor_SMD:C_0805_2012Metric_Pad1.18x1.45mm_HandSolder
- C37, C54: value 10uF 25V -> 10uF 10V; footprint Capacitor_SMD:C_0603_1608Metric -> Capacitor_SMD:C_1210_3225Metric_Pad1.33x2.70mm_HandSolder; moved to B.Cu
- J1: value Conn_01x20 -> Conn_01x04_Pin; footprint Connector_PinSocket_2.00mm:PinSocket_1x20_P2.00mm_Vertical -> Connector_PinHeader_2.54mm:PinHeader_1x04_P2.54mm_Vertical; moved to F.Cu
- J2: value JTAG -> Conn_01x08_Pin; footprint Connector_PinHeader_2.00mm:PinHeader_1x08_P2.00mm_Vertical -> Connector_PinHeader_2.54mm:PinHeader_1x08_P2.54mm_Vertical; moved to F.Cu
- L1, L11, L2, L3, L4, L5, L6, L7, L8, L9: footprint Inductor_SMD:L_0603_1608Metric -> Inductor_SMD:L_1206_3216Metric_Pad1.22x1.90mm_HandSolder
- L10: footprint Inductor_SMD:L_1206_3216Metric -> Inductor_SMD:L_1206_3216Metric_Pad1.22x1.90mm_HandSolder
- R1, R16, R19, R2, R6, R7, R8, R9: footprint Resistor_SMD:R_0603_1608Metric -> Resistor_SMD:R_1206_3216Metric_Pad1.30x1.75mm_HandSolder
- R3, R5: value R_Small -> 2.5k; footprint Resistor_SMD:R_0603_1608Metric -> Resistor_SMD:R_1206_3216Metric_Pad1.30x1.75mm_HandSolder
- TP2: value TestPoint -> GPIO_2R; moved to F.Cu
- TP5: value TestPoint -> 1V2; moved to F.Cu
- moved C56 29.5 mm to (148.8, 75.8), turned to 180 degrees
- moved C2 29.2 mm to (90.0, 70.7), turned to -90 degrees
- moved R8 27.7 mm to (130.2, 48.0), turned to -90 degrees
- moved J1 27.5 mm to (88.2, 66.8), turned to 180 degrees
- moved C5 26.6 mm to (94.2, 72.2), turned to 180 degrees
- moved C51 26.4 mm to (144.1, 46.3), turned to 0 degrees
- moved D2 26.0 mm to (99.8, 75.1), turned to 0 degrees
- moved D1 25.3 mm to (99.7, 66.5), turned to 0 degrees
- moved C42 25.0 mm to (161.2, 46.2), turned to 0 degrees
- moved C6 24.5 mm to (94.4, 69.4), turned to 180 degrees
- moved R7 24.2 mm to (133.9, 45.6), turned to 0 degrees
- moved C10 23.9 mm to (104.8, 74.8), turned to 90 degrees
- moved C35 23.7 mm to (121.0, 77.4), turned to 180 degrees
- moved D3 23.4 mm to (99.7, 69.0), turned to 180 degrees
- moved D4 23.0 mm to (99.8, 72.7), turned to 180 degrees
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Connections:
- C13 pad 2: Net-(C13-Pad2) -> GND
- C14 pad 1: Net-(C13-Pad2) -> GND
- D10 pad 14: SERIAL_IO_4 -> SERIAL_IO_4_MOSI
- D10 pad 15: SERIAL_IO_3 -> SERIAL_IO_3_MISO
- D10 pad 16: SERIAL_IO_2 -> SERIAL_IO_2_CS
- D10 pad 19: SERIAL_IO_1 -> SERIAL_IO_1_CLK
- D10 pad 20: SERIAL_IO_0 -> SERIAL_IO_0_INT
- D10 pad 22: TDI -> GND
- D10 pad 23: TCK -> GND
- D10 pad 24: TDO -> unconnected-(D10-TDO-Pad24)
- D10 pad 25: TMS -> GND
- D10 pad 26: RTCK -> unconnected-(D10-RTCK-Pad26)
- D10 pad 27: TRST_L -> GND
- D10 pad 34: Net-(D10-Pad34) -> unconnected-(D10-ATB_N-Pad34)
- D10 pad 35: Net-(D10-Pad35) -> unconnected-(D10-ATB_P-Pad35)
- D10 pad 41: ZC -> GND
- D10 pad 44: Net-(D10-Pad44) -> unconnected-(D10-PLL_BYPASS-Pad44)
- D10 pad 53: Net-(D10-Pad53) -> unconnected-(D10-RSVD06-Pad53)
- D10 pad 54: Net-(D10-Pad54) -> unconnected-(D10-RSVD07-Pad54)
- D10 pad 60: GPIO_0 -> unconnected-(D10-GPIO_0-Pad60)
- D10 pad 63: GPIO_3 -> unconnected-(D10-GPIO_3-Pad63)
- J1 pad 1: RX_N -> TX_P
- J1 pad 2: RX_P -> TX_N
- J1 pad 3: TX_N -> RX_P
- J1 pad 4: TX_P -> RX_N
- J2 pad 1: +3V3_D -> GND
- J2 pad 2: TDI -> +3V3_D
- J2 pad 3: TCK -> RESET#
- J2 pad 4: TDO -> SERIAL_IO_4_MOSI
- J2 pad 5: TMS -> SERIAL_IO_3_MISO
- J2 pad 6: RTCK -> SERIAL_IO_2_CS
- J2 pad 7: TRST_L -> SERIAL_IO_1_CLK
- J2 pad 8: GND -> SERIAL_IO_0_INT
- L8 pad 2: Net-(C13-Pad2) -> GND
- L9 pad 1: Net-(C13-Pad2) -> GND
- R16 pad 2: Net-(J1-Pad17) -> GND
- R19 pad 2: Net-(J1-Pad18) -> Net-(R19-Pad2)
- TP2 pad 1: Net-(D10-Pad34) -> Net-(R19-Pad2)
Routing:
- net GND: track 45.2 -> 87.5 mm, vias 115 -> 71
- net +1V2_C: track 171.2 -> 134.4 mm, vias 12 -> 9
- net TXOUT_P: track 12.6 -> 44.1 mm
- net TXOUT_N: track 13.9 -> 42.6 mm
- net SERIAL_IO_0_INT: track 0.00 -> 27.8 mm
- net SERIAL_IO_4: track 26.3 -> 0.00 mm, vias 1 -> 0
- net SERIAL_IO_1_CLK: track 0.00 -> 26.2 mm
- net TRST_L: track 24.9 -> 0.00 mm, vias 1 -> 0
- net SERIAL_IO_3: track 23.1 -> 0.00 mm, vias 1 -> 0
- net RESET#: track 28.2 -> 6.30 mm, vias 1 -> 0
- net SERIAL_IO_2: track 21.6 -> 0.00 mm, vias 1 -> 0
- net GPIO_3: track 21.0 -> 0.00 mm, vias 3 -> 0
- net TMS: track 21.0 -> 0.00 mm, vias 1 -> 0
- net RTCK: track 20.5 -> 0.00 mm, vias 1 -> 0
- net +3V3_A: track 32.5 -> 52.7 mm
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- added copper zone on F.Cu, net +3V3_D
- removed copper zone on F.Cu, net GND
- removed copper zone on In1.Cu, net GND
- removed copper zone on In2.Cu, net GND
Other:
- board size 41.6 x 28.2 mm -> 82.4 x 40.7 mm

Commit message: board: more width for supply, fill, shrink
Parts:
- C18: footprint Capacitor_SMD:C_1206_3216Metric_Pad1.33x1.80mm_HandSolder -> Capacitor_SMD:C_0805_2012Metric_Pad1.18x1.45mm_HandSolder; moved to B.Cu
- moved C18 20.8 mm to (134.9, 58.0), turned to 180 degrees
- moved C2 4.63 mm to (94.6, 70.0)
- moved J1 4.43 mm to (92.6, 66.8)
- moved C5 2.92 mm to (96.8, 73.7), turned to 90 degrees
- moved C6 2.86 mm to (96.7, 67.7), turned to -90 degrees
- moved D3 1.75 mm to (101.4, 68.8)
- moved D1 1.71 mm to (101.4, 66.4)
- moved D2 1.34 mm to (101.1, 75.0)
- moved D4 1.24 mm to (101.1, 72.7)
- moved TP6 0.83 mm to (155.9, 51.3)
- moved C9 0.72 mm to (105.7, 67.1)
- moved C47 0.70 mm to (127.5, 61.5)
- moved C10 0.68 mm to (105.5, 74.7)
- moved L9 0.50 mm to (119.5, 61.5)
- moved J2 0.40 mm to (136.7, 42.5)
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Routing:
- net +3V3_D: track 170.7 -> 58.5 mm
- net GND: track 87.5 -> 64.0 mm, vias 71 -> 86
- net +1V2_C: track 134.4 -> 143.7 mm, vias 9 -> 10
- net RX_P: track 9.07 -> 4.64 mm
- net RX_N: track 9.27 -> 4.95 mm
- net Net-(D3-K): track 22.4 -> 19.1 mm
- net TX_N: track 9.80 -> 7.77 mm
- net SERIAL_IO_1_CLK: track 26.2 -> 24.3 mm
- net SERIAL_IO_0_INT: track 27.8 -> 26.1 mm
- net TX_P: track 9.27 -> 7.68 mm
- net TXOUT_P: track 44.1 -> 43.0 mm
- net TXOUT_N: track 42.6 -> 41.6 mm
- net SERIAL_IO_4_MOSI: track 19.3 -> 18.7 mm
- added copper zone on F.Cu, net GND
Other:
- board size 82.4 x 40.7 mm -> 76 x 40 mm

Commit message: v1 ready for production
Parts:
- moved C2 0.51 mm to (94.6, 70.5)
- moved D2 0.50 mm to (101.1, 75.5)
Routing:
- net TX_P: track 7.68 -> 8.29 mm
Other:
- copper layers 4 -> 2
- board text added: "3V3"
- board text added: "CLK"
- board text added: "CS"
- board text added: "GND"
- board text added: "INT"
- board text added: "MISO"
- board text added: "MOSI"
- board text added: "QCA7005 homeplug modem github.com/uhi22/QCA7000board version June 2023"
- board text added: "RES"

Commit message: started adding power supply
Parts:
- removed the TP2 at (152.5, 60.2)
- added C56: 100nF, Capacitor_SMD:C_1206_3216Metric_Pad1.33x1.80mm_HandSolder, F.Cu at (130.4, 67.6)
- added C57: 470uF, Capacitor_SMD:CP_Elec_10x10, F.Cu at (128.6, 84.3)
- added C58: 100nF, Capacitor_SMD:C_1206_3216Metric_Pad1.33x1.80mm_HandSolder, F.Cu at (174.7, 72.3)
- added C59: 100uF, Capacitor_SMD:CP_Elec_8x10, F.Cu at (177.2, 66.4)
- added C60: 100nF, Capacitor_SMD:C_1206_3216Metric_Pad1.33x1.80mm_HandSolder, F.Cu at (139.9, 83.8)
- added C61: 100nF, Capacitor_SMD:C_1206_3216Metric_Pad1.33x1.80mm_HandSolder, F.Cu at (170.0, 84.7)
- added C62: 100uF, Capacitor_SMD:CP_Elec_8x10, F.Cu at (161.9, 82.6)
- added C63: 100nF, Capacitor_SMD:C_1206_3216Metric_Pad1.33x1.80mm_HandSolder, F.Cu at (194.9, 81.1)
- added C64: 100nF, Capacitor_SMD:C_1206_3216Metric_Pad1.33x1.80mm_HandSolder, F.Cu at (185.1, 64.1)
- added C65: 100nF, Capacitor_SMD:C_1206_3216Metric_Pad1.33x1.80mm_HandSolder, F.Cu at (189.2, 81.2)
- added C66: 100uF, Capacitor_SMD:CP_Elec_8x10, F.Cu at (179.8, 81.6)
- added D10: SS54B-HF, Diode_SMD:D_SMB_Handsoldering, F.Cu at (145.0, 69.1)
- added D9: SS54B-HF, Diode_SMD:D_SMB_Handsoldering, F.Cu at (127.0, 74.7)
- added J3: 12V_in, Connector_PinHeader_2.54mm:PinHeader_1x02_P2.54mm_Vertical, F.Cu at (123.9, 68.4)
- added L12: 68uH, Inductor_SMD:L_Wuerth_WE-PD-Typ-LS_Handsoldering, F.Cu at (158.4, 69.1)
- added TP3V3uC1: TP3V3uC, TestPoint:TestPoint_THTPad_D1.0mm_Drill0.5mm, F.Cu at (191.6, 64.5)
- added TP5V1: TP5V, TestPoint:TestPoint_THTPad_D1.0mm_Drill0.5mm, F.Cu at (170.0, 61.8)
- added U2: XL1509-5.0, Package_SO:SOIC-8_3.9x4.9mm_P1.27mm, F.Cu at (136.6, 68.3)
- added U3: AMS1117-3.3, Package_TO_SOT_SMD:SOT-223-3_TabPin2, F.Cu at (147.5, 82.5)
- added U4: AMS1117-3.3, Package_TO_SOT_SMD:SOT-223-3_TabPin2, F.Cu at (188.9, 71.9)
- L11: renamed from L10; footprint Inductor_SMD:L_1206_3216Metric_Pad1.22x1.90mm_HandSolder -> Inductor_SMD:L_1812_4532Metric_Pad1.30x3.40mm_HandSolder
- moved C48 57.3 mm to (172.9, 102.3)
- moved C11 57.0 mm to (136.1, 115.3)
- moved C14 57.0 mm to (171.8, 102.1)
- moved C15 57.0 mm to (172.3, 120.7)
- moved C2 57.0 mm to (130.1, 103.9)
- moved C21 57.0 mm to (151.4, 125.5)
- moved C28 57.0 mm to (157.9, 112.7)
- moved C29 57.0 mm to (155.7, 120.5)
- moved C36 57.0 mm to (175.8, 103.5)
- moved C38 57.0 mm to (157.6, 106.9)
- moved C4 57.0 mm to (138.7, 104.7)
- moved C49 57.0 mm to (157.8, 109.7)
- moved C50 57.0 mm to (157.1, 105.5)
- moved D5 57.0 mm to (141.4, 123.8)
- moved D7 57.0 mm to (131.5, 120.9)
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- renumbered C7 to C1, C2 to C10, C9 to C11, C5 to C12, C10 to C13, C27 to C14, C28 to C15, C29 to C16, C32 to C17, C11 to C18, C12 to C19, C3 to C2, C51 to C20, C35 to C21, C36 to C22, C41 to C23, C42 to C24, C52 to C25, C53 to C26, C56 to C27, C33 to C28, C49 to C29, C13 to C3, C37 to C30, C25 to C31, C38 to C32, C39 to C33, C16 to C34, C50 to C35, C54 to C36, C17 to C37, C40 to C38, C55 to C39, C15 to C4, C18 to C40, C19 to C41, C43 to C42, C44 to C43, C45 to C44, C20 to C45, C22 to C46, C46 to C47, C47 to C49, C24 to C5, C34 to C50, C21 to C51, C23 to C52, C26 to C53, C30 to C54, C31 to C55, C4 to C6, C14 to C7, C6 to C9, D6 to D1, D7 to D2, D1 to D3, D3 to D4, D2 to D6, D4 to D7, D10 to D8, L3 to L1, L5 to L10, L6 to L2, L11 to L3, L1 to L4, L8 to L5, L2 to L6, L9 to L7, L4 to L8, L7 to L9, R8 to R10, R16 to R3, R19 to R4, R6 to R5, R3 to R6, R9 to R7, R7 to R8, R5 to R9, TP5 to TP1, TP8 to TP2, TP7 to TP3, TP6 to TP4, TP9 to TP5
Connections:
- C15 pad 2: +3V3_D -> 3V3_D
- C20 pad 1: +3V3_D -> 3V3_D
- C21 pad 2: +3V3_D -> 3V3_D
- C22 pad 2: +3V3_D -> 3V3_D
- C23 pad 2: +3V3_D -> 3V3_D
- C24 pad 2: +3V3_D -> 3V3_D
- C30 pad 2: +3V3_D -> 3V3_D
- C32 pad 1: +3V3_D -> 3V3_D
- C35 pad 1: +3V3_D -> 3V3_D
- C37 pad 2: +3V3_D -> 3V3_D
- C39 pad 1: +3V3_D -> 3V3_D
- C42 pad 1: +3V3_D -> 3V3_D
- C43 pad 1: +3V3_D -> 3V3_D
- C45 pad 2: +3V3_D -> 3V3_D
- C47 pad 1: +3V3_D -> 3V3_D
- C54 pad 2: +3V3_D -> 3V3_D
- C55 pad 2: +3V3_D -> 3V3_D
- D8 pad 13: +3V3_D -> 3V3_D
- D8 pad 17: +3V3_D -> 3V3_D
- D8 pad 2: +3V3_D -> 3V3_D
- D8 pad 21: +3V3_D -> 3V3_D
- D8 pad 43: +3V3_D -> 3V3_D
- D8 pad 47: +3V3_D -> 3V3_D
- D8 pad 59: +3V3_D -> 3V3_D
- D8 pad 6: +3V3_D -> 3V3_D
- D8 pad 64: +3V3_D -> 3V3_D
- D8 pad 7: +3V3_D -> 3V3_D
- D8 pad 8: +3V3_D -> 3V3_D
- J2 pad 2: +3V3_D -> 3V3_D
- L2 pad 2: +3V3_D -> 3V3_D
- L9 pad 2: +3V3_D -> 3V3_D
- R4 pad 2: Net-(R19-Pad2) -> +3V3_D
- R7 pad 2: +3V3_D -> 3V3_D
- U1 pad 3: +3V3_D -> 3V3_D
- U1 pad 7: +3V3_D -> 3V3_D
- U1 pad 8: +3V3_D -> 3V3_D
Routing:
- net +3V3_D: track 58.5 -> 2.77 mm, vias 11 -> 2
- net 3V3_D: track 0.00 -> 55.7 mm, vias 0 -> 9
- net Net-(R19-Pad2): track 3.47 -> 0.00 mm
Other:
- board size 76 x 40 mm -> 76 x 68.4 mm
- board text added: "QCA7005 homeplug modem github.com/uhi22/QCA7000board version 2023-07-06"
- board text removed: "QCA7005 homeplug modem github.com/uhi22/QCA7000board version June 2023"

Commit message: added sheets for inputs and outputs. layout draft.
Parts:
- added C67: 22uF, Capacitor_SMD:C_1206_3216Metric_Pad1.33x1.80mm_HandSolder, F.Cu at (154.9, 81.5)
- added C68: 68pF, Capacitor_SMD:C_1206_3216Metric_Pad1.33x1.80mm_HandSolder, F.Cu at (182.5, 75.8)
- added C69: 470uF, Capacitor_SMD:CP_Elec_10x10, F.Cu at (173.4, 64.8)
- added C70: 100nF, Capacitor_SMD:C_0805_2012Metric_Pad1.18x1.45mm_HandSolder, F.Cu at (179.8, 83.3)
- added C72: 100uF, Capacitor_SMD:CP_Elec_8x10, F.Cu at (193.6, 123.1)
- added C73: 100nF, Capacitor_SMD:C_0805_2012Metric_Pad1.18x1.45mm_HandSolder, F.Cu at (158.2, 81.6)
- added C74: 100nF, Capacitor_SMD:C_0805_2012Metric_Pad1.18x1.45mm_HandSolder, F.Cu at (154.0, 73.6)
- added C75: 100uF, Capacitor_SMD:CP_Elec_8x10, F.Cu at (170.9, 76.5)
- added C76: 1nF, Capacitor_SMD:C_0805_2012Metric_Pad1.18x1.45mm_HandSolder, F.Cu at (128.5, 94.9)
- added C77: 100nF, Capacitor_SMD:C_1206_3216Metric_Pad1.33x1.80mm_HandSolder, F.Cu at (127.4, 66.8)
- added C78: 100nF, Capacitor_SMD:C_1206_3216Metric_Pad1.33x1.80mm_HandSolder, F.Cu at (131.6, 70.5)
- added C79: 100nF, Capacitor_SMD:C_1206_3216Metric_Pad1.33x1.80mm_HandSolder, F.Cu at (132.4, 75.7)
- added D11: LED, LED_SMD:LED_0805_2012Metric_Pad1.15x1.40mm_HandSolder, F.Cu at (124.3, 86.8)
- added D12: LED, LED_SMD:LED_0805_2012Metric_Pad1.15x1.40mm_HandSolder, F.Cu at (169.0, 42.5)
- added D13: SS54B-HF, Diode_SMD:D_SMB_Handsoldering, F.Cu at (193.9, 67.5)
- added D14: 1N4148W, Diode_SMD:D_SOD-123, F.Cu at (128.4, 91.4)
- added J10: CP/PE, Connector_PinHeader_2.54mm:PinHeader_1x02_P2.54mm_Vertical, F.Cu at (123.3, 91.0)
- added J4: DEBUG, Connector_PinHeader_2.54mm:PinHeader_1x03_P2.54mm_Vertical, F.Cu at (148.0, 53.3)
- added J5: UART, Connector_PinHeader_2.54mm:PinHeader_1x03_P2.54mm_Vertical, F.Cu at (155.0, 43.5)
- added J6: 12V_in, Connector_PinHeader_2.54mm:PinHeader_1x02_P2.54mm_Vertical, F.Cu at (200.6, 67.8)
- added J7: RF, Connector_PinHeader_2.54mm:PinHeader_1x02_P2.54mm_Vertical, F.Cu at (122.9, 103.1)
- added J8: CONTACTORS, Connector_PinHeader_2.54mm:PinHeader_1x02_P2.54mm_Vertical, F.Cu at (198.6, 50.9)
- added J9: Temps, Connector_PinHeader_2.54mm:PinHeader_1x04_P2.54mm_Vertical, F.Cu at (123.0, 74.7)
- added JP1: SolderJumper3V3together, Jumper:SolderJumper-2_P1.3mm_Open_TrianglePad1.0x1.5mm, F.Cu at (170.3, 84.6)
- added L13: 10uH, Inductor_SMD:L_Wuerth_WE-PD-Typ-LS_Handsoldering, F.Cu at (198.1, 83.6)
- added Q1: BC846, Package_TO_SOT_SMD:SOT-23, F.Cu at (140.1, 88.7)
- added Q2: NCV8402xST, Package_TO_SOT_SMD:SOT-223, F.Cu at (189.1, 58.4)
- added Q3: NCV8402xST, Package_TO_SOT_SMD:SOT-223, F.Cu at (189.2, 45.9)
- added R11: 220, Resistor_SMD:R_1206_3216Metric_Pad1.30x1.75mm_HandSolder, F.Cu at (150.9, 86.9)
- added R12: 220, Resistor_SMD:R_1206_3216Metric_Pad1.30x1.75mm_HandSolder, F.Cu at (145.2, 86.8)
- added R13: 220, Resistor_SMD:R_1206_3216Metric_Pad1.30x1.75mm_HandSolder, F.Cu at (156.3, 87.0)
- added R14: 220, Resistor_SMD:R_1206_3216Metric_Pad1.30x1.75mm_HandSolder, F.Cu at (161.8, 87.2)
- added R15: 33, Resistor_SMD:R_1206_3216Metric_Pad1.30x1.75mm_HandSolder, F.Cu at (133.1, 60.9)
- added R16: 1k, Resistor_SMD:R_1206_3216Metric_Pad1.30x1.75mm_HandSolder, F.Cu at (163.7, 59.1)
- added R17: 1k, Resistor_SMD:R_1206_3216Metric_Pad1.30x1.75mm_HandSolder, F.Cu at (151.0, 73.3)
- added R18: 1k, Resistor_SMD:R_1206_3216Metric_Pad1.30x1.75mm_HandSolder, F.Cu at (141.4, 53.4)
- added R19: 1k, Resistor_SMD:R_1206_3216Metric_Pad1.30x1.75mm_HandSolder, F.Cu at (129.1, 86.9)
- added R20: 1k, Resistor_SMD:R_1206_3216Metric_Pad1.30x1.75mm_HandSolder, F.Cu at (173.7, 42.5)
- added R21: 220, Resistor_SMD:R_1206_3216Metric_Pad1.30x1.75mm_HandSolder, F.Cu at (149.2, 47.3)
- added R22: 220, Resistor_SMD:R_1206_3216Metric_Pad1.30x1.75mm_HandSolder, F.Cu at (149.2, 44.7)
- added R23: 10k, Resistor_SMD:R_1206_3216Metric_Pad1.30x1.75mm_HandSolder, F.Cu at (179.4, 75.2)
- added R24: 10k, Resistor_SMD:R_1206_3216Metric_Pad1.30x1.75mm_HandSolder, F.Cu at (186.3, 76.8)
- added R25: 180, Resistor_SMD:R_1206_3216Metric_Pad1.30x1.75mm_HandSolder, F.Cu at (128.1, 98.7)
- added R26: 2k7, Resistor_SMD:R_1206_3216Metric_Pad1.30x1.75mm_HandSolder, F.Cu at (133.6, 93.4)
- added R27: 1k2, Resistor_SMD:R_1206_3216Metric_Pad1.30x1.75mm_HandSolder, F.Cu at (133.7, 91.0)
- added R28: 10k, Resistor_SMD:R_1206_3216Metric_Pad1.30x1.75mm_HandSolder, F.Cu at (134.8, 86.9)
- added R29: 10k, Resistor_SMD:R_1206_3216Metric_Pad1.30x1.75mm_HandSolder, F.Cu at (135.8, 43.5)
- added R30: 10k, Resistor_SMD:R_1206_3216Metric_Pad1.30x1.75mm_HandSolder, F.Cu at (135.6, 46.2)
- added R31: 10k, Resistor_SMD:R_1206_3216Metric_Pad1.30x1.75mm_HandSolder, B.Cu at (125.8, 73.0)
- added R32: 47k, Resistor_SMD:R_1206_3216Metric_Pad1.30x1.75mm_HandSolder, F.Cu at (124.9, 69.1)
- added R33: 10k, Resistor_SMD:R_1206_3216Metric_Pad1.30x1.75mm_HandSolder, B.Cu at (128.0, 74.2)
- added R34: 47k, Resistor_SMD:R_1206_3216Metric_Pad1.30x1.75mm_HandSolder, F.Cu at (127.5, 72.2)
- added R35: 10k, Resistor_SMD:R_1206_3216Metric_Pad1.30x1.75mm_HandSolder, B.Cu at (130.2, 76.0)
- added R36: 47k, Resistor_SMD:R_1206_3216Metric_Pad1.30x1.75mm_HandSolder, F.Cu at (129.6, 78.8)
- added TP10: ~, TestPoint:TestPoint_THTPad_D1.0mm_Drill0.5mm, F.Cu at (137.2, 77.2)
- added TP11: ~, TestPoint:TestPoint_THTPad_D1.0mm_Drill0.5mm, F.Cu at (143.7, 43.3)
- added TP12: ~, TestPoint:TestPoint_THTPad_D1.0mm_Drill0.5mm, F.Cu at (157.3, 63.0)
- added TP13: ~, TestPoint:TestPoint_THTPad_D1.0mm_Drill0.5mm, F.Cu at (154.9, 62.8)
- added TP14: ~, TestPoint:TestPoint_THTPad_D1.0mm_Drill0.5mm, F.Cu at (152.9, 62.4)
- added TP15: ~, TestPoint:TestPoint_THTPad_D1.0mm_Drill0.5mm, F.Cu at (132.6, 79.5)
- added TP16: ~, TestPoint:TestPoint_THTPad_D1.0mm_Drill0.5mm, F.Cu at (140.7, 78.0)
- added TP17: ~, TestPoint:TestPoint_THTPad_D1.0mm_Drill0.5mm, F.Cu at (141.8, 79.6)
- added TP18: ~, TestPoint:TestPoint_THTPad_D1.0mm_Drill0.5mm, F.Cu at (163.1, 67.1)
- added TP19: ~, TestPoint:TestPoint_THTPad_D1.0mm_Drill0.5mm, F.Cu at (165.2, 66.7)
- added TP20: ~, TestPoint:TestPoint_THTPad_D1.0mm_Drill0.5mm, F.Cu at (147.8, 50.4)
- added TP21: ~, TestPoint:TestPoint_THTPad_D1.0mm_Drill0.5mm, F.Cu at (163.6, 64.5)
- added TP22: ~, TestPoint:TestPoint_THTPad_D1.0mm_Drill0.5mm, F.Cu at (159.9, 63.5)
- added TP23: ~, TestPoint:TestPoint_THTPad_D1.0mm_Drill0.5mm, F.Cu at (143.2, 78.1)
- added TP24: ~, TestPoint:TestPoint_THTPad_D1.0mm_Drill0.5mm, F.Cu at (144.6, 79.7)
- added TP25: ~, TestPoint:TestPoint_THTPad_D1.0mm_Drill0.5mm, F.Cu at (145.6, 77.9)
- added TP26: ~, TestPoint:TestPoint_THTPad_D1.0mm_Drill0.5mm, F.Cu at (145.4, 44.4)
- added TP27: ~, TestPoint:TestPoint_THTPad_D1.0mm_Drill0.5mm, F.Cu at (134.7, 52.6)
- added TP28: ~, TestPoint:TestPoint_THTPad_D1.0mm_Drill0.5mm, F.Cu at (134.3, 55.2)
- added TP29: ~, TestPoint:TestPoint_THTPad_D1.0mm_Drill0.5mm, F.Cu at (132.4, 56.5)
- added TP30: ~, TestPoint:TestPoint_THTPad_D1.0mm_Drill0.5mm, F.Cu at (137.0, 51.3)
- added TP31: ~, TestPoint:TestPoint_THTPad_D1.0mm_Drill0.5mm, F.Cu at (138.6, 52.7)
- added TP32: ~, TestPoint:TestPoint_THTPad_D1.0mm_Drill0.5mm, F.Cu at (147.0, 79.6)
- added TP33: ~, TestPoint:TestPoint_THTPad_D1.0mm_Drill0.5mm, F.Cu at (147.9, 77.7)
- added TP34: ~, TestPoint:TestPoint_THTPad_D1.0mm_Drill0.5mm, F.Cu at (155.0, 69.3)
- added TP35: SWO, TestPoint:TestPoint_THTPad_D1.0mm_Drill0.5mm, F.Cu at (143.5, 46.9)
- added TP36: ~, TestPoint:TestPoint_THTPad_D1.0mm_Drill0.5mm, F.Cu at (157.1, 68.9)
- added TP37: ~, TestPoint:TestPoint_THTPad_D1.0mm_Drill0.5mm, F.Cu at (159.1, 68.5)
- added TP38: ~, TestPoint:TestPoint_THTPad_D1.0mm_Drill0.5mm, F.Cu at (161.1, 67.8)
- added TP6: uC_RESET, TestPoint:TestPoint_THTPad_D1.0mm_Drill0.5mm, F.Cu at (125.3, 64.0)
- added TP7: ~, TestPoint:TestPoint_THTPad_D1.0mm_Drill0.5mm, F.Cu at (132.4, 81.6)
- added TP8: ~, TestPoint:TestPoint_THTPad_D1.0mm_Drill0.5mm, F.Cu at (137.0, 81.7)
- added TP9: ~, TestPoint:TestPoint_THTPad_D1.0mm_Drill0.5mm, F.Cu at (137.1, 79.5)
- added U5: AMS1117-3.3, Package_TO_SOT_SMD:SOT-223-3_TabPin2, F.Cu at (185.0, 90.1)
- added U6: AMS1117-3.3, Package_TO_SOT_SMD:SOT-223-3_TabPin2, F.Cu at (160.0, 74.7)
- added U7: 74HCT04, Package_SO:SO-14_3.9x8.65mm_P1.27mm, F.Cu at (178.0, 53.1)
- added Y2: 8MHz, Crystal:Crystal_SMD_TXC_7M-4Pin_3.2x2.5mm, F.Cu at (129.5, 60.9)
- C56, C58: footprint Capacitor_SMD:C_1206_3216Metric_Pad1.33x1.80mm_HandSolder -> Capacitor_SMD:C_0805_2012Metric_Pad1.18x1.45mm_HandSolder
- C57: value 470uF -> 100nF; footprint Capacitor_SMD:CP_Elec_10x10 -> Capacitor_SMD:C_0805_2012Metric_Pad1.18x1.45mm_HandSolder
- C59: value 100uF -> 100nF; footprint Capacitor_SMD:CP_Elec_8x10 -> Capacitor_SMD:C_0805_2012Metric_Pad1.18x1.45mm_HandSolder
- C61: footprint Capacitor_SMD:C_1206_3216Metric_Pad1.33x1.80mm_HandSolder -> Capacitor_SMD:C_0805_2012Metric_Pad1.18x1.45mm_HandSolder; moved to B.Cu
- C62: value 100uF -> 22p; footprint Capacitor_SMD:CP_Elec_8x10 -> Capacitor_SMD:C_0805_2012Metric_Pad1.18x1.45mm_HandSolder
- C63: value 100nF -> 22p; footprint Capacitor_SMD:C_1206_3216Metric_Pad1.33x1.80mm_HandSolder -> Capacitor_SMD:C_0805_2012Metric_Pad1.18x1.45mm_HandSolder
- C65: value 100nF -> 10uF
- C66: value 100uF -> 22uF; footprint Capacitor_SMD:CP_Elec_8x10 -> Capacitor_SMD:C_1206_3216Metric_Pad1.33x1.80mm_HandSolder
- D10, D9: value SS54B-HF -> LED; footprint Diode_SMD:D_SMB_Handsoldering -> LED_SMD:LED_0805_2012Metric_Pad1.15x1.40mm_HandSolder
- J3: value 12V_in -> CAN; footprint Connector_PinHeader_2.54mm:PinHeader_1x02_P2.54mm_Vertical -> Connector_PinHeader_2.54mm:PinHeader_1x03_P2.54mm_Vertical
- L12: value 68uH -> Bead 600; footprint Inductor_SMD:L_Wuerth_WE-PD-Typ-LS_Handsoldering -> Inductor_SMD:L_0805_2012Metric_Pad1.15x1.40mm_HandSolder
- R6: value 2.5k -> 6k2
- U2: value XL1509-5.0 -> SN65HVD234
- U3: value AMS1117-3.3 -> STM32F103RETx; footprint Package_TO_SOT_SMD:SOT-223-3_TabPin2 -> Package_QFP:LQFP-64_10x10mm_P0.5mm
- U4: value AMS1117-3.3 -> TPS54302; footprint Package_TO_SOT_SMD:SOT-223-3_TabPin2 -> Package_TO_SOT_SMD:SOT-23-6
- moved C63 69.4 mm to (129.5, 57.9), turned to 0 degrees
- moved J3 45.0 mm to (166.2, 53.2), turned to -90 degrees
- moved C62 37.3 mm to (129.6, 64.1), turned to 180 degrees
- moved C61 36.4 mm to (135.5, 73.0), turned to -90 degrees
- moved C58 36.2 mm to (138.5, 72.1), turned to 0 degrees
- moved TP3V3uC1 32.9 mm to (163.9, 82.2), turned to 0 degrees
- moved C57 29.9 mm to (137.8, 55.8), turned to 180 degrees
- moved C60 28.8 mm to (124.9, 59.3)
- moved C59 26.7 mm to (151.5, 59.2), turned to 90 degrees
- moved TP5V1 26.1 mm to (178.8, 86.3), turned to 0 degrees
- moved D9 24.5 mm to (151.2, 77.9), turned to 90 degrees
- moved U2 22.7 mm to (157.4, 59.0), turned to 0 degrees
- moved L12 21.7 mm to (137.3, 74.0)
- moved D10 19.9 mm to (140.4, 49.7), turned to 0 degrees
- moved U3 19.6 mm to (142.3, 63.7)
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Connections:
- C56 pad 2: 12V_P -> 3V3_uC
- C57 pad 1: 12V_P -> GND
- C57 pad 2: GND -> 3V3_uC
- C58 pad 2: 5V -> 3V3_uC
- C59 pad 1: 5V -> GND
- C59 pad 2: GND -> 3V3_uC
- C60 pad 2: 5V -> uC_RESET
- C61 pad 2: 3V3_D -> Net-(U3-VDDA)
- C62 pad 1: 3V3_D -> GND
- C62 pad 2: GND -> /controller/OCS_IN
- C63 pad 1: 3V3_uC -> GND
- C63 pad 2: GND -> Net-(C63-Pad2)
- C64 pad 1: GND -> Net-(U4-SW)
- C64 pad 2: 5V -> Net-(U4-BOOT)
- C65 pad 2: 3V3_uC -> 12V_P
- C66 pad 1: 3V3_uC -> GND
- C66 pad 2: GND -> 5V
- D10 pad 1: Net-(D10-K) -> GND
- D10 pad 2: GND -> Net-(D10-A)
- D9 pad 1: 12V_P -> GND
- D9 pad 2: 12V -> Net-(D9-A)
- J3 pad 1: 12V -> CANL
- L12 pad 1: Net-(D10-K) -> Net-(U3-VDDA)
- L12 pad 2: 5V -> 3V3_uC
- R10 pad 2: +3V3_D -> 3V3_D
- R4 pad 2: +3V3_D -> 3V3_D
- U2 pad 1: 12V_P -> CAN_TX
- U2 pad 2: Net-(D10-K) -> GND
- U2 pad 3: 5V -> 3V3_uC
- U2 pad 4: GND -> CAN_RX
- U2 pad 5: GND -> unconnected-(U2-EN-Pad5)
- U2 pad 6: GND -> CANL
- U2 pad 7: GND -> CANH
- U3 pad 1: GND -> 3V3_uC
- U3 pad 2: 3V3_D -> Net-(U3-PC13)
- U3 pad 3: 5V -> Net-(U3-PC14)
- U4 pad 2: 3V3_uC -> Net-(U4-SW)
- U4 pad 3: 5V -> 12V_P
Routing:
- net 3V3_uC: track 0.00 -> 125.3 mm, vias 0 -> 1
- net GND: track 63.9 -> 127.7 mm, vias 86 -> 136
- net SPI1_MOSI: track 0.00 -> 36.4 mm
- net SPI1_MISO: track 0.00 -> 31.4 mm
- net SPI1_NSS: track 0.00 -> 30.5 mm
- net SPI1_CLK: track 0.00 -> 21.0 mm
- net Net-(U3-PC7): track 0.00 -> 17.9 mm
- net 12V_P: track 0.00 -> 17.8 mm
- net Net-(U3-PA0): track 0.00 -> 17.5 mm
- net Net-(U3-PA1): track 0.00 -> 16.8 mm
- net Net-(U3-PC3): track 0.00 -> 16.7 mm
- net ADC123_IN12: track 0.00 -> 16.2 mm
- net uC_RESET: track 0.00 -> 16.1 mm
- net Net-(U3-PC6): track 0.00 -> 15.8 mm
- net Net-(U3-PC8): track 0.00 -> 15.7 mm
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- added copper zone on F.Cu, net 3V3_D
- added copper zone on F.Cu, net CONTACTOR1_LS
- removed copper zone on F.Cu, net +3V3_D
Other:
- board size 76 x 68.4 mm -> 83 x 89 mm

Commit message: layout for stm, supply, drivers, flash programming connector
Parts:
- added D15: UARTTX, LED_SMD:LED_0805_2012Metric_Pad1.15x1.40mm_HandSolder, F.Cu at (151.1, 45.7)
- added J11: spare, Connector_PinHeader_2.54mm:PinHeader_1x06_P2.54mm_Vertical, F.Cu at (124.7, 54.9)
- added R37: 1k, Resistor_SMD:R_1206_3216Metric_Pad1.30x1.75mm_HandSolder, F.Cu at (150.1, 49.6)
- added TP39: FL_GND, TestPoint:TestPoint_THTPad_D1.5mm_Drill0.7mm, F.Cu at (201.7, 111.3)
- added TP40: FL_RES, TestPoint:TestPoint_THTPad_D1.5mm_Drill0.7mm, F.Cu at (199.1, 111.8)
- D10: value LED -> ALIVE
- D11: value LED -> STATEC
- D12: value LED -> CONTACTOR1
- D9: value LED -> PWR
- JP1: moved to B.Cu
- L10, L2, L9: footprint Inductor_SMD:L_1206_3216Metric_Pad1.22x1.90mm_HandSolder -> Inductor_SMD:L_0805_2012Metric_Pad1.15x1.40mm_HandSolder
- TP2, TP3, TP4, TP5: footprint TestPoint:TestPoint_THTPad_D1.0mm_Drill0.5mm -> TestPoint:TestPoint_THTPad_D1.5mm_Drill0.7mm
- moved TP4 12.9 mm to (191.5, 111.3)
- moved TP5 9.85 mm to (189.0, 111.8)
- moved TP3 9.58 mm to (196.6, 111.3)
- moved JP1 5.32 mm to (165.0, 84.2)
- moved TP19 4.67 mm to (160.7, 68.2)
- moved TP18 4.65 mm to (159.1, 69.5)
- moved R21 4.63 mm to (153.3, 49.5), turned to -90 degrees
- moved TP2 4.36 mm to (194.1, 111.8)
- moved TP38 3.66 mm to (157.5, 68.4)
- moved TP37 3.59 mm to (155.6, 69.2)
- moved R20 3.59 mm to (172.4, 45.8), turned to 90 degrees
- moved TP26 3.42 mm to (147.1, 47.4)
- moved TP21 3.41 mm to (160.5, 66.0)
- moved TP11 3.34 mm to (145.4, 46.2)
- moved TP36 3.33 mm to (153.8, 68.2)
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Routing:
- net 5V: track 0.00 -> 94.8 mm
- net RESET#: track 6.30 -> 63.3 mm, vias 0 -> 2
- net CONTACTOR_CONTROL1: track 12.2 -> 61.9 mm, vias 0 -> 2
- net CONTACTOR_CONTROL2: track 11.8 -> 50.1 mm, vias 0 -> 2
- net STATE_C_CONTROL: track 14.3 -> 36.8 mm, vias 0 -> 6
- net 3V3_uC: track 125.3 -> 139.0 mm
- net 3V3_D: track 58.5 -> 70.8 mm, vias 11 -> 13
- net SPI_DI: track 24.5 -> 36.0 mm, vias 2 -> 4
- net Net-(U4-SW): track 5.54 -> 15.9 mm
- net Net-(U4-FB): track 0.00 -> 9.23 mm
- net SPI_CS_L: track 36.5 -> 45.4 mm, vias 2 -> 4
- net SPI_CLK: track 29.5 -> 36.8 mm
- net UART4_TX: track 11.8 -> 17.0 mm
- net UART4_RX: track 14.6 -> 19.1 mm
- net SPI_DO: track 27.3 -> 31.6 mm
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- added copper zone on F.Cu, net CONTACTOR2_LS
Other:
- board size 83 x 89 mm -> 84.7 x 89.1 mm
- board text added: "CANH GND CANL"
- board text added: "CP"
- board text added: "GND 12V"
- board text added: "SWCLK G SWDIO"
- board text added: "UART RX GND TX"
- board text added: "fully open CCS charge controller github.com/uhi22/foccci version 2023-07-11"
- board text removed: "QCA7005 homeplug modem github.com/uhi22/QCA7000board version 2023-07-06"

Commit message: fix: can transceiver enable high. fix: uart LED low active. fix: contactor LED low active. fix: LED names in silkscreen.
Connections:
- D12 pad 1: GND -> Net-(D12-K)
- D12 pad 2: Net-(D12-A) -> 3V3_uC
- D15 pad 1: GND -> Net-(D15-K)
- D15 pad 2: Net-(D15-A) -> 3V3_uC
- R20 pad 2: Net-(D12-A) -> Net-(D12-K)
- R37 pad 2: Net-(D15-A) -> Net-(D15-K)
- U2 pad 5: unconnected-(U2-EN-Pad5) -> 3V3_uC
Routing:
- net 3V3_uC: track 139.0 -> 180.4 mm, vias 1 -> 5
- net Net-(D12-K): track 0.00 -> 3.70 mm
- net Net-(D15-A): track 3.16 -> 0.00 mm
- net Net-(D12-A): track 2.95 -> 0.00 mm
- net Net-(D15-K): track 0.00 -> 2.31 mm
- net GND: vias 156 -> 154
