File: pcb/qca7000.kicad_pcb (KiCad board)
At the start: 4 copper layers, 100 x 82.6 mm, 253 parts, among them IC1 DRV8874QPWPRQ1, J1 Conn_01x04_Pin, J10 CP/PE, J16 uC_NRST, J17 3V3_uC, J18 SWO, J2 Conn_01x08_Pin, J20 DTM1312PA12PBR008, J4 DEBUG, J5 UART, J7 RF, Q1 BC846, Q2 NCV8402xST, Q3 NCV8402xST, Q4 DTA143Z, Q5 DTA143Z, Q6 DTA143Z, Q7 DTC114E, Q8 DTC114E, Q9 DTC114E, U1 25Q16, U2 SN65HVD230, U3 STM32F103RETx, U4 TPS54302, U6 AMS1117-3.3, U7 74HCT04, U8 EEC-325X4B, Y1 25MHz, Y2 12MHz

Commit message: BOM consolidation: XTAL options and back to 8MHz. Replace internal connectors by testpoints. Use T with integrated R for CP switching. Fix: Footprint Q7-Q9 corrected.
Parts:
- removed J1: Conn_01x04_Pin, Connector_PinHeader_2.54mm:PinHeader_1x04_P2.54mm_Vertical
- removed J10: CP/PE, Connector_PinHeader_2.54mm:PinHeader_1x02_P2.54mm_Vertical
- removed J16: uC_NRST, Connector_PinHeader_2.54mm:PinHeader_1x01_P2.54mm_Vertical
- removed J17: 3V3_uC, Connector_PinHeader_2.54mm:PinHeader_1x01_P2.54mm_Vertical
- removed J18: SWO, Connector_PinHeader_2.54mm:PinHeader_1x01_P2.54mm_Vertical
- removed J2: Conn_01x08_Pin, Connector_PinHeader_2.54mm:PinHeader_1x08_P2.54mm_Vertical
- removed J4: DEBUG, Connector_PinHeader_2.54mm:PinHeader_1x03_P2.54mm_Vertical
- removed J5: UART, Connector_PinHeader_2.54mm:PinHeader_1x03_P2.54mm_Vertical
- removed J7: RF, Connector_PinHeader_2.54mm:PinHeader_1x02_P2.54mm_Vertical
- removed R28: 10k, Resistor_SMD:R_0805_2012Metric_Pad1.20x1.40mm_HandSolder
- added 3V3: ~, speciallib:TestPoint_Special_THTPad_D1.9mm_Drill1mm, F.Cu at (94.7, 106.3)
- added 3V3_uC1: ~, speciallib:TestPoint_Special_THTPad_D1.9mm_Drill1mm, F.Cu at (102.3, 60.5)
- added CLK1: ~, speciallib:TestPoint_Special_THTPad_D1.9mm_Drill1mm, F.Cu at (82.0, 106.3)
- added CS1: ~, speciallib:TestPoint_Special_THTPad_D1.9mm_Drill1mm, F.Cu at (84.5, 106.3)
- added GND1: ~, speciallib:TestPoint_Special_THTPad_D1.9mm_Drill1mm, F.Cu at (97.2, 106.3)
- added GND2: ~, speciallib:TestPoint_Special_THTPad_D1.9mm_Drill1mm, F.Cu at (57.5, 117.0)
- added INT1: ~, speciallib:TestPoint_Special_THTPad_D1.9mm_Drill1mm, F.Cu at (79.4, 106.3)
- added MISO1: ~, speciallib:TestPoint_Special_THTPad_D1.9mm_Drill1mm, F.Cu at (87.1, 106.3)
- added MOSI1: ~, speciallib:TestPoint_Special_THTPad_D1.9mm_Drill1mm, F.Cu at (89.6, 106.3)
- added RES1: ~, speciallib:TestPoint_Special_THTPad_D1.9mm_Drill1mm, F.Cu at (92.1, 106.3)
- added RF1: ~, speciallib:TestPoint_Special_THTPad_D1.9mm_Drill1mm, F.Cu at (57.5, 114.6)
- added RX_N1: ~, TestPoint:TestPoint_THTPad_D1.0mm_Drill0.5mm, F.Cu at (57.6, 124.1)
- added RX_P1: ~, TestPoint:TestPoint_THTPad_D1.0mm_Drill0.5mm, F.Cu at (57.6, 126.7)
- added SWCLK1: ~, speciallib:TestPoint_Special_THTPad_D1.9mm_Drill1mm, F.Cu at (82.0, 68.8)
- added SWDIO1: ~, speciallib:TestPoint_Special_THTPad_D1.9mm_Drill1mm, F.Cu at (87.1, 68.8)
- added SWGND1: ~, speciallib:TestPoint_Special_THTPad_D1.9mm_Drill1mm, F.Cu at (84.5, 68.8)
- added SWO1: ~, speciallib:TestPoint_Special_THTPad_D1.9mm_Drill1mm, F.Cu at (64.3, 60.5)
- added TX_N1: ~, TestPoint:TestPoint_THTPad_D1.0mm_Drill0.5mm, F.Cu at (57.6, 129.2)
- added TX_P1: ~, TestPoint:TestPoint_THTPad_D1.0mm_Drill0.5mm, F.Cu at (57.6, 131.7)
- added UART_GND1: ~, speciallib:TestPoint_Special_THTPad_D1.9mm_Drill1mm, F.Cu at (92.1, 64.4)
- added UART_RX1: ~, speciallib:TestPoint_Special_THTPad_D1.9mm_Drill1mm, F.Cu at (92.1, 61.8)
- added UART_TX1: ~, speciallib:TestPoint_Special_THTPad_D1.9mm_Drill1mm, F.Cu at (92.1, 66.9)
- added Y3: 8MHz, Crystal:Crystal_SMD_5032-2Pin_5.0x3.2mm, F.Cu at (64.3, 74.0)
- added uC_NRST1: ~, speciallib:TestPoint_Special_THTPad_D1.9mm_Drill1mm, F.Cu at (56.6, 75.2)
- Q1: value BC846 -> DTC114E
- Y2: value 12MHz -> 8MHz; moved to B.Cu
- moved TP50 79.7 mm to (57.3, 120.7)
- moved C63 3.09 mm to (61.2, 72.9), turned to 90 degrees
- moved TP27 2.51 mm to (67.9, 65.2)
- moved TP29 1.74 mm to (68.6, 70.1)
- moved TP28 1.70 mm to (69.0, 67.9)
- moved PB6 1.47 mm to (68.1, 63.1)
- moved Y2 1.35 mm to (64.3, 73.9), turned to 90 degrees
- moved PB5 1.21 mm to (69.9, 61.9)
- moved C60 0.63 mm to (61.1, 77.0)
- moved Q1 0.19 mm to (66.6, 104.5)
Connections:
- C62 pad 1: GND -> /controller/OCS_IN
- C62 pad 2: /controller/OCS_IN -> GND
- Q1 pad 1: Net-(Q1-B) -> STATE_C_CONTROL
Routing:
- net Net-(C63-Pad2): track 4.66 -> 7.77 mm, vias 0 -> 1
- net STATE_C_CONTROL: track 45.6 -> 48.3 mm
- net Net-(U3-PC13): track 8.87 -> 11.6 mm
- net Net-(Q1-B): track 2.15 -> 0.00 mm
- net /controller/OCS_IN: track 12.5 -> 10.4 mm, vias 0 -> 1
- net uC_NRST: track 17.3 -> 19.2 mm
- net Net-(R21-Pad2): track 5.21 -> 7.05 mm
- net Net-(R22-Pad2): track 12.0 -> 13.9 mm
- net Net-(U3-PC14): track 7.26 -> 8.95 mm
- net SWO: track 23.1 -> 24.1 mm
- net Net-(U3-PB6): track 13.3 -> 13.9 mm
- net GND: track 70.2 -> 70.7 mm

Commit message: docu: V4 2023-09-10 finished. Added board history.
Other:
- board text added: "fully open CCS charge controller / github.com/uhi22/foccci / version 2023-09-10"
- board text removed: "fully open CCS charge controller / github.com/uhi22/foccci / version 2023-08-26"
Changed lines of the file:
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@@
     (effects (font (size 1.5 1.5) (thickness 0.3) bold) (justify left bottom))
   )
-  (gr_text "fully open CCS charge controller / github.com/uhi22/foccci / version 2023-08-26" (at 76.78 57.75) (layer "F.SilkS")
+  (gr_text "fully open CCS charge controller / github.com/uhi22/foccci / version 2023-09-10" (at 76.78 57.75) (layer "F.SilkS")
     (effects (font (size 0.9 0.9) (thickness 0.2) bold) (justify left bottom))
   )
