File: pcb/qca7000.kicad_pcb (KiCad board)
At the start: 4 copper layers, 100 x 82.6 mm, 267 parts, among them IC1 DRV8874QPWPRQ1, J20 DTM1312PA12PBR008, Q1 DTC114E, Q2 NCV8402xST, Q3 NCV8402xST, Q4 DTA143Z, Q5 DTA143Z, Q6 DTA143Z, Q7 DTC114E, Q8 DTC114E, Q9 DTC114E, U1 25Q16, U2 SN65HVD230, U3 STM32F103RETx, U4 TPS54302, U6 AMS1117-3.3, U7 74HCT04, U8 EEC-325X4B, Y1 25MHz, Y2 8MHz, Y3 8MHz

Commit message: layout fix: bigger gap between QCA corner and via, to avoid solder bridge to corner frame metal. Silkscreen improvements.
Parts:
- D8: value QCA 7000 -> QCA 7005
Routing:
- net +1V2_C: track 90.7 -> 92.7 mm
Other:
- board text added: "fully open CCS charge controller / github.com/uhi22/foccci / version 2023-10-25 / v4.1"
- board text removed: "fully open CCS charge controller / github.com/uhi22/foccci / version 2023-09-10"

Commit message: fix rx shortcut. add transformer. correct part number of NCV. Correct footprints of U1 and L11. add mounting holes. stepdown layout improved. added TVS at 12V
Parts:
- removed GND2, RF1: ~, speciallib:TestPoint_Special_THTPad_D1.9mm_Drill1mm
- removed RX_N1, RX_P1, TX_N1, TX_P1: ~, TestPoint:TestPoint_THTPad_D1.0mm_Drill0.5mm
- added C32: 1.5nF, Capacitor_SMD:C_0805_2012Metric_Pad1.18x1.45mm_HandSolder, F.Cu at (79.7, 118.0)
- added C33: 1.5nF, Capacitor_SMD:C_0805_2012Metric_Pad1.18x1.45mm_HandSolder, F.Cu at (79.5, 121.7)
- added H2: MountingHole, MountingHole:MountingHole_3.2mm_M3, F.Cu at (57.8, 60.7)
- added H3: MountingHole, MountingHole:MountingHole_3.2mm_M3, F.Cu at (138.8, 71.2)
- added H4: MountingHole, MountingHole:MountingHole_3.2mm_M3, F.Cu at (57.9, 132.8)
- added H5: MountingHole, MountingHole:MountingHole_3.2mm_M3, F.Cu at (127.2, 126.3)
- added T1: ~, transformerCL4532A-201:transformerCL4532A-201, F.Cu at (59.7, 111.9)
- added U5: SMAJ18A-TR, tvs:SMA_UNI_STM, F.Cu at (138.0, 94.1)
- D8: value QCA 7005 -> QCA 7000
- L11: footprint Inductor_SMD:L_1812_4532Metric_Pad1.30x3.40mm_HandSolder -> Inductor_SMD:L_1206_3216Metric_Pad1.22x1.90mm_HandSolder
- L13: footprint Inductor_SMD:L_Wuerth_WE-PD-Typ-LS_Handsoldering -> Inductor_SMD:L_12x12mm_H4.5mm
- U1: footprint Package_SO:SOP-8_5.28x5.23mm_P1.27mm -> Package_SO:SOIC-8_3.9x4.9mm_P1.27mm
- moved TP50 79.9 mm to (109.9, 60.5)
- moved C65 17.0 mm to (128.1, 79.2), turned to 90 degrees
- moved R44 12.3 mm to (58.3, 119.9), turned to 0 degrees
- moved R8 10.4 mm to (58.3, 117.9), turned to 180 degrees
- moved D6 9.07 mm to (58.7, 128.2), turned to 180 degrees
- moved C12 9.02 mm to (58.3, 123.9), turned to 180 degrees
- moved C64 7.07 mm to (125.1, 81.9), turned to 180 degrees
- moved D3 7.00 mm to (62.6, 131.4), turned to -90 degrees
- moved C6 6.42 mm to (63.4, 126.3), turned to 90 degrees
- moved L6 6.05 mm to (65.2, 126.5), turned to 90 degrees
- moved L4 6.01 mm to (65.2, 122.9)
- moved C2 5.99 mm to (63.4, 121.9)
- moved U4 5.76 mm to (124.6, 79.1), turned to 180 degrees
- moved R24 5.46 mm to (121.2, 83.2), turned to 0 degrees
- moved R38 5.31 mm to (120.6, 81.2), turned to 0 degrees
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Connections:
- C3 pad 1: RXIN_N -> Net-(C3-Pad1)
- C7 pad 2: RXIN_P -> Net-(C33-Pad2)
- D1 pad 3: RXIN_P -> Net-(C33-Pad2)
- D2 pad 3: RXIN_N -> Net-(C3-Pad1)
- L1 pad 2: RXIN_N -> Net-(C3-Pad1)
- L5 pad 1: RXIN_N -> Net-(C3-Pad1)
- L7 pad 2: RXIN_P -> Net-(C33-Pad2)
- L8 pad 2: RXIN_P -> Net-(C33-Pad2)
Routing:
- net RXIN_P: track 20.0 -> 9.07 mm
- net Net-(D4-K): track 22.4 -> 11.7 mm
- net Net-(C3-Pad1): track 0.00 -> 10.5 mm
- net Net-(C33-Pad2): track 0.00 -> 8.88 mm
- net RXIN_N: track 19.8 -> 11.4 mm
- net Net-(C10-Pad2): track 12.0 -> 4.98 mm
- net TXOUT_P: track 31.6 -> 38.3 mm
- net SPI_CS_L: track 50.9 -> 44.4 mm
- net RX_N: track 9.49 -> 3.40 mm
- net Net-(D1-A): track 26.1 -> 20.4 mm
- net TXOUT_N: track 31.2 -> 36.9 mm
- net CP: track 131.2 -> 126.2 mm, vias 0 -> 1
- net GND: track 70.7 -> 74.6 mm, vias 170 -> 177
- net BUTTON: track 50.3 -> 53.5 mm
- net SPI_DO: track 41.7 -> 38.7 mm
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Other:
- board text added: "fully open CCS charge controller / github.com/uhi22/foccci / version 2023-12-18 / v4.2pre"
- board text removed: "fully open CCS charge controller / github.com/uhi22/foccci / version 2023-10-25 / v4.1"

Commit message: fix: origin of the transformer into the middle. Fix: rotation attributes for jlcpcb
Parts:
- moved T1 2.33 mm to (58.5, 114.0)

Commit message: stepdown L and layout further optimized. fix rotation and layout
Parts:
- L13: footprint Inductor_SMD:L_12x12mm_H4.5mm -> Inductor_SMD:L_6.3x6.3_H3
- moved L13 2.87 mm to (133.5, 82.6)
- moved C66 2.36 mm to (127.7, 85.6)
Routing:
- net 5V: track 96.7 -> 101.9 mm
- net Net-(U4-SW): track 14.2 -> 12.0 mm
- net GND: vias 177 -> 176
