File: pcb/controller.kicad_sch (KiCad schematic)
At the start: 41 parts, among them J4 DEBUG, J5 CAN, J6 UART, J7 RF, Q1 BC846, U5 STM32F103RETx, U6 SN65HVD234, Y1 8MHz

Commit message: added sheets for inputs and outputs. layout draft.
Parts:
- removed C17: 1nF, Capacitor_SMD:C_0805_2012Metric_Pad1.18x1.45mm_HandSolder, symbol Device:C_Small
- removed D10: 1N4148W, Diode_SMD:D_SOD-123, symbol Diode:1N4148W
- removed J7: RF, symbol Connector:Conn_01x02_Pin
- removed L13: 10uH, Inductor_SMD:L_Wuerth_WE-PD-Typ-LS_Handsoldering, symbol Device:L
- removed Q1: BC846, Package_TO_SOT_SMD:SOT-23, symbol Transistor_BJT:BC846
- removed R3: 180, Resistor_SMD:R_1206_3216Metric_Pad1.30x1.75mm_HandSolder, symbol Device:R_Small
- removed R3: 2k7, Resistor_SMD:R_1206_3216Metric_Pad1.30x1.75mm_HandSolder, symbol Device:R_Small
- removed R3: 1k2, Resistor_SMD:R_1206_3216Metric_Pad1.30x1.75mm_HandSolder, symbol Device:R_Small
- removed R3: 10k, Resistor_SMD:R_1206_3216Metric_Pad1.30x1.75mm_HandSolder, symbol Device:R_Small
- added L10: Bead 600, Inductor_SMD:L_0805_2012Metric_Pad1.15x1.40mm_HandSolder, symbol Device:L
- added TP5V1 (x31): ~, TestPoint:TestPoint_THTPad_D1.0mm_Drill0.5mm, symbol Connector:TestPoint
- C61: footprint Capacitor_SMD:C_1206_3216Metric_Pad1.33x1.80mm_HandSolder -> Capacitor_SMD:C_0805_2012Metric_Pad1.18x1.45mm_HandSolder
- J3: renamed from J5; footprint (none) -> Connector_PinHeader_2.54mm:PinHeader_1x03_P2.54mm_Vertical
- J4: footprint (none) -> Connector_PinHeader_2.54mm:PinHeader_1x03_P2.54mm_Vertical
- J5: renamed from J6; footprint (none) -> Connector_PinHeader_2.54mm:PinHeader_1x03_P2.54mm_Vertical
- renumbered D12 to D10, D13 to D11, D14 to D12, D11 to D9, U6 to U2, U5 to U3
Connections:
- net CP_CONTROL is gone; now on net STATE_C_CONTROL: R3.1
- net 3V3_uC: now also L10.2
- net GND: now also U3.60 (BOOT0)
- net at C61.2, U3.13 (VDDA): now also L10.1
- net CANL: now reaches J3.1 (Pin_1), R3.1, U2.6 (CANL)
- net CANH: now reaches J3.3 (Pin_3), R3.2, U2.7 (CANH)
- net at U3.11 (PC3): now also TP5V1.1
- net at U3.14 (PA0): now also TP5V1.1
- net at U3.15 (PA1): now also TP5V1.1
- net at U3.16 (PA2): now also TP5V1.1
- net at U3.17 (PA3): now also TP5V1.1
- net at U3.2 (PC13): now also TP5V1.1
- net at U3.24 (PC4): now also TP5V1.1
- net at U3.25 (PC5): now also TP5V1.1
- net at U3.26 (PB0): now also TP5V1.1
- net at U3.27 (PB1): now also TP5V1.1
- net at U3.28 (PB2): now also TP5V1.1
- net at U3.29 (PB10): now also TP5V1.1
- net at U3.3 (PC14): now also TP5V1.1
- net at U3.30 (PB11): now also TP5V1.1
- net at U3.33 (PB12): now also TP5V1.1
- net at U3.34 (PB13): now also TP5V1.1
- net at U3.35 (PB14): now also TP5V1.1
- net at U3.36 (PB15): now also TP5V1.1
- net at U3.37 (PC6): now also TP5V1.1
- net at U3.38 (PC7): now also TP5V1.1
- net at U3.39 (PC8): now also TP5V1.1
- net at U3.4 (PC15): now also TP5V1.1
- net at U3.40 (PC9): now also TP5V1.1
- net at U3.41 (PA8): now also TP5V1.1
- net at U3.42 (PA9): now also TP5V1.1
- net at U3.43 (PA10): now also TP5V1.1
- net at U3.50 (PA15): now also TP5V1.1
- net at U3.53 (PC12): now also TP5V1.1
- net at U3.54 (PD2): now also TP5V1.1
- net at U3.61 (PB8): now also TP5V1.1
- net at U3.62 (PB9): now also TP5V1.1
Other:
- note added: "boot0=0 boots from the user flash"
- note removed: "ControlPilot circuit for StateB (2k7) and StateC (additional 1k2)."
- note removed: "Todo: Contactor drivers, Temperature sensors, ..."
- note removed: "Todo: TVS etc for protecting the CP"

Commit message: layout for stm, supply, drivers, flash programming connector
Parts:
- added D15: UARTTX, LED_SMD:LED_0805_2012Metric_Pad1.15x1.40mm_HandSolder, symbol Device:LED
- added R3: 1k, Resistor_SMD:R_1206_3216Metric_Pad1.30x1.75mm_HandSolder, symbol Device:R_Small
- D10: value LED -> ALIVE
- D11: value LED -> STATEC
- D12: value LED -> CONTACTOR1
- D9: value LED -> PWR
Connections:
- net GND: now also D15.1 (K)
- net UART4_TX: now also R3.1
- new net: D15.2 (A), R3.2
Changed lines of the file:
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@@
+    (stroke (width 0) (type default))
+  )
+  (wire (pts (xy 67.31 132.08) (xy 71.12 132.08))
     (stroke (width 0) (type default))
   )
@@
     (stroke (width 0) (type default))
   )
+  (wire (pts (xy 44.45 132.08) (xy 50.8 132.08))
+    (stroke (width 0) (type default))
+  )
   (wire (pts (xy 92.71 76.2) (xy 92.71 74.93))
     (stroke (width 0) (type default))
@@
   )
   (wire (pts (xy 153.67 52.07) (xy 151.13 52.07))
+    (stroke (width 0) (type default))
+  )
+  (wire (pts (xy 55.88 132.08) (xy 59.69 132.08))
     (stroke (width 0) (type default))
   )
@@
     (property "Intersheetrefs" "${INTERSHEET_REFS}" (at 199.6954 120.65 0)
       (effects (font (size 1.27 1.27)) (justify left) hide)
+    )
+  )
+  (global_label "UART4_TX" (shape input) (at 44.45 132.08 180) (fields_autoplaced)
+    (effects (font (size 1.27 1.27)) (justify right))
+    (property "Intersheetrefs" "${INTERSHEET_REFS}" (at 32.5333 132.08 0)
+      (effects (font (size 1.27 1.27)) (justify right) hide)
     )
   )
@@
       (effects (font (size 1.27 1.27)))
     )
-    (property "Value" "LED" (at 64.77 111.76 0)
+    (property "Value" "STATEC" (at 64.77 111.76 0)
       (effects (font (size 1.27 1.27)))
     )
@@
     )
   )
+  (symbol (lib_id "Device:LED") (at 63.5 132.08 180) (unit 1)
+    (in_bom yes) (on_board yes) (dnp no)
+    (property "Reference" "D15" (at 59.69 129.54 0)
+      (effects (font (size 1.27 1.27)))
+    )
+    (property "Value" "UARTTX" (at 64.77 129.54 0)
+      (effects (font (size 1.27 1.27)))
+    )
+    (property "Footprint" "LED_SMD:LED_0805_2012Metric_Pad1.15x1.40mm_HandSolder" (at 63.5 132.08 0)
+      (effects (font (size 1.27 1.27)) hide)
+    )
+    (property "Datasheet" "~" (at 63.5 132.08 0)
+      (effects (font (size 1.27 1.27)) hide)
+    )
+    (pin "1")
+    (pin "2")
+    (instances
+      (project "qca7000"
+        (path "/e63e39d7-6ac0-4ffd-8aa3-1841a4541b55/5666e7cf-6b6c-4583-8335-aa3be69ccd45"
+          (reference "D15") (unit 1)
+        )
+      )
+    )
+  )
   (symbol (lib_id "Connector:TestPoint") (at 176.53 85.09 270) (unit 1)
     (in_bom yes) (on_board yes) (dnp no)
@@
         (path "/e63e39d7-6ac0-4ffd-8aa3-1841a4541b55/5666e7cf-6b6c-4583-8335-aa3be69ccd45"
           (reference "TP16") (unit 1)
+        )
+      )
+    )
+  )
+  (symbol (lib_id "Device:R_Small") (at 53.34 132.08 90) (unit 1)
+    (in_bom yes) (on_board yes) (dnp no)
+    (property "Reference" "R3" (at 53.34 129.54 90)
+      (effects (font (size 1.27 1.27)))
+    )
+    (property "Value" "1k" (at 53.34 134.62 90)
+      (effects (font (size 1.27 1.27)))
+    )
+    (property "Footprint" "Resistor_SMD:R_1206_3216Metric_Pad1.30x1.75mm_HandSolder" (at 53.34 132.08 0)
+      (effects (font (size 1.27 1.27)) hide)
+    )
+    (property "Datasheet" "https://datasheet.lcsc.com/lcsc/1811101920_UNI-ROYAL-Uniroyal-Elec-0603WAF3301T5E_C22978.pdf" (at 53.34 132.08 0)
+      (effects (font (size 1.27 1.27)) hide)
+    )
+    (property "LCSC" "C22978" (at 53.34 132.08 90)
+      (effects (font (size 1.27 1.27)) hide)
+    )
+    (pin "1")
+    (pin "2")
+    (instances
+      (project "qca7000"
+        (path "/e63e39d7-6ac0-4ffd-8aa3-1841a4541b55"
+          (reference "R3") (unit 1)
+        )
+        (path "/e63e39d7-6ac0-4ffd-8aa3-1841a4541b55/5666e7cf-6b6c-4583-8335-aa3be69ccd45"
+          (reference "R37") (unit 1)
         )
       )
@@
       (effects (font (size 1.27 1.27)))
     )
-    (property "Value" "LED" (at 64.77 120.65 0)
+    (property "Value" "CONTACTOR1" (at 64.77 120.65 0)
       (effects (font (size 1.27 1.27)))
     )
@@
         (path "/e63e39d7-6ac0-4ffd-8aa3-1841a4541b55/5666e7cf-6b6c-4583-8335-aa3be69ccd45"
           (reference "TP34") (unit 1)
+        )
+      )
+    )
+  )
+  (symbol (lib_id "power:GND") (at 71.12 132.08 90) (unit 1)
+    (in_bom yes) (on_board yes) (dnp no)
+    (property "Reference" "#PWR048" (at 77.47 132.08 0)
+      (effects (font (size 1.27 1.27)) hide)
+    )
+    (property "Value" "GND" (at 74.93 129.54 0)
+      (effects (font (size 1.27 1.27)) (justify right))
+    )
+    (property "Footprint" "" (at 71.12 132.08 0)
+      (effects (font (size 1.27 1.27)) hide)
+    )
+    (property "Datasheet" "" (at 71.12 132.08 0)
+      (effects (font (size 1.27 1.27)) hide)
+    )
+    (pin "1")
+    (instances
+      (project "qca7000"
+        (path "/e63e39d7-6ac0-4ffd-8aa3-1841a4541b55"
+          (reference "#PWR048") (unit 1)
+        )
+        (path "/e63e39d7-6ac0-4ffd-8aa3-1841a4541b55/5666e7cf-6b6c-4583-8335-aa3be69ccd45"
+          (reference "#PWR068") (unit 1)
         )
       )
@@
       (effects (font (size 1.27 1.27)))
     )
-    (property "Value" "LED" (at 65.0875 101.6 0)
+    (property "Value" "ALIVE" (at 65.0875 101.6 0)
       (effects (font (size 1.27 1.27)))
     )
@@
       (effects (font (size 1.27 1.27)))
     )
-    (property "Value" "LED" (at 64.77 92.71 0)
-      (effects (font (size 1.27 1.27)))
-    )
+    (property "Value" "PWR" (at 64.77 92.71 0)
+      (effects (font (size 1.27 1.27)))
+    )

Commit message: fix: can transceiver enable high. fix: uart LED low active. fix: contactor LED low active. fix: LED names in silkscreen.
Connections:
- net 3V3_uC: now also D12.2 (A), D15.2 (A), U2.5 (EN)
- net GND: no longer D12.1 (K), D15.1 (K)
- net at R3.2: now also D15.1 (K); no longer D15.2 (A)
- net at R3.2: now also D12.1 (K); no longer D12.2 (A)
- no-connect marks 1 -> 0
Other:
- note added: "EN=High enables the transceiver. Low or open would disable it."
- moved on the sheet: D12, D15
Changed lines of the file:
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@@
   (junction (at 156.21 52.07) (diameter 0) (color 0 0 0 0)
   )
+  (junction (at 69.85 132.08) (diameter 0) (color 0 0 0 0)
+  )
   (junction (at 232.41 97.79) (diameter 0) (color 0 0 0 0)
   )
   (junction (at 92.71 76.2) (diameter 0) (color 0 0 0 0)
   )
+  (junction (at 232.41 78.74) (diameter 0) (color 0 0 0 0)
+  )
   (junction (at 92.71 64.77) (diameter 0) (color 0 0 0 0)
   )
@@
   (junction (at 248.92 86.36) (diameter 0) (color 0 0 0 0)
   )
-  (no_connect (at 222.25 90.17))
   (wire (pts (xy 128.27 113.03) (xy 135.89 113.03))
     (stroke (width 0) (type default))
@@
     (stroke (width 0) (type default))
   )
+  (wire (pts (xy 55.88 132.08) (xy 59.69 132.08))
+    (stroke (width 0) (type default))
+  )
   (wire (pts (xy 161.29 54.61) (xy 161.29 57.15))
     (stroke (width 0) (type default))
@@
     (stroke (width 0) (type default))
   )
+  (wire (pts (xy 67.31 123.19) (xy 69.85 123.19))
+    (stroke (width 0) (type default))
+  )
   (wire (pts (xy 250.19 157.48) (xy 251.46 157.48))
     (stroke (width 0) (type default))
   )
-  (wire (pts (xy 67.31 123.19) (xy 71.12 123.19))
+  (wire (pts (xy 220.98 90.17) (xy 222.25 90.17))
     (stroke (width 0) (type default))
   )
@@
     (stroke (width 0) (type default))
   )
+  (wire (pts (xy 55.88 123.19) (xy 59.69 123.19))
+    (stroke (width 0) (type default))
+  )
   (wire (pts (xy 252.73 93.98) (xy 251.46 93.98))
     (stroke (width 0) (type default))
@@
     (stroke (width 0) (type default))
   )
-  (wire (pts (xy 55.88 123.19) (xy 59.69 123.19))
-    (stroke (width 0) (type default))
-  )
   (wire (pts (xy 133.35 105.41) (xy 135.89 105.41))
     (stroke (width 0) (type default))
@@
     (stroke (width 0) (type default))
   )
+  (wire (pts (xy 69.85 123.19) (xy 69.85 132.08))
+    (stroke (width 0) (type default))
+  )
   (wire (pts (xy 161.29 46.99) (xy 158.75 46.99))
     (stroke (width 0) (type default))
@@
     (stroke (width 0) (type default))
   )
+  (wire (pts (xy 220.98 78.74) (xy 220.98 90.17))
+    (stroke (width 0) (type default))
+  )
+  (wire (pts (xy 69.85 132.08) (xy 71.12 132.08))
+    (stroke (width 0) (type default))
+  )
   (wire (pts (xy 222.25 97.79) (xy 232.41 97.79))
     (stroke (width 0) (type default))
@@
     (stroke (width 0) (type default))
   )
-  (wire (pts (xy 67.31 132.08) (xy 71.12 132.08))
+  (wire (pts (xy 232.41 78.74) (xy 220.98 78.74))
     (stroke (width 0) (type default))
   )
@@
     (stroke (width 0) (type default))
   )
+  (wire (pts (xy 232.41 78.74) (xy 232.41 76.2))
+    (stroke (width 0) (type default))
+  )
   (wire (pts (xy 236.22 59.69) (xy 240.03 59.69))
     (stroke (width 0) (type default))
@@
     (stroke (width 0) (type default))
   )
-  (wire (pts (xy 232.41 80.01) (xy 232.41 76.2))
+  (wire (pts (xy 232.41 80.01) (xy 232.41 78.74))
     (stroke (width 0) (type default))
   )
@@
     (stroke (width 0) (type default))
   )
+  (wire (pts (xy 67.31 132.08) (xy 69.85 132.08))
+    (stroke (width 0) (type default))
+  )
   (wire (pts (xy 236.22 46.99) (xy 240.03 46.99))
     (stroke (width 0) (type default))
@@
   )
   (wire (pts (xy 153.67 52.07) (xy 151.13 52.07))
-    (stroke (width 0) (type default))
-  )
-  (wire (pts (xy 55.88 132.08) (xy 59.69 132.08))
     (stroke (width 0) (type default))
   )
@@
   (text "There are more VSS pins (31, 47, 63)\nwhich are not shown here. Strange."
     (at 137.16 162.56 0)
+    (effects (font (size 1.27 1.27)) (justify left bottom))
+  )
+  (text "EN=High enables\nthe transceiver.\nLow or open would\ndisable it."
+    (at 203.2 99.06 0)
     (effects (font (size 1.27 1.27)) (justify left bottom))
   )
@@
     (property "Intersheetrefs" "${INTERSHEET_REFS}" (at 228.0528 139.7 0)
       (effects (font (size 1.27 1.27)) (justify right) hide)
+    )
+  )
+  (global_label "3V3_uC" (shape input) (at 71.12 132.08 0) (fields_autoplaced)
+    (effects (font (size 1.27 1.27)) (justify left))
+    (property "Intersheetrefs" "${INTERSHEET_REFS}" (at 80.92 132.08 0)
+      (effects (font (size 1.27 1.27)) (justify left) hide)
     )
   )
@@
     )
   )
-  (symbol (lib_id "Device:LED") (at 63.5 132.08 180) (unit 1)
-    (in_bom yes) (on_board yes) (dnp no)
-    (property "Reference" "D15" (at 59.69 129.54 0)
-      (effects (font (size 1.27 1.27)))
-    )
-    (property "Value" "UARTTX" (at 64.77 129.54 0)
+  (symbol (lib_id "Device:LED") (at 63.5 132.08 0) (unit 1)
+    (in_bom yes) (on_board yes) (dnp no)
+    (property "Reference" "D15" (at 67.31 134.62 0)
+      (effects (font (size 1.27 1.27)))
+    )
+    (property "Value" "UARTTX" (at 63.5 129.54 0)
       (effects (font (size 1.27 1.27)))
     )
@@
         (path "/e63e39d7-6ac0-4ffd-8aa3-1841a4541b55/5666e7cf-6b6c-4583-8335-aa3be69ccd45"
           (reference "R37") (unit 1)
-        )
-      )
-    )
-  )
-  (symbol (lib_id "power:GND") (at 71.12 123.19 90) (unit 1)
-    (in_bom yes) (on_board yes) (dnp no)
-    (property "Reference" "#PWR048" (at 77.47 123.19 0)
-      (effects (font (size 1.27 1.27)) hide)
-    )
-    (property "Value" "GND" (at 74.93 120.65 0)
-      (effects (font (size 1.27 1.27)) (justify right))
-    )
-    (property "Footprint" "" (at 71.12 123.19 0)
-      (effects (font (size 1.27 1.27)) hide)
-    )
-    (property "Datasheet" "" (at 71.12 123.19 0)
-      (effects (font (size 1.27 1.27)) hide)
-    )
-    (pin "1")
-    (instances
-      (project "qca7000"
-        (path "/e63e39d7-6ac0-4ffd-8aa3-1841a4541b55"
-          (reference "#PWR048") (unit 1)
-        )
-        (path "/e63e39d7-6ac0-4ffd-8aa3-1841a4541b55/5666e7cf-6b6c-4583-8335-aa3be69ccd45"
-          (reference "#PWR054") (unit 1)
         )
       )
@@
     )
   )
-  (symbol (lib_id "Device:LED") (at 63.5 123.19 180) (unit 1)
-    (in_bom yes) (on_board yes) (dnp no)
-    (property "Reference" "D12" (at 59.69 120.65 0)
+  (symbol (lib_id "Device:LED") (at 63.5 123.19 0) (unit 1)
+    (in_bom yes) (on_board yes) (dnp no)
+    (property "Reference" "D12" (at 67.31 125.73 0)
       (effects (font (size 1.27 1.27)))
     )
@@
         )
       )
-    )
-  )
-  (symbol (lib_id "power:GND") (at 71.12 132.08 90) (unit 1)
-    (in_bom yes) (on_board yes) (dnp no)
-    (property "Reference" "#PWR048" (at 77.47 132.08 0)
-      (effects (font (size 1.27 1.27)) hide)
-    )
-    (property "Value" "GND" (at 74.93 129.54 0)
-      (effects (font (size 1.27 1.27)) (justify right))
-    )
-    (property "Footprint" "" (at 71.12 132.08 0)
-      (effects (font (size 1.27 1.27)) hide)
-    )
-    (property "Datasheet" "" (at 71.12 132.08 0)
-      (effects (font (size 1.27 1.27)) hide)
-    )
-    (pin "1")
-    (instances
-      (project "qca7000"
-        (path "/e63e39d7-6ac0-4ffd-8aa3-1841a4541b55"
-          (reference "#PWR048") (unit 1)
-        )
-        (path "/e63e39d7-6ac0-4ffd-8aa3-1841a4541b55/5666e7cf-6b6c-4583-8335-aa3be69ccd45"
-          (reference "#PWR068") (unit 1)
-        )
-      )

Commit message: fix: divider on the stepdown. fix: non-inverted contactor drivers. fix: part number of 8MHz. add: mounting holes and spare grid. add: LIM HVDC input. docu: todo list
Parts:
- removed TP4: SWO, TestPoint:TestPoint_THTPad_D1.0mm_Drill0.5mm, symbol Connector:TestPoint
- removed TP4: uC_RESET, TestPoint:TestPoint_THTPad_D1.0mm_Drill0.5mm, symbol Connector:TestPoint
- removed TP5V1: ~, TestPoint:TestPoint_THTPad_D1.0mm_Drill0.5mm, symbol Connector:TestPoint
- added J16: uC_NRST, Connector_PinHeader_2.54mm:PinHeader_1x01_P2.54mm_Vertical, symbol Connector:Conn_01x01_Pin
- added J17: 3V3_uC, Connector_PinHeader_2.54mm:PinHeader_1x01_P2.54mm_Vertical, symbol Connector:Conn_01x01_Pin
- added J18: SWO, Connector_PinHeader_2.54mm:PinHeader_1x01_P2.54mm_Vertical, symbol Connector:Conn_01x01_Pin
- Y1: LCSC C9006 -> tbd
Connections:
- net 3V3_uC: now also J17.1 (Pin_1); no longer D12.2 (A)
- net GND: now also D12.1 (K)
- net SWO: now also J18.1 (Pin_1)
- net ADC_U_HVDC: now reaches U3.11 (PC3)
- net at R3.2: now also D12.2 (A); no longer D12.1 (K)
- net uC_RESET renamed uC_NRST
- net uC_NRST: now also J16.1 (Pin_1)
Other:
- note added: "No external pull-up on the reset. This is the recommended circuit, the STM32F103 has internal pull-up."
- note added: "There are more VSS pins (31, 47, 63) which are not shown here. Strange. Nevertheless, in the layout they are correct."
- note removed: "There are more VSS pins (31, 47, 63) which are not shown here. Strange."
- moved on the sheet: D12, J4

Commit message: added TE DEUTSCH connector and housing
Parts:
- removed J3: CAN, Connector_PinHeader_2.54mm:PinHeader_1x03_P2.54mm_Vertical, symbol Connector:Conn_01x03_Pin
Changed lines of the file:
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@@
   (junction (at 161.29 57.15) (diameter 0) (color 0 0 0 0)
   )
-  (junction (at 251.46 86.36) (diameter 0) (color 0 0 0 0)
-  )
-  (junction (at 251.46 91.44) (diameter 0) (color 0 0 0 0)
-  )
   (junction (at 148.59 52.07) (diameter 0) (color 0 0 0 0)
   )
@@
     (stroke (width 0) (type default))
   )
-  (wire (pts (xy 251.46 91.44) (xy 257.81 91.44))
-    (stroke (width 0) (type default))
-  )
   (wire (pts (xy 55.88 96.52) (xy 59.69 96.52))
     (stroke (width 0) (type default))
@@
     (stroke (width 0) (type default))
   )
-  (wire (pts (xy 251.46 86.36) (xy 257.81 86.36))
-    (stroke (width 0) (type default))
-  )
   (wire (pts (xy 226.06 53.34) (xy 231.14 53.34))
     (stroke (width 0) (type default))
@@
     (stroke (width 0) (type default))
   )
-  (wire (pts (xy 252.73 93.98) (xy 251.46 93.98))
-    (stroke (width 0) (type default))
-  )
   (wire (pts (xy 123.19 69.85) (xy 135.89 69.85))
     (stroke (width 0) (type default))
@@
     (stroke (width 0) (type default))
   )
-  (wire (pts (xy 252.73 82.55) (xy 251.46 82.55))
+  (wire (pts (xy 248.92 86.36) (xy 252.73 86.36))
     (stroke (width 0) (type default))
   )
@@
     (stroke (width 0) (type default))
   )
-  (wire (pts (xy 251.46 82.55) (xy 251.46 86.36))
-    (stroke (width 0) (type default))
-  )
   (wire (pts (xy 171.45 72.39) (xy 176.53 72.39))
     (stroke (width 0) (type default))
@@
     (stroke (width 0) (type default))
   )
-  (wire (pts (xy 248.92 86.36) (xy 251.46 86.36))
-    (stroke (width 0) (type default))
-  )
   (wire (pts (xy 171.45 125.73) (xy 175.26 125.73))
     (stroke (width 0) (type default))
@@
     (stroke (width 0) (type default))
   )
-  (wire (pts (xy 251.46 93.98) (xy 251.46 91.44))
-    (stroke (width 0) (type default))
-  )
   (wire (pts (xy 171.45 92.71) (xy 175.26 92.71))
     (stroke (width 0) (type default))
@@
     (stroke (width 0) (type default))
   )
-  (wire (pts (xy 248.92 91.44) (xy 251.46 91.44))
+  (wire (pts (xy 248.92 91.44) (xy 252.73 91.44))
     (stroke (width 0) (type default))
   )
@@
     )
   )
-  (global_label "CANL" (shape input) (at 252.73 93.98 0) (fields_autoplaced)
+  (global_label "CANL" (shape input) (at 252.73 91.44 0) (fields_autoplaced)
     (effects (font (size 1.27 1.27)) (justify left))
-    (property "Intersheetrefs" "${INTERSHEET_REFS}" (at 260.353 93.98 0)
+    (property "Intersheetrefs" "${INTERSHEET_REFS}" (at 260.353 91.44 0)
       (effects (font (size 1.27 1.27)) (justify left) hide)
     )
   )
-  (global_label "CANH" (shape input) (at 252.73 82.55 0) (fields_autoplaced)
+  (global_label "CANH" (shape input) (at 252.73 86.36 0) (fields_autoplaced)
     (effects (font (size 1.27 1.27)) (justify left))
-    (property "Intersheetrefs" "${INTERSHEET_REFS}" (at 260.6554 82.55 0)
+    (property "Intersheetrefs" "${INTERSHEET_REFS}" (at 260.6554 86.36 0)
       (effects (font (size 1.27 1.27)) (justify left) hide)
     )
@@
     )
   )
-  (symbol (lib_id "Connector:Conn_01x03_Pin") (at 262.89 88.9 180) (unit 1)
-    (in_bom yes) (on_board yes) (dnp no) (fields_autoplaced)
-    (property "Reference" "J3" (at 264.16 88.265 0)
-      (effects (font (size 1.27 1.27)) (justify right))
-    )
-    (property "Value" "CAN" (at 264.16 90.805 0)
-      (effects (font (size 1.27 1.27)) (justify right))
-    )
-    (property "Footprint" "Connector_PinHeader_2.54mm:PinHeader_1x03_P2.54mm_Vertical" (at 262.89 88.9 0)
-      (effects (font (size 1.27 1.27)) hide)
-    )
-    (property "Datasheet" "~" (at 262.89 88.9 0)
-      (effects (font (size 1.27 1.27)) hide)
-    )
-    (pin "1")
-    (pin "2")
-    (pin "3")
-    (instances
-      (project "qca7000"
-        (path "/e63e39d7-6ac0-4ffd-8aa3-1841a4541b55/5666e7cf-6b6c-4583-8335-aa3be69ccd45"
-          (reference "J3") (unit 1)
-        )
-      )
-    )
-  )
   (symbol (lib_id "Connector:Conn_01x03_Pin") (at 256.54 154.94 180) (unit 1)
     (in_bom yes) (on_board yes) (dnp no) (fields_autoplaced)
@@
         )
       )
-    )
-  )
-  (symbol (lib_id "power:GND") (at 257.81 88.9 270) (unit 1)
-    (in_bom yes) (on_board yes) (dnp no)
-    (property "Reference" "#PWR048" (at 251.46 88.9 0)
-      (effects (font (size 1.27 1.27)) hide)
-    )
-    (property "Value" "GND" (at 255.27 88.9 90)
-      (effects (font (size 1.27 1.27)) (justify right))
-    )
-    (property "Footprint" "" (at 257.81 88.9 0)
-      (effects (font (size 1.27 1.27)) hide)
-    )
-    (property "Datasheet" "" (at 257.81 88.9 0)
-      (effects (font (size 1.27 1.27)) hide)
-    )
-    (pin "1")
-    (instances
-      (project "qca7000"
-        (path "/e63e39d7-6ac0-4ffd-8aa3-1841a4541b55"
-          (reference "#PWR048") (unit 1)
-        )
-        (path "/e63e39d7-6ac0-4ffd-8aa3-1841a4541b55/5666e7cf-6b6c-4583-8335-aa3be69ccd45"
-          (reference "#PWR049") (unit 1)
-        )
-      )
