File: pcb/controller.kicad_sch (KiCad schematic)
At the start: 59 parts, among them J16 uC_NRST, J17 3V3_uC, J18 SWO, J4 DEBUG, J5 UART, U2 SN65HVD234, U3 STM32F103RETx, Y1 8MHz

Commit message: routed driver outputs for contactors and lock motor to PWM TIM3 ports. Use protected 12V for DRV.
Parts:
- removed TP5V1 (x4): ~, TestPoint:TestPoint_THTPad_D1.0mm_Drill0.5mm, symbol Connector:TestPoint
- added TP5V1 (x4): ~, TestPoint:TestPoint_THTPad_D1.0mm_Drill0.5mm, symbol Connector:TestPoint
Connections:
- net CONTACTOR_CONTROL1: now also U3.39 (PC8); no longer U3.57 (PB5)
- net CONTACTOR_CONTROL2: now also U3.40 (PC9); no longer U3.58 (PB6)
- net DRV_IN1: now also U3.37 (PC6); no longer U3.33 (PB12)
- net DRV_IN2: now also U3.38 (PC7); no longer U3.34 (PB13)
- new net: TP5V1.1, U3.58 (PB6)
- new net: TP5V1.1, U3.33 (PB12)
- new net: TP5V1.1, U3.34 (PB13)
- new net: TP5V1.1, U3.57 (PB5)

Commit message: all 100nF now 0805. Todo list cleaned up.
Parts:
- C61: footprint Capacitor_SMD:C_1206_3216Metric_Pad1.33x1.80mm_HandSolder -> Capacitor_SMD:C_0805_2012Metric_Pad1.18x1.45mm_HandSolder
Changed lines of the file:
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@@
       (effects (font (size 1.27 1.27)))
     )
-    (property "Footprint" "Capacitor_SMD:C_1206_3216Metric_Pad1.33x1.80mm_HandSolder" (at 110.49 46.99 0)
+    (property "Footprint" "Capacitor_SMD:C_0805_2012Metric_Pad1.18x1.45mm_HandSolder" (at 110.49 46.99 0)
       (effects (font (size 1.27 1.27)) hide)
     )

Commit message: added CP sensing. Added 5V on the connector. Created gerber and pdf
Parts:
- removed TP5V1: ~, TestPoint:TestPoint_THTPad_D1.0mm_Drill0.5mm, symbol Connector:TestPoint
Connections:
- net CP_SENSE: now reaches U3.50 (PA15)
Changed lines of the file:
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@@
+    )
+  )
+  (global_label "CP_SENSE" (shape input) (at 176.53 102.87 0) (fields_autoplaced)
+    (effects (font (size 1.27 1.27)) (justify left))
+    (property "Intersheetrefs" "${INTERSHEET_REFS}" (at 188.9909 102.87 0)
+      (effects (font (size 1.27 1.27)) (justify left) hide)
     )
   )
@@
         )
       )
-    )
-  )
-  (symbol (lib_id "Connector:TestPoint") (at 176.53 102.87 270) (unit 1)
-    (in_bom yes) (on_board yes) (dnp no)
-    (property "Reference" "TP5V1" (at 181.61 102.87 90)
-      (effects (font (size 1.27 1.27)) (justify left))
-    )
-    (property "Value" "~" (at 181.61 101.6 0)
-      (effects (font (size 1.27 1.27)) (justify left))
-    )
-    (property "Footprint" "TestPoint:TestPoint_THTPad_D1.0mm_Drill0.5mm" (at 176.53 107.95 0)
-      (effects (font (size 1.27 1.27)) hide)
-    )
-    (property "Datasheet" "~" (at 176.53 107.95 0)
-      (effects (font (size 1.27 1.27)) hide)
-    )
-    (pin "1")
-    (instances
-      (project "qca7000"
-        (path "/e63e39d7-6ac0-4ffd-8aa3-1841a4541b55"
-          (reference "TP5V1") (unit 1)
-        )
-        (path "/e63e39d7-6ac0-4ffd-8aa3-1841a4541b55/81db238c-e53f-4d52-98ea-36a1df697651"
-          (reference "TP5V1") (unit 1)
-        )
-        (path "/e63e39d7-6ac0-4ffd-8aa3-1841a4541b55/5666e7cf-6b6c-4583-8335-aa3be69ccd45"
-          (reference "TP20") (unit 1)
-        )
-      )

Commit message: added some jlcpcb part numbers, adjusted some footprints and values accordingly.
Parts:
- C17: value 22p -> 22pF; LCSC C1679 -> C1804; LINK (none) -> https://jlcpcb.com/partdetail/2156-CL21C220JBANNNC/C1804
- C61: LCSC C14663 -> C49678; LINK (none) -> https://jlcpcb.com/partdetail/Yageo-CC0805KRX7R9BB104/C49678
- C67: footprint Capacitor_SMD:C_1210_3225Metric_Pad1.33x2.70mm_HandSolder -> Capacitor_SMD:C_0805_2012Metric_Pad1.18x1.45mm_HandSolder; LCSC tbd -> C28323; LINK (none) -> https://jlcpcb.com/partdetail/29074-CL21B105KBFNNNE/C28323
- R5: footprint Resistor_SMD:R_1206_3216Metric_Pad1.30x1.75mm_HandSolder -> Resistor_SMD:R_0805_2012Metric_Pad1.20x1.40mm_HandSolder; LCSC C23140 -> C17634; LINK (none) -> https://jlcpcb.com/partdetail/18322-0805W8F330JT5E/C17634
- Y1: value 8MHz -> 12MHz; LCSC tbd -> C9002; LINK (none) -> https://jlcpcb.com/partdetail/YangxingTech-X322512MSB4SI/C9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
Changed lines of the file:
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@@
       (effects (font (size 1.27 1.27)) hide)
     )
-    (property "LCSC" "C14663" (at 110.49 46.99 90)
+    (property "LCSC" "C49678" (at 110.49 46.99 90)
+      (effects (font (size 1.27 1.27)) hide)
+    )
+    (property "LINK" "https://jlcpcb.com/partdetail/Yageo-CC0805KRX7R9BB104/C49678" (at 110.49 46.99 0)
       (effects (font (size 1.27 1.27)) hide)
     )
@@
       (effects (font (size 1.27 1.27)) hide)
     )
-    (property "LCSC" "C14663" (at 166.37 57.15 90)
+    (property "LCSC" "C49678" (at 166.37 57.15 90)
+      (effects (font (size 1.27 1.27)) hide)
+    )
+    (property "LINK" "https://jlcpcb.com/partdetail/Yageo-CC0805KRX7R9BB104/C49678" (at 166.37 57.15 0)
       (effects (font (size 1.27 1.27)) hide)
     )
@@
       (effects (font (size 1.27 1.27)))
     )
-    (property "Value" "22p" (at 86.36 62.23 90)
+    (property "Value" "22pF" (at 86.36 62.23 90)
       (effects (font (size 1.27 1.27)))
     )
@@
       (effects (font (size 1.27 1.27)) hide)
     )
-    (property "LCSC" "C1679" (at 82.55 64.77 0)
+    (property "LCSC" "C1804" (at 82.55 64.77 0)
+      (effects (font (size 1.27 1.27)) hide)
+    )
+    (property "LINK" "https://jlcpcb.com/partdetail/2156-CL21C220JBANNNC/C1804" (at 82.55 64.77 0)
       (effects (font (size 1.27 1.27)) hide)
     )
@@
       (effects (font (size 1.27 1.27)) hide)
     )
-    (property "LCSC" "C14663" (at 64.77 25.4 90)
+    (property "LCSC" "C49678" (at 64.77 25.4 90)
+      (effects (font (size 1.27 1.27)) hide)
+    )
+    (property "LINK" "https://jlcpcb.com/partdetail/Yageo-CC0805KRX7R9BB104/C49678" (at 64.77 25.4 0)
       (effects (font (size 1.27 1.27)) hide)
     )
@@
       (effects (font (size 1.27 1.27)))
     )
-    (property "Footprint" "Capacitor_SMD:C_1210_3225Metric_Pad1.33x2.70mm_HandSolder" (at 166.37 44.45 0)
+    (property "Footprint" "Capacitor_SMD:C_0805_2012Metric_Pad1.18x1.45mm_HandSolder" (at 166.37 44.45 0)
       (effects (font (size 1.27 1.27)) hide)
     )
@@
       (effects (font (size 1.27 1.27)) hide)
     )
-    (property "LCSC" "tbd" (at 166.37 44.45 90)
+    (property "LCSC" "C28323" (at 166.37 44.45 90)
+      (effects (font (size 1.27 1.27)) hide)
+    )
+    (property "LINK" "https://jlcpcb.com/partdetail/29074-CL21B105KBFNNNE/C28323" (at 166.37 44.45 0)
       (effects (font (size 1.27 1.27)) hide)
     )
@@
       (effects (font (size 1.27 1.27)))
     )
-    (property "Footprint" "Resistor_SMD:R_1206_3216Metric_Pad1.30x1.75mm_HandSolder" (at 99.06 76.2 0)
+    (property "Footprint" "Resistor_SMD:R_0805_2012Metric_Pad1.20x1.40mm_HandSolder" (at 99.06 76.2 0)
       (effects (font (size 1.27 1.27)) hide)
     )
@@
       (effects (font (size 1.27 1.27)) hide)
     )
-    (property "LCSC" "C23140" (at 99.06 76.2 90)
+    (property "LCSC" "C17634" (at 99.06 76.2 90)
+      (effects (font (size 1.27 1.27)) hide)
+    )
+    (property "LINK" "https://jlcpcb.com/partdetail/18322-0805W8F330JT5E/C17634" (at 99.06 76.2 0)
       (effects (font (size 1.27 1.27)) hide)
     )
@@
       (effects (font (size 1.27 1.27)) hide)
     )
-    (property "LCSC" "C14663" (at 53.34 25.4 90)
+    (property "LCSC" "C49678" (at 53.34 25.4 90)
+      (effects (font (size 1.27 1.27)) hide)
+    )
+    (property "LINK" "https://jlcpcb.com/partdetail/Yageo-CC0805KRX7R9BB104/C49678" (at 53.34 25.4 0)
       (effects (font (size 1.27 1.27)) hide)
     )
@@
       (effects (font (size 1.27 1.27)))
     )
-    (property "Value" "22p" (at 86.36 78.74 90)
+    (property "Value" "22pF" (at 86.36 78.74 90)
       (effects (font (size 1.27 1.27)))
     )
@@
       (effects (font (size 1.27 1.27)) hide)
     )
-    (property "LCSC" "C1679" (at 82.55 76.2 0)
+    (property "LCSC" "C1804" (at 82.55 76.2 0)
+      (effects (font (size 1.27 1.27)) hide)
+    )
+    (property "LINK" "https://jlcpcb.com/partdetail/2156-CL21C220JBANNNC/C1804" (at 82.55 76.2 0)
       (effects (font (size 1.27 1.27)) hide)
     )
@@
       (effects (font (size 1.27 1.27)) hide)
     )
-    (property "LCSC" "C14663" (at 76.2 25.4 90)
+    (property "LCSC" "C49678" (at 76.2 25.4 90)
+      (effects (font (size 1.27 1.27)) hide)
+    )
+    (property "LINK" "https://jlcpcb.com/partdetail/Yageo-CC0805KRX7R9BB104/C49678" (at 76.2 25.4 0)
       (effects (font (size 1.27 1.27)) hide)
     )
@@
       (effects (font (size 1.27 1.27)))
     )
-    (property "Value" "8MHz" (at 80.01 71.12 90)
+    (property "Value" "12MHz" (at 80.01 71.12 90)
       (effects (font (size 1.27 1.27)))
     )
@@
       (effects (font (size 1.27 1.27)) hide)
     )
-    (property "LCSC" "tbd" (at 92.71 71.12 0)
+    (property "LCSC" "C9002" (at 92.71 71.12 0)
+      (effects (font (size 1.27 1.27)) hide)
+    )
+    (property "LINK" "https://jlcpcb.com/partdetail/YangxingTech-X322512MSB4SI/C9002" (at 92.71 71.12 0)
       (effects (font (size 1.27 1.27)) hide)
     )
@@
       (effects (font (size 1.27 1.27)) hide)
     )
-    (property "LCSC" "C14663" (at 40.64 25.4 90)
-      (effects (font (size 1.27 1.27)) hide)
-    )
+    (property "LCSC" "C49678" (at 40.64 25.4 90)
+      (effects (font (size 1.27 1.27)) hide)
+    )
+    (property "LINK" "https://jlcpcb.com/partdetail/Yageo-CC0805KRX7R9BB104/C49678" (at 40.64 25.4 0)
+      (effects (font (size 1.27 1.27)) hide)
+    )

Commit message: added more part numbers
Parts:
- D10, D11, D12, D15, D9: LCSC (none) -> C2296; LINK (none) -> https://jlcpcb.com/partdetail/Hubei_KentoElec-C2296/C2296
- R3: footprint Resistor_SMD:R_1206_3216Metric_Pad1.30x1.75mm_HandSolder -> Resistor_SMD:R_0805_2012Metric_Pad1.20x1.40mm_HandSolder; LCSC C22978 -> C17557; LINK (none) -> https://jlcpcb.com/partdetail/18245-0805W8F2200T5E/C17557
- U2: value SN65HVD234 -> SN65HVD230; LCSC (none) -> C12084; LINK (none) -> https://jlcpcb.com/partdetail/TexasInstruments-SN65HVD230DR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
- U3: LCSC (none) -> C8322; LINK (none) -> https://jlcpcb.com/partdetail/Stmicroelectronics-STM32F103R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
Changed lines of the file:
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@@
       (effects (font (size 1.27 1.27)) (justify left))
     )
-    (property "Value" "SN65HVD234" (at 234.3659 81.28 0)
+    (property "Value" "SN65HVD230" (at 234.3659 81.28 0)
       (effects (font (size 1.27 1.27)) (justify left))
     )
@@
     )
     (property "Datasheet" "http://www.ti.com/lit/ds/symlink/sn65hvd234.pdf" (at 229.87 77.47 0)
+      (effects (font (size 1.27 1.27)) hide)
+    )
+    (property "LCSC" "C12084" (at 232.41 87.63 0)
+      (effects (font (size 1.27 1.27)) hide)
+    )
+    (property "LINK" "https://jlcpcb.com/partdetail/TexasInstruments-SN65HVD230DR/C12084" (at 232.41 87.63 0)
       (effects (font (size 1.27 1.27)) hide)
     )
@@
       (effects (font (size 1.27 1.27)) hide)
     )
+    (property "LCSC" "C2296" (at 63.5 114.3 0)
+      (effects (font (size 1.27 1.27)) hide)
+    )
+    (property "LINK" "https://jlcpcb.com/partdetail/Hubei_KentoElec-C2296/C2296" (at 63.5 114.3 0)
+      (effects (font (size 1.27 1.27)) hide)
+    )
     (pin "1")
     (pin "2")
@@
       (effects (font (size 1.27 1.27)))
     )
-    (property "Footprint" "Resistor_SMD:R_1206_3216Metric_Pad1.30x1.75mm_HandSolder" (at 247.65 157.48 0)
+    (property "Footprint" "Resistor_SMD:R_0805_2012Metric_Pad1.20x1.40mm_HandSolder" (at 247.65 157.48 0)
       (effects (font (size 1.27 1.27)) hide)
     )
@@
       (effects (font (size 1.27 1.27)) hide)
     )
-    (property "LCSC" "C22978" (at 247.65 157.48 90)
+    (property "LCSC" "C17557" (at 247.65 157.48 90)
+      (effects (font (size 1.27 1.27)) hide)
+    )
+    (property "LINK" "https://jlcpcb.com/partdetail/18245-0805W8F2200T5E/C17557" (at 247.65 157.48 0)
       (effects (font (size 1.27 1.27)) hide)
     )
@@
       (effects (font (size 1.27 1.27)))
     )
-    (property "Footprint" "Resistor_SMD:R_1206_3216Metric_Pad1.30x1.75mm_HandSolder" (at 247.65 152.4 0)
+    (property "Footprint" "Resistor_SMD:R_0805_2012Metric_Pad1.20x1.40mm_HandSolder" (at 247.65 152.4 0)
       (effects (font (size 1.27 1.27)) hide)
     )
@@
       (effects (font (size 1.27 1.27)) hide)
     )
-    (property "LCSC" "C22978" (at 247.65 152.4 90)
+    (property "LCSC" "C17557" (at 247.65 152.4 90)
+      (effects (font (size 1.27 1.27)) hide)
+    )
+    (property "LINK" "https://jlcpcb.com/partdetail/18245-0805W8F2200T5E/C17557" (at 247.65 152.4 0)
       (effects (font (size 1.27 1.27)) hide)
     )
@@
       (effects (font (size 1.27 1.27)) hide)
     )
+    (property "LCSC" "C2296" (at 63.5 132.08 0)
+      (effects (font (size 1.27 1.27)) hide)
+    )
+    (property "LINK" "https://jlcpcb.com/partdetail/Hubei_KentoElec-C2296/C2296" (at 63.5 132.08 0)
+      (effects (font (size 1.27 1.27)) hide)
+    )
     (pin "1")
     (pin "2")
@@
       (effects (font (size 1.27 1.27)))
     )
-    (property "Footprint" "Resistor_SMD:R_1206_3216Metric_Pad1.30x1.75mm_HandSolder" (at 233.68 46.99 0)
+    (property "Footprint" "Resistor_SMD:R_0805_2012Metric_Pad1.20x1.40mm_HandSolder" (at 233.68 46.99 0)
       (effects (font (size 1.27 1.27)) hide)
     )
@@
       (effects (font (size 1.27 1.27)) hide)
     )
-    (property "LCSC" "C22978" (at 233.68 46.99 90)
+    (property "LCSC" "C17557" (at 233.68 46.99 90)
+      (effects (font (size 1.27 1.27)) hide)
+    )
+    (property "LINK" "https://jlcpcb.com/partdetail/18245-0805W8F2200T5E/C17557" (at 233.68 46.99 0)
       (effects (font (size 1.27 1.27)) hide)
     )
@@
     )
     (property "Datasheet" "https://www.st.com/resource/en/datasheet/stm32f103re.pdf" (at 153.67 107.95 0)
+      (effects (font (size 1.27 1.27)) hide)
+    )
+    (property "LCSC" "C8322" (at 153.67 107.95 0)
+      (effects (font (size 1.27 1.27)) hide)
+    )
+    (property "LINK" "https://jlcpcb.com/partdetail/Stmicroelectronics-STM32F103RET6/C8322" (at 153.67 107.95 0)
       (effects (font (size 1.27 1.27)) hide)
     )
@@
       (effects (font (size 1.27 1.27)))
     )
-    (property "Footprint" "Resistor_SMD:R_1206_3216Metric_Pad1.30x1.75mm_HandSolder" (at 233.68 40.64 0)
+    (property "Footprint" "Resistor_SMD:R_0805_2012Metric_Pad1.20x1.40mm_HandSolder" (at 233.68 40.64 0)
       (effects (font (size 1.27 1.27)) hide)
     )
@@
       (effects (font (size 1.27 1.27)) hide)
     )
-    (property "LCSC" "C22978" (at 233.68 40.64 90)
+    (property "LCSC" "C17557" (at 233.68 40.64 90)
+      (effects (font (size 1.27 1.27)) hide)
+    )
+    (property "LINK" "https://jlcpcb.com/partdetail/18245-0805W8F2200T5E/C17557" (at 233.68 40.64 0)
       (effects (font (size 1.27 1.27)) hide)
     )
@@
       (effects (font (size 1.27 1.27)))
     )
-    (property "Footprint" "Resistor_SMD:R_1206_3216Metric_Pad1.30x1.75mm_HandSolder" (at 233.68 59.69 0)
+    (property "Footprint" "Resistor_SMD:R_0805_2012Metric_Pad1.20x1.40mm_HandSolder" (at 233.68 59.69 0)
       (effects (font (size 1.27 1.27)) hide)
     )
@@
       (effects (font (size 1.27 1.27)) hide)
     )
-    (property "LCSC" "C22978" (at 233.68 59.69 90)
+    (property "LCSC" "C17557" (at 233.68 59.69 90)
+      (effects (font (size 1.27 1.27)) hide)
+    )
+    (property "LINK" "https://jlcpcb.com/partdetail/18245-0805W8F2200T5E/C17557" (at 233.68 59.69 0)
       (effects (font (size 1.27 1.27)) hide)
     )
@@
     )
     (property "Datasheet" "~" (at 63.5 123.19 0)
+      (effects (font (size 1.27 1.27)) hide)
+    )
+    (property "LCSC" "C2296" (at 63.5 123.19 0)
+      (effects (font (size 1.27 1.27)) hide)
+    )
+    (property "LINK" "https://jlcpcb.com/partdetail/Hubei_KentoElec-C2296/C2296" (at 63.5 123.19 0)
       (effects (font (size 1.27 1.27)) hide)
     )
@@
       (effects (font (size 1.27 1.27)))
     )
-    (property "Footprint" "Resistor_SMD:R_1206_3216Metric_Pad1.30x1.75mm_HandSolder" (at 233.68 53.34 0)
+    (property "Footprint" "Resistor_SMD:R_0805_2012Metric_Pad1.20x1.40mm_HandSolder" (at 233.68 53.34 0)
       (effects (font (size 1.27 1.27)) hide)
     )
@@
       (effects (font (size 1.27 1.27)) hide)
     )
-    (property "LCSC" "C22978" (at 233.68 53.34 90)
+    (property "LCSC" "C17557" (at 233.68 53.34 90)
+      (effects (font (size 1.27 1.27)) hide)
+    )
+    (property "LINK" "https://jlcpcb.com/partdetail/18245-0805W8F2200T5E/C17557" (at 233.68 53.34 0)
       (effects (font (size 1.27 1.27)) hide)
     )
@@
       (effects (font (size 1.27 1.27)) hide)
     )
+    (property "LCSC" "C2296" (at 63.5 105.41 0)
+      (effects (font (size 1.27 1.27)) hide)
+    )
+    (property "LINK" "https://jlcpcb.com/partdetail/Hubei_KentoElec-C2296/C2296" (at 63.5 105.41 0)
+      (effects (font (size 1.27 1.27)) hide)
+    )
     (pin "1")
     (pin "2")
@@
       (effects (font (size 1.27 1.27)) hide)
     )
+    (property "LCSC" "C2296" (at 63.5 96.52 0)
+      (effects (font (size 1.27 1.27)) hide)
+    )
+    (property "LINK" "https://jlcpcb.com/partdetail/Hubei_KentoElec-C2296/C2296" (at 63.5 96.52 0)
+      (effects (font (size 1.27 1.27)) hide)
+    )

Commit message: more partnumbers assigned. split difficult values into two parts. add protection of CP_SENSE port
Parts:
- L10: LCSC C1002 -> C1017; LINK (none) -> https://jlcpcb.com/partdetail/Sunlord-GZ2012D601TF/C1017
- R3: footprint Resistor_SMD:R_1206_3216Metric_Pad1.30x1.75mm_HandSolder -> Resistor_SMD:R_0805_2012Metric_Pad1.20x1.40mm_HandSolder; LCSC C22978 -> C17513; LINK (none) -> https://jlcpcb.com/partdetail/18201-0805W8F1001T5E/C17513
Changed lines of the file:
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@@
       (effects (font (size 1.27 1.27)))
     )
-    (property "Footprint" "Resistor_SMD:R_1206_3216Metric_Pad1.30x1.75mm_HandSolder" (at 53.34 105.41 0)
+    (property "Footprint" "Resistor_SMD:R_0805_2012Metric_Pad1.20x1.40mm_HandSolder" (at 53.34 105.41 0)
       (effects (font (size 1.27 1.27)) hide)
     )
@@
       (effects (font (size 1.27 1.27)) hide)
     )
-    (property "LCSC" "C22978" (at 53.34 105.41 90)
+    (property "LCSC" "C17513" (at 53.34 105.41 90)
+      (effects (font (size 1.27 1.27)) hide)
+    )
+    (property "LINK" "https://jlcpcb.com/partdetail/18201-0805W8F1001T5E/C17513" (at 53.34 105.41 0)
       (effects (font (size 1.27 1.27)) hide)
     )
@@
       (effects (font (size 1.27 1.27)))
     )
-    (property "Footprint" "Resistor_SMD:R_1206_3216Metric_Pad1.30x1.75mm_HandSolder" (at 248.92 88.9 0)
+    (property "Footprint" "Resistor_SMD:R_0805_2012Metric_Pad1.20x1.40mm_HandSolder" (at 248.92 88.9 0)
       (effects (font (size 1.27 1.27)) hide)
     )
@@
       (effects (font (size 1.27 1.27)) hide)
     )
-    (property "LCSC" "C22978" (at 248.92 88.9 90)
+    (property "LCSC" "C17513" (at 248.92 88.9 90)
+      (effects (font (size 1.27 1.27)) hide)
+    )
+    (property "LINK" "https://jlcpcb.com/partdetail/18201-0805W8F1001T5E/C17513" (at 248.92 88.9 0)
       (effects (font (size 1.27 1.27)) hide)
     )
@@
       (effects (font (size 1.27 1.27)) hide)
     )
-    (property "LCSC" "C1002" (at 161.29 35.56 0)
+    (property "LCSC" "C1017" (at 161.29 35.56 0)
+      (effects (font (size 1.27 1.27)) hide)
+    )
+    (property "LINK" "https://jlcpcb.com/partdetail/Sunlord-GZ2012D601TF/C1017" (at 161.29 35.56 0)
       (effects (font (size 1.27 1.27)) hide)
     )
@@
       (effects (font (size 1.27 1.27)))
     )
-    (property "Footprint" "Resistor_SMD:R_1206_3216Metric_Pad1.30x1.75mm_HandSolder" (at 53.34 132.08 0)
+    (property "Footprint" "Resistor_SMD:R_0805_2012Metric_Pad1.20x1.40mm_HandSolder" (at 53.34 132.08 0)
       (effects (font (size 1.27 1.27)) hide)
     )
@@
       (effects (font (size 1.27 1.27)) hide)
     )
-    (property "LCSC" "C22978" (at 53.34 132.08 90)
+    (property "LCSC" "C17513" (at 53.34 132.08 90)
+      (effects (font (size 1.27 1.27)) hide)
+    )
+    (property "LINK" "https://jlcpcb.com/partdetail/18201-0805W8F1001T5E/C17513" (at 53.34 132.08 0)
       (effects (font (size 1.27 1.27)) hide)
     )
@@
       (effects (font (size 1.27 1.27)))
     )
-    (property "Footprint" "Resistor_SMD:R_1206_3216Metric_Pad1.30x1.75mm_HandSolder" (at 53.34 114.3 0)
+    (property "Footprint" "Resistor_SMD:R_0805_2012Metric_Pad1.20x1.40mm_HandSolder" (at 53.34 114.3 0)
       (effects (font (size 1.27 1.27)) hide)
     )
@@
       (effects (font (size 1.27 1.27)) hide)
     )
-    (property "LCSC" "C22978" (at 53.34 114.3 90)
+    (property "LCSC" "C17513" (at 53.34 114.3 90)
+      (effects (font (size 1.27 1.27)) hide)
+    )
+    (property "LINK" "https://jlcpcb.com/partdetail/18201-0805W8F1001T5E/C17513" (at 53.34 114.3 0)
       (effects (font (size 1.27 1.27)) hide)
     )
@@
       (effects (font (size 1.27 1.27)))
     )
-    (property "Footprint" "Resistor_SMD:R_1206_3216Metric_Pad1.30x1.75mm_HandSolder" (at 53.34 96.52 0)
+    (property "Footprint" "Resistor_SMD:R_0805_2012Metric_Pad1.20x1.40mm_HandSolder" (at 53.34 96.52 0)
       (effects (font (size 1.27 1.27)) hide)
     )
@@
       (effects (font (size 1.27 1.27)) hide)
     )
-    (property "LCSC" "C22978" (at 53.34 96.52 90)
+    (property "LCSC" "C17513" (at 53.34 96.52 90)
+      (effects (font (size 1.27 1.27)) hide)
+    )
+    (property "LINK" "https://jlcpcb.com/partdetail/18201-0805W8F1001T5E/C17513" (at 53.34 96.52 0)
       (effects (font (size 1.27 1.27)) hide)
     )
@@
       (effects (font (size 1.27 1.27)))
     )
-    (property "Footprint" "Resistor_SMD:R_1206_3216Metric_Pad1.30x1.75mm_HandSolder" (at 53.34 123.19 0)
+    (property "Footprint" "Resistor_SMD:R_0805_2012Metric_Pad1.20x1.40mm_HandSolder" (at 53.34 123.19 0)
       (effects (font (size 1.27 1.27)) hide)
     )
@@
       (effects (font (size 1.27 1.27)) hide)
     )
-    (property "LCSC" "C22978" (at 53.34 123.19 90)
-      (effects (font (size 1.27 1.27)) hide)
-    )
+    (property "LCSC" "C17513" (at 53.34 123.19 90)
+      (effects (font (size 1.27 1.27)) hide)
+    )
+    (property "LINK" "https://jlcpcb.com/partdetail/18201-0805W8F1001T5E/C17513" (at 53.34 123.19 0)
+      (effects (font (size 1.27 1.27)) hide)
+    )

Commit message: footprint corrections. some layout adaptions for new footprints (ongoing)
Other:
- note added: "8MHz would be "standard" as on the NUCLEO. But 8MHz is not available at JLCPCB, so we go for 12MHz."
- note removed: "Todo: XTAL frequency, footprint, Cs"
Changed lines of the file:
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@@
     (effects (font (size 1.27 1.27)) (justify left bottom))
   )
-  (text "Todo: XTAL frequency, footprint, Cs" (at 67.31 85.09 0)
+  (text "8MHz would be \"standard\" as on the NUCLEO.\nBut 8MHz is not available at JLCPCB, so\nwe go for 12MHz."
+    (at 29.21 74.93 0)
     (effects (font (size 1.27 1.27)) (justify left bottom))
   )
