File: pcb/controller.kicad_sch (KiCad schematic)
At the start: 58 parts, among them J16 uC_NRST, J17 3V3_uC, J18 SWO, J4 DEBUG, J5 UART, U2 SN65HVD230, U3 STM32F103RETx, Y1 12MHz

Commit message: BOM consolidation: XTAL options and back to 8MHz. Replace internal connectors by testpoints. Use T with integrated R for CP switching. Fix: Footprint Q7-Q9 corrected.
Parts:
- removed J16: uC_NRST, Connector_PinHeader_2.54mm:PinHeader_1x01_P2.54mm_Vertical, symbol Connector:Conn_01x01_Pin
- removed J17: 3V3_uC, Connector_PinHeader_2.54mm:PinHeader_1x01_P2.54mm_Vertical, symbol Connector:Conn_01x01_Pin
- removed J18: SWO, Connector_PinHeader_2.54mm:PinHeader_1x01_P2.54mm_Vertical, symbol Connector:Conn_01x01_Pin
- removed J4: DEBUG, Connector_PinHeader_2.54mm:PinHeader_1x03_P2.54mm_Vertical, symbol Connector:Conn_01x03_Pin
- removed J5: UART, Connector_PinHeader_2.54mm:PinHeader_1x03_P2.54mm_Vertical, symbol Connector:Conn_01x03_Pin
- added TP3 (x9): ~, speciallib:TestPoint_Special_THTPad_D1.9mm_Drill1mm, symbol Connector:TestPoint
- added Y3: 8MHz, Crystal:Crystal_SMD_5032-2Pin_5.0x3.2mm, symbol Device:Crystal
- Y1: value 12MHz -> 8MHz; LCSC C9002 -> none; LINK https://jlcpcb.com/partdetail/YangxingTech-X322512MSB4SI/C9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 -> (none)
Connections:
- net 3V3_uC: now also TP3.1
- net GND: now also C17.2, TP3.1, TP3.1; no longer C17.1
- net OCS_IN: now also C17.1, Y3.2; no longer C17.2
- net SWCLK: now also TP3.1
- net SWDIO: now also TP3.1
- net SWO: now also TP3.1
- net uC_NRST: now also TP3.1
- net at R3.2: now also TP3.1 (x2)
- net at C17.2, R5.1, Y1.3: now also Y3.1
Other:
- note added: "XTAL options: Use the two-pin on top, available at JLCPCB. Or use the four-pin on bottom, if available and handsolder is intended. Both 8 MHz."
- note removed: "8MHz would be "standard" as on the NUCLEO. But 8MHz is not available at JLCPCB, so we go for 12MHz."
- moved on the sheet: C17
