File: pcb/controller.kicad_sch (KiCad schematic)
At the start: 63 parts, among them U2 SN65HVD230, U3 STM32F103RETx, Y1 8MHz, Y3 8MHz

Commit message: added rotation attribute to get the correct footprint rotation at JLCPCB
Parts:
- U2, U3: JLCPCB Rotation Offset (none) -> -90
Changed lines of the file:
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@@
+      (effects (font (size 1.27 1.27)) hide)
+    )
+    (property "JLCPCB Rotation Offset" "-90" (at 232.41 87.63 0)
       (effects (font (size 1.27 1.27)) hide)
     )
@@
       (effects (font (size 1.27 1.27)) hide)
     )
+    (property "JLCPCB Rotation Offset" "-90" (at 153.67 107.95 0)
+      (effects (font (size 1.27 1.27)) hide)
+    )

Commit message: WIP: PP pull-up and divider. variant detection. ipropi connected to ADC.
Parts:
- removed TP5V1 (x2): ~, TestPoint:TestPoint_THTPad_D1.0mm_Drill0.5mm, symbol Connector:TestPoint
Connections:
- net ADC_HWVARIANT: now reaches U3.16 (PA2)
- net ADC_IPROPI: now reaches U3.17 (PA3)
Changed lines of the file:
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@@
+    )
+  )
+  (global_label "ADC_HWVARIANT" (shape input) (at 176.53 69.85 0) (fields_autoplaced)
+    (effects (font (size 1.27 1.27)) (justify left))
+    (property "Intersheetrefs" "${INTERSHEET_REFS}" (at 194.2526 69.85 0)
+      (effects (font (size 1.27 1.27)) (justify left) hide)
     )
   )
@@
     (property "Intersheetrefs" "${INTERSHEET_REFS}" (at 228.1133 152.4 0)
       (effects (font (size 1.27 1.27)) (justify right) hide)
+    )
+  )
+  (global_label "ADC_IPROPI" (shape input) (at 176.53 72.39 0) (fields_autoplaced)
+    (effects (font (size 1.27 1.27)) (justify left))
+    (property "Intersheetrefs" "${INTERSHEET_REFS}" (at 190.3821 72.39 0)
+      (effects (font (size 1.27 1.27)) (justify left) hide)
     )
   )
@@
         (path "/e63e39d7-6ac0-4ffd-8aa3-1841a4541b55/5666e7cf-6b6c-4583-8335-aa3be69ccd45"
           (reference "#PWR042") (unit 1)
-        )
-      )
-    )
-  )
-  (symbol (lib_id "Connector:TestPoint") (at 176.53 69.85 270) (unit 1)
-    (in_bom yes) (on_board yes) (dnp no)
-    (property "Reference" "TP5V1" (at 181.61 69.85 90)
-      (effects (font (size 1.27 1.27)) (justify left))
-    )
-    (property "Value" "~" (at 181.61 68.58 0)
-      (effects (font (size 1.27 1.27)) (justify left))
-    )
-    (property "Footprint" "TestPoint:TestPoint_THTPad_D1.0mm_Drill0.5mm" (at 176.53 74.93 0)
-      (effects (font (size 1.27 1.27)) hide)
-    )
-    (property "Datasheet" "~" (at 176.53 74.93 0)
-      (effects (font (size 1.27 1.27)) hide)
-    )
-    (pin "1")
-    (instances
-      (project "qca7000"
-        (path "/e63e39d7-6ac0-4ffd-8aa3-1841a4541b55"
-          (reference "TP5V1") (unit 1)
-        )
-        (path "/e63e39d7-6ac0-4ffd-8aa3-1841a4541b55/81db238c-e53f-4d52-98ea-36a1df697651"
-          (reference "TP5V1") (unit 1)
-        )
-        (path "/e63e39d7-6ac0-4ffd-8aa3-1841a4541b55/5666e7cf-6b6c-4583-8335-aa3be69ccd45"
-          (reference "TP9") (unit 1)
         )
       )
@@
         )
       )
-    )
-  )
-  (symbol (lib_id "Connector:TestPoint") (at 176.53 72.39 270) (unit 1)
-    (in_bom yes) (on_board yes) (dnp no)
-    (property "Reference" "TP5V1" (at 181.61 72.39 90)
-      (effects (font (size 1.27 1.27)) (justify left))
-    )
-    (property "Value" "~" (at 181.61 71.12 0)
-      (effects (font (size 1.27 1.27)) (justify left))
-    )
-    (property "Footprint" "TestPoint:TestPoint_THTPad_D1.0mm_Drill0.5mm" (at 176.53 77.47 0)
-      (effects (font (size 1.27 1.27)) hide)
-    )
-    (property "Datasheet" "~" (at 176.53 77.47 0)
-      (effects (font (size 1.27 1.27)) hide)
-    )
-    (pin "1")
-    (instances
-      (project "qca7000"
-        (path "/e63e39d7-6ac0-4ffd-8aa3-1841a4541b55"
-          (reference "TP5V1") (unit 1)
-        )
-        (path "/e63e39d7-6ac0-4ffd-8aa3-1841a4541b55/81db238c-e53f-4d52-98ea-36a1df697651"
-          (reference "TP5V1") (unit 1)
-        )
-        (path "/e63e39d7-6ac0-4ffd-8aa3-1841a4541b55/5666e7cf-6b6c-4583-8335-aa3be69ccd45"
-          (reference "TP10") (unit 1)
-        )
-      )

Commit message: feature: Added wakeup logic
Parts:
- removed TP5V1 (x2): ~, TestPoint:TestPoint_THTPad_D1.0mm_Drill0.5mm, symbol Connector:TestPoint
- renumbered TP3 to 3V3_uC1, C67 to C14, C61 to C56, C61 to C57, C61 to C58, C61 to C59, C61 to C60, C17 to C62, C17 to C63, L10 to L12, TP5V1 to PB12, TP5V1 to PB13, TP5V1 to PB5, TP5V1 to PB6, R3 to R11, R3 to R12, R3 to R13, R3 to R14, R5 to R15, R3 to R16, R3 to R17, R3 to R18, R3 to R19, R3 to R20, R3 to R21, R3 to R22, R3 to R37, TP3 to SWCLK1, TP3 to SWDIO1, TP3 to SWGND1, TP3 to SWO1, TP5V1 to TP11, TP5V1 to TP12, TP5V1 to TP13, TP5V1 to TP14, TP5V1 to TP26, TP5V1 to TP27, TP5V1 to TP28, TP5V1 to TP29, TP5V1 to TP30, TP5V1 to TP31, TP5V1 to TP38, TP5V1 to TP8, TP3 to UART_GND1, TP3 to UART_RX1, TP3 to UART_TX1, Y1 to Y2, TP3 to uC_NRST1
Connections:
- net TRIGGER_WAKEUP: now reaches U3.26 (PB0)
- net KEEP_POWER_ON: now reaches U3.27 (PB1)

Commit message: Using another motor driver IC for contactor control
Parts:
- removed TP8: ~, TestPoint:TestPoint_THTPad_D1.0mm_Drill0.5mm, symbol Connector:TestPoint
Connections:
- net CONTACTOR_ENABLE: now reaches U3.15 (PA1)
Changed lines of the file:
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@@
+    (stroke (width 0) (type default))
+  )
+  (wire (pts (xy 128.27 110.49) (xy 135.89 110.49))
+    (stroke (width 0) (type default))
+  )
+  (wire (pts (xy 171.45 100.33) (xy 175.26 100.33))
+    (stroke (width 0) (type default))
+  )
+  (wire (pts (xy 92.71 64.77) (xy 92.71 67.31))
+    (stroke (width 0) (type default))
+  )
+  (wire (pts (xy 67.31 114.3) (xy 71.12 114.3))
+    (stroke (width 0) (type default))
+  )
+  (wire (pts (xy 226.06 40.64) (xy 231.14 40.64))
+    (stroke (width 0) (type default))
+  )
+  (wire (pts (xy 44.45 105.41) (xy 50.8 105.41))
+    (stroke (width 0) (type default))
+  )
+  (wire (pts (xy 222.25 97.79) (xy 232.41 97.79))
+    (stroke (width 0) (type default))
+  )
+  (wire (pts (xy 236.22 120.65) (xy 240.03 120.65))
+    (stroke (width 0) (type default))
+  )
+  (wire (pts (xy 236.22 40.64) (xy 240.03 40.64))
+    (stroke (width 0) (type default))
+  )
+  (wire (pts (xy 92.71 83.82) (xy 92.71 87.63))
+    (stroke (width 0) (type default))
+  )
+  (wire (pts (xy 226.06 46.99) (xy 231.14 46.99))
+    (stroke (width 0) (type default))
+  )
+  (wire (pts (xy 171.45 80.01) (xy 175.26 80.01))
     (stroke (width 0) (type default))
   )
   (wire (pts (xy 171.45 67.31) (xy 176.53 67.31))
-    (stroke (width 0) (type default))
-  )
-  (wire (pts (xy 128.27 110.49) (xy 135.89 110.49))
-    (stroke (width 0) (type default))
-  )
-  (wire (pts (xy 171.45 100.33) (xy 175.26 100.33))
-    (stroke (width 0) (type default))
-  )
-  (wire (pts (xy 92.71 64.77) (xy 92.71 67.31))
-    (stroke (width 0) (type default))
-  )
-  (wire (pts (xy 67.31 114.3) (xy 71.12 114.3))
-    (stroke (width 0) (type default))
-  )
-  (wire (pts (xy 226.06 40.64) (xy 231.14 40.64))
-    (stroke (width 0) (type default))
-  )
-  (wire (pts (xy 44.45 105.41) (xy 50.8 105.41))
-    (stroke (width 0) (type default))
-  )
-  (wire (pts (xy 222.25 97.79) (xy 232.41 97.79))
-    (stroke (width 0) (type default))
-  )
-  (wire (pts (xy 236.22 120.65) (xy 240.03 120.65))
-    (stroke (width 0) (type default))
-  )
-  (wire (pts (xy 236.22 40.64) (xy 240.03 40.64))
-    (stroke (width 0) (type default))
-  )
-  (wire (pts (xy 92.71 83.82) (xy 92.71 87.63))
-    (stroke (width 0) (type default))
-  )
-  (wire (pts (xy 226.06 46.99) (xy 231.14 46.99))
-    (stroke (width 0) (type default))
-  )
-  (wire (pts (xy 171.45 80.01) (xy 175.26 80.01))
     (stroke (width 0) (type default))
   )
@@
     (effects (font (size 1.27 1.27)) (justify left))
     (property "Intersheetrefs" "${INTERSHEET_REFS}" (at 188.0234 80.01 0)
+      (effects (font (size 1.27 1.27)) (justify left) hide)
+    )
+  )
+  (global_label "CONTACTOR_ENABLE" (shape output) (at 176.53 67.31 0) (fields_autoplaced)
+    (effects (font (size 1.27 1.27)) (justify left))
+    (property "Intersheetrefs" "${INTERSHEET_REFS}" (at 198.3233 67.31 0)
       (effects (font (size 1.27 1.27)) (justify left) hide)
     )
@@
         )
       )
-    )
-  )
-  (symbol (lib_id "Connector:TestPoint") (at 176.53 67.31 270) (unit 1)
-    (in_bom yes) (on_board yes) (dnp no)
-    (property "Reference" "TP8" (at 181.61 67.31 90)
-      (effects (font (size 1.27 1.27)) (justify left))
-    )
-    (property "Value" "~" (at 181.61 66.04 0)
-      (effects (font (size 1.27 1.27)) (justify left))
-    )
-    (property "Footprint" "TestPoint:TestPoint_THTPad_D1.0mm_Drill0.5mm" (at 176.53 72.39 0)
-      (effects (font (size 1.27 1.27)) hide)
-    )
-    (property "Datasheet" "~" (at 176.53 72.39 0)
-      (effects (font (size 1.27 1.27)) hide)
-    )
-    (pin "1")
-    (instances
-      (project "qca7000"
-        (path "/e63e39d7-6ac0-4ffd-8aa3-1841a4541b55/5666e7cf-6b6c-4583-8335-aa3be69ccd45"
-          (reference "TP8") (unit 1)
-        )
-      )

Commit message: added alternative 6-pin headers. Added uart3 test points. V5.2pre2
Parts:
- added TP3, TP4: TestPoint, speciallib:TestPoint_Special_THTPad_D1.9mm_Drill1mm, symbol Connector:TestPoint
Connections:
- net LED_CTL_BLUE: now also TP4.1
- net LED_CTL_GREEN: now also TP3.1
Other:
- note added: "Spare serial interface UART3, could be used for serial flashing. Discussion: https://openinverter.org/forum/viewtopic.php?p=76465#p76465"
- moved on the sheet: R21, R22, UART_GND1, UART_RX1, UART_TX1

Commit message: corrected some rotations for JLC. Version 5.2p7
Parts:
- U2, U3: JLCPCB Rotation Offset -90 -> 0
Changed lines of the file:
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@@
 			)
 		)
-		(property "JLCPCB Rotation Offset" "-90"
+		(property "JLCPCB Rotation Offset" "0"
 			(at 232.41 87.63 0)
 			(effects
@@
 			)
 		)
-		(property "JLCPCB Rotation Offset" "-90"
+		(property "JLCPCB Rotation Offset" "0"
 			(at 153.67 107.95 0)
 			(effects

Commit message: Added TC2030 for programming STM32
Parts:
- added J6: Conn_ARM_SWD_TagConnect_TC2030, Connector:Tag-Connect_TC2030-IDC-FP_2x03_P1.27mm_Vertical, symbol Connector:Conn_ARM_SWD_TagConnect_TC2030
Connections:
- net 3V3_uC: now also J6.1 (VCC)
- net GND: now also J6.5 (GND)
- net SWCLK: now also J6.4 (SWCLK)
- net SWDIO: now also J6.2 (SWDIO)
Other:
- moved on the sheet: SWCLK1, SWDIO1, SWGND1
