File: pcb/outputdrivers.kicad_sch (KiCad schematic)
At the start: 15 parts, among them J7 CONTACTORS, J7 CP/PE, J7 RF, Q1 BC846, Q2 NCV8402xST, Q3 NCV8402xST, U7 74HCT04

Commit message: fix: divider on the stepdown. fix: non-inverted contactor drivers. fix: part number of 8MHz. add: mounting holes and spare grid. add: LIM HVDC input. docu: todo list
Connections:
- net 3V3_uC is gone; now on net GND: R11.1, R11.2
- net CONTACTOR_CONTROL1: now also U7.3; no longer U7.5
- net CONTACTOR_CONTROL2: now also U7.11; no longer U7.9
- net at U7.2: no longer U7.3
- net at U7.12: no longer U7.11
- net at U7.10: now also U7.9
- net at U7.4: now also U7.5
Other:
- note added: "HCT as level shifter from 3.3V to 5V, because the NCV needs at least 5V gate voltage. Non-inverting is important, so that a fail of the 3V3 will lead to "contactors off"."
- note added: "pull down, to make sure that if the controller is in reset, the contactors are off."
- note removed: "HCT as level shifter from 3.3V to 5V, because the NCV needs at least 5V gate voltage"
- note removed: "pull up, to make sure that if the controller is in reset, the contactors are off."
- moved on the sheet: J7, Q2, Q3, U7B, U7C, U7D, U7E

Commit message: added TE DEUTSCH connector and housing
Parts:
- removed J7: CONTACTORS, Connector_PinHeader_2.54mm:PinHeader_1x02_P2.54mm_Vertical, symbol Connector:Conn_01x02_Pin
Changed lines of the file:
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@@
-    (stroke (width 0) (type default))
-  )
-  (wire (pts (xy 140.97 100.33) (xy 143.51 100.33))
     (stroke (width 0) (type default))
   )
@@
   )
   (wire (pts (xy 93.98 35.56) (xy 97.79 35.56))
-    (stroke (width 0) (type default))
-  )
-  (wire (pts (xy 140.97 102.87) (xy 143.51 102.87))
     (stroke (width 0) (type default))
   )
@@
     (at 121.92 88.9 0)
     (effects (font (size 1.27 1.27)) (justify left bottom))
-  )
-  (global_label "CONTACTOR1_LS" (shape input) (at 140.97 100.33 180) (fields_autoplaced)
-    (effects (font (size 1.27 1.27)) (justify right))
-    (property "Intersheetrefs" "${INTERSHEET_REFS}" (at 122.8242 100.33 0)
-      (effects (font (size 1.27 1.27)) (justify right) hide)
-    )
   )
   (global_label "5V" (shape input) (at 67.31 153.67 0) (fields_autoplaced)
@@
     (effects (font (size 1.27 1.27)) (justify right))
     (property "Intersheetrefs" "${INTERSHEET_REFS}" (at 81.0957 35.56 0)
-      (effects (font (size 1.27 1.27)) (justify right) hide)
-    )
-  )
-  (global_label "CONTACTOR2_LS" (shape input) (at 140.97 102.87 180) (fields_autoplaced)
-    (effects (font (size 1.27 1.27)) (justify right))
-    (property "Intersheetrefs" "${INTERSHEET_REFS}" (at 122.8242 102.87 0)
       (effects (font (size 1.27 1.27)) (justify right) hide)
     )
@@
         )
       )
-    )
-  )
-  (symbol (lib_id "Connector:Conn_01x02_Pin") (at 148.59 102.87 180) (unit 1)
-    (in_bom yes) (on_board yes) (dnp no) (fields_autoplaced)
-    (property "Reference" "J7" (at 149.86 100.965 0)
-      (effects (font (size 1.27 1.27)) (justify right))
-    )
-    (property "Value" "CONTACTORS" (at 149.86 103.505 0)
-      (effects (font (size 1.27 1.27)) (justify right))
-    )
-    (property "Footprint" "Connector_PinHeader_2.54mm:PinHeader_1x02_P2.54mm_Vertical" (at 148.59 102.87 0)
-      (effects (font (size 1.27 1.27)) hide)
-    )
-    (property "Datasheet" "~" (at 148.59 102.87 0)
-      (effects (font (size 1.27 1.27)) hide)
-    )
-    (pin "1")
-    (pin "2")
-    (instances
-      (project "qca7000"
-        (path "/e63e39d7-6ac0-4ffd-8aa3-1841a4541b55/5666e7cf-6b6c-4583-8335-aa3be69ccd45"
-          (reference "J7") (unit 1)
-        )
-        (path "/e63e39d7-6ac0-4ffd-8aa3-1841a4541b55/539ec63d-ac7e-42ea-858e-ff2bf33430ea"
-          (reference "J8") (unit 1)
-        )
-      )

Commit message: added RGB LED highside drivers
Parts:
- added Q4 (x3): DTA143Z, Package_TO_SOT_SMD:SOT-23, symbol Transistor_BJT:DTA143Z
- added Q7: DTC114E, Package_TO_SOT_SMD:SOT-23, symbol Transistor_BJT:DTC114E
- added Q8, Q9: DTC114E, Package_TO_SOT_SMD:SOT-23, symbol Transistor_BJT:DTC113Z
- added R3 (x3): 220, Resistor_SMD:R_1206_3216Metric_Pad1.30x1.75mm_HandSolder, symbol Device:R_Small
Connections:
- net GND: now also Q7.2 (E), Q8.2 (E), Q9.2 (E)
- new net: Q4.1 (B), Q7.3 (C)
- new net: Q4.1 (B), Q8.3 (C)
- new net: Q4.3 (C), R3.2 (x3)
- new net: Q4.1 (B), Q9.3 (C)
- new net 12V_P: Q4.2 (E), Q4.2 (E), Q4.2 (E)
- new net LED_BLUE: R3.1
- new net LED_CTL_BLUE: Q9.1 (B)
- new net LED_CTL_GREEN: Q8.1 (B)
- new net LED_CTL_RED: Q7.1 (B)
- new net LED_GREEN: R3.1
- new net LED_RED: R3.1
Other:
- note added: "12V highside outputs for the LEDs in the button. (or low-current-general-purpose)"
- note added: "Series resistors to protect the output in case of short circuit. With 12V and 220ohms we get 54mA and 0.6W. This may burn the resistors after a short time, but better than burning the transistors."

Commit message: first draft with the DRV8874 hbridge driver. Added 3D models.
Parts:
- added IC1: DRV8874QPWPRQ1, SOP65P640X120-17N, symbol DRV8874QPWPRQ1:DRV8874QPWPRQ1
Connections:
- net GND: now also IC1.15 (GND), IC1.9 (PGND)
- new net CONN_LOCK_MOT1: IC1.8 (OUT1)
- new net CONN_LOCK_MOT2: IC1.10 (OUT2)
Changed lines of the file:
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@@
   (junction (at 57.15 39.37) (diameter 0) (color 0 0 0 0)
+  )
+  (junction (at 238.76 144.78) (diameter 0) (color 0 0 0 0)
   )
   (no_connect (at 100.33 184.15))
   (no_connect (at 43.18 187.96))
+  (wire (pts (xy 238.76 129.54) (xy 238.76 144.78))
+    (stroke (width 0) (type default))
+  )
   (wire (pts (xy 250.19 53.34) (xy 270.51 53.34))
     (stroke (width 0) (type default))
@@
     (stroke (width 0) (type default))
   )
+  (wire (pts (xy 234.95 142.24) (xy 251.46 142.24))
+    (stroke (width 0) (type default))
+  )
   (wire (pts (xy 229.87 97.79) (xy 229.87 87.63))
     (stroke (width 0) (type default))
   )
+  (wire (pts (xy 234.95 129.54) (xy 238.76 129.54))
+    (stroke (width 0) (type default))
+  )
   (wire (pts (xy 203.2 87.63) (xy 208.28 87.63))
     (stroke (width 0) (type default))
@@
     (stroke (width 0) (type default))
   )
+  (wire (pts (xy 189.23 144.78) (xy 199.39 144.78))
+    (stroke (width 0) (type default))
+  )
   (wire (pts (xy 240.03 64.77) (xy 240.03 58.42))
     (stroke (width 0) (type default))
@@
   )
   (wire (pts (xy 48.26 106.68) (xy 48.26 110.49))
+    (stroke (width 0) (type default))
+  )
+  (wire (pts (xy 234.95 144.78) (xy 238.76 144.78))
     (stroke (width 0) (type default))
   )
@@
     (effects (font (size 1.27 1.27)) (justify left bottom))
   )
+  (global_label "CONN_LOCK_MOT1" (shape output) (at 189.23 144.78 180) (fields_autoplaced)
+    (effects (font (size 1.27 1.27)) (justify right))
+    (property "Intersheetrefs" "${INTERSHEET_REFS}" (at 169.2699 144.78 0)
+      (effects (font (size 1.27 1.27)) (justify right) hide)
+    )
+  )
   (global_label "5V" (shape input) (at 67.31 153.67 0) (fields_autoplaced)
     (effects (font (size 1.27 1.27)) (justify left))
     (property "Intersheetrefs" "${INTERSHEET_REFS}" (at 72.5139 153.67 0)
+      (effects (font (size 1.27 1.27)) (justify left) hide)
+    )
+  )
+  (global_label "CONN_LOCK_MOT2" (shape output) (at 251.46 142.24 0) (fields_autoplaced)
+    (effects (font (size 1.27 1.27)) (justify left))
+    (property "Intersheetrefs" "${INTERSHEET_REFS}" (at 271.4201 142.24 0)
       (effects (font (size 1.27 1.27)) (justify left) hide)
     )
@@
     )
   )
+  (symbol (lib_id "power:GND") (at 238.76 144.78 0) (unit 1)
+    (in_bom yes) (on_board yes) (dnp no)
+    (property "Reference" "#PWR048" (at 238.76 151.13 0)
+      (effects (font (size 1.27 1.27)) hide)
+    )
+    (property "Value" "GND" (at 241.3 148.59 0)
+      (effects (font (size 1.27 1.27)) (justify right))
+    )
+    (property "Footprint" "" (at 238.76 144.78 0)
+      (effects (font (size 1.27 1.27)) hide)
+    )
+    (property "Datasheet" "" (at 238.76 144.78 0)
+      (effects (font (size 1.27 1.27)) hide)
+    )
+    (pin "1")
+    (instances
+      (project "qca7000"
+        (path "/e63e39d7-6ac0-4ffd-8aa3-1841a4541b55"
+          (reference "#PWR048") (unit 1)
+        )
+        (path "/e63e39d7-6ac0-4ffd-8aa3-1841a4541b55/5666e7cf-6b6c-4583-8335-aa3be69ccd45"
+          (reference "#PWR069") (unit 1)
+        )
+        (path "/e63e39d7-6ac0-4ffd-8aa3-1841a4541b55/539ec63d-ac7e-42ea-858e-ff2bf33430ea"
+          (reference "#PWR059") (unit 1)
+        )
+      )
+    )
+  )
   (symbol (lib_id "74xx:74HCT04") (at 67.31 170.18 0) (unit 7)
     (in_bom yes) (on_board yes) (dnp no) (fields_autoplaced)
@@
         )
       )
+    )
+  )
+  (symbol (lib_id "DRV8874QPWPRQ1:DRV8874QPWPRQ1") (at 199.39 127 0) (unit 1)
+    (in_bom yes) (on_board yes) (dnp no) (fields_autoplaced)
+    (property "Reference" "IC1" (at 217.17 120.65 0)
+      (effects (font (size 1.27 1.27)))
+    )
+    (property "Value" "DRV8874QPWPRQ1" (at 217.17 123.19 0)
+      (effects (font (size 1.27 1.27)))
+    )
+    (property "Footprint" "SOP65P640X120-17N" (at 231.14 124.46 0)
+      (effects (font (size 1.27 1.27)) (justify left) hide)
+    )
+    (property "Datasheet" "https://www.ti.com/lit/gpn/drv8874-q1?HQS=ti-null-null-sf-df-pf-sep-wwe&DCM=yes" (at 231.14 127 0)
+      (effects (font (size 1.27 1.27)) (justify left) hide)
+    )
+    (property "Description" "Motor Drives Automotive 38-V, 6-A, H-bridge motor driver with integrated current sensing & current sense feedback" (at 231.14 129.54 0)
+      (effects (font (size 1.27 1.27)) (justify left) hide)
+    )
+    (property "Height" "1.2" (at 231.14 132.08 0)
+      (effects (font (size 1.27 1.27)) (justify left) hide)
+    )
+    (property "Mouser Part Number" "595-DRV8874QPWPRQ1" (at 231.14 134.62 0)
+      (effects (font (size 1.27 1.27)) (justify left) hide)
+    )
+    (property "Mouser Price/Stock" "https://www.mouser.co.uk/ProductDetail/Texas-Instruments/DRV8874QPWPRQ1?qs=mAH9sUMRCttZUT1myh3Itg%3D%3D" (at 231.14 137.16 0)
+      (effects (font (size 1.27 1.27)) (justify left) hide)
+    )
+    (property "Manufacturer_Name" "Texas Instruments" (at 231.14 139.7 0)
+      (effects (font (size 1.27 1.27)) (justify left) hide)
+    )
+    (property "Manufacturer_Part_Number" "DRV8874QPWPRQ1" (at 231.14 142.24 0)
+      (effects (font (size 1.27 1.27)) (justify left) hide)
+    )
+    (pin "1")
+    (pin "10")
+    (pin "11")
+    (pin "12")
+    (pin "13")
+    (pin "14")
+    (pin "15")
+    (pin "16")
+    (pin "17")
+    (pin "2")
+    (pin "3")
+    (pin "4")
+    (pin "5")
+    (pin "6")
+    (pin "7")
+    (pin "8")
+    (pin "9")
+    (instances
+      (project "qca7000"
+        (path "/e63e39d7-6ac0-4ffd-8aa3-1841a4541b55/539ec63d-ac7e-42ea-858e-ff2bf33430ea"
+          (reference "IC1") (unit 1)
+        )
+      )

Commit message: wired the drv8874. Added spare holes. Flash connector larger holes
Parts:
- added C17: 100nF, Capacitor_SMD:C_0805_2012Metric_Pad1.18x1.45mm_HandSolder, symbol Device:C_Small
- added C17: 22nF, Capacitor_SMD:C_0805_2012Metric_Pad1.18x1.45mm_HandSolder, symbol Device:C_Small
- added R3: 3k3, Resistor_SMD:R_1206_3216Metric_Pad1.30x1.75mm_HandSolder, symbol Device:R_Small
- added R3: 220, Resistor_SMD:R_1206_3216Metric_Pad1.30x1.75mm_HandSolder, symbol Device:R_Small
- added R3 (x2): 10k, Resistor_SMD:R_1206_3216Metric_Pad1.30x1.75mm_HandSolder, symbol Device:R_Small
Connections:
- net GND: now also IC1.17 (EP), IC1.7 (IMODE), R3.1, R3.1
- net DRV_IN1: now reaches IC1.1 (EN/IN1)
- net 12V: now reaches IC1.11 (VM)
- net 12V: now also C17.2
- net at IC1.12 (VCP): now also C17.1
- net at IC1.13 (CPH): now also C17.2
- net at IC1.14 (CPL): now also C17.1
- net DRV_IN2: now reaches IC1.2 (PH/IN2)
- net 3V3_uC: now reaches IC1.3 (NSLEEP)
- net 3V3_uC: now also R3.2, R3.2
- net DRV_FAULT: now reaches IC1.4 (NFAULT)
- net DRV_FAULT: now also R3.1
- net at IC1.5 (VREF): now also R3.1, R3.2
- net at IC1.6 (IPROPI): now also R3.2
- no-connect marks 2 -> 3
Other:
- note added: "IMode=GND leads to Fixed Off-time and automatic retry"
- note added: "PMode=open leads to independent control of both half bridges"

Commit message: changed to 4 layers. Added button, PP and lock feedback. New testpoints to avoid courtyard warnings.
Parts:
- IC1: footprint SOP65P640X120-17N -> KiCad:SOP65P640X120-17N
- R3: value 3k3 -> 560
- R3: value 220 -> 1k
- R3: value 10k -> 2k7
Other:
- note added: "IPROPI is 450µA/A. With 6A peak output this is 2.7mA. With R=1k we get 2.7V for the 6A. On VREF, we have 3.3V divided by 560 ohms and 2k7, this results in 2.73V. This means, the current limitation will jump in when the output current is above 6A."
Changed lines of the file:
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@@
     (stroke (width 0) (type default))
   )
-  (text "IMode=GND leads to Fixed Off-time\nand automatic retry"
-    (at 171.45 157.48 0)
+  (text "IMode=GND leads\nto Fixed Off-time\nand automatic retry"
+    (at 195.58 160.02 0)
+    (effects (font (size 1.27 1.27)) (justify left bottom))
+  )
+  (text "IPROPI is 450µA/A.\nWith 6A peak output this is 2.7mA.\nWith R=1k we get 2.7V for the 6A.\n\nOn VREF, we have 3.3V divided by 560 ohms and 2k7,\nthis results in 2.73V.\n\nThis means, the current limitation will\njump in when the output current is above 6A."
+    (at 128.27 167.64 0)
     (effects (font (size 1.27 1.27)) (justify left bottom))
   )
@@
       (effects (font (size 1.27 1.27)))
     )
-    (property "Footprint" "SOP65P640X120-17N" (at 231.14 124.46 0)
+    (property "Footprint" "KiCad:SOP65P640X120-17N" (at 231.14 124.46 0)
       (effects (font (size 1.27 1.27)) (justify left) hide)
     )
@@
       (effects (font (size 1.27 1.27)))
     )
-    (property "Value" "3k3" (at 170.18 124.46 90)
+    (property "Value" "560" (at 170.18 124.46 90)
       (effects (font (size 1.27 1.27)))
     )
@@
       (effects (font (size 1.27 1.27)))
     )
-    (property "Value" "220" (at 157.48 142.24 90)
+    (property "Value" "1k" (at 157.48 142.24 90)
       (effects (font (size 1.27 1.27)))
     )
@@
       (effects (font (size 1.27 1.27)))
     )
-    (property "Value" "10k" (at 172.72 138.43 90)
-      (effects (font (size 1.27 1.27)))
-    )
+    (property "Value" "2k7" (at 172.72 138.43 90)
+      (effects (font (size 1.27 1.27)))
+    )

Commit message: routed driver outputs for contactors and lock motor to PWM TIM3 ports. Use protected 12V for DRV.
Connections:
- net 12V is gone; now on net 12V_P: C17.2, IC1.11 (VM)
Other:
- note added: "The DRV is not specified for inverse polarity. So we need the protected 12V here."
Changed lines of the file:
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@@
+    (effects (font (size 1.27 1.27)) (justify left bottom))
+  )
+  (text "The DRV is not\nspecified for inverse\npolarity. So we need\nthe protected 12V\nhere."
+    (at 261.62 130.81 0)
     (effects (font (size 1.27 1.27)) (justify left bottom))
   )
@@
     )
   )
-  (global_label "12V" (shape input) (at 259.08 128.27 90) (fields_autoplaced)
+  (global_label "12V_P" (shape input) (at 259.08 128.27 90) (fields_autoplaced)
     (effects (font (size 1.27 1.27)) (justify left))
-    (property "Intersheetrefs" "${INTERSHEET_REFS}" (at 259.08 121.8566 90)
+    (property "Intersheetrefs" "${INTERSHEET_REFS}" (at 259.08 119.619 90)
       (effects (font (size 1.27 1.27)) (justify left) hide)
     )
