File: pcb/outputdrivers.kicad_sch (KiCad schematic)
At the start: 32 parts, among them IC1 DRV8874QPWPRQ1, Q1 DTC114E, Q2 NCV8402xST, Q3 NCV8402xST, Q4 DTA143Z, Q7 DTC114E, Q8 DTC114E, Q9 DTC114E, U7 74HCT04

Commit message: fix rx shortcut. add transformer. correct part number of NCV. Correct footprints of U1 and L11. add mounting holes. stepdown layout improved. added TVS at 12V
Parts:
- removed INT (x2): ~, speciallib:TestPoint_Special_THTPad_D1.9mm_Drill1mm, symbol Connector:TestPoint
- Q2, Q3: LCSC C236053 -> C77755; LINK https://jlcpcb.com/partdetail/Onsemi-NCV8402ASTT3G/C236053 -> https://jlcpcb.com/partdetail/C77755
Other:
- note removed: "RF transformer, free-wired, no footprint"
Changed lines of the file:
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@@
-    (stroke (width 0) (type default))
-  )
-  (wire (pts (xy 121.92 24.13) (xy 124.46 24.13))
     (stroke (width 0) (type default))
   )
@@
     (stroke (width 0) (type default))
   )
-  (wire (pts (xy 118.11 21.59) (xy 124.46 21.59))
-    (stroke (width 0) (type default))
-  )
   (wire (pts (xy 54.61 54.61) (xy 58.42 54.61))
     (stroke (width 0) (type default))
@@
   (wire (pts (xy 234.95 144.78) (xy 238.76 144.78))
     (stroke (width 0) (type default))
-  )
-  (text "RF transformer,\nfree-wired,\nno footprint" (at 134.62 24.13 0)
-    (effects (font (size 1.27 1.27)) (justify left bottom))
   )
   (text "IMode=GND leads\nto Fixed Off-time\nand automatic retry"
@@
     (effects (font (size 1.27 1.27)) (justify right))
     (property "Intersheetrefs" "${INTERSHEET_REFS}" (at 47.8942 26.67 0)
-      (effects (font (size 1.27 1.27)) (justify right) hide)
-    )
-  )
-  (global_label "MODEM_RF" (shape input) (at 118.11 21.59 180) (fields_autoplaced)
-    (effects (font (size 1.27 1.27)) (justify right))
-    (property "Intersheetrefs" "${INTERSHEET_REFS}" (at 105.2257 21.59 0)
       (effects (font (size 1.27 1.27)) (justify right) hide)
     )
@@
     )
   )
-  (symbol (lib_id "power:GND") (at 121.92 24.13 0) (unit 1)
-    (in_bom yes) (on_board yes) (dnp no)
-    (property "Reference" "#PWR048" (at 121.92 30.48 0)
-      (effects (font (size 1.27 1.27)) hide)
-    )
-    (property "Value" "GND" (at 124.46 27.94 0)
-      (effects (font (size 1.27 1.27)) (justify right))
-    )
-    (property "Footprint" "" (at 121.92 24.13 0)
-      (effects (font (size 1.27 1.27)) hide)
-    )
-    (property "Datasheet" "" (at 121.92 24.13 0)
-      (effects (font (size 1.27 1.27)) hide)
-    )
-    (pin "1")
-    (instances
-      (project "qca7000"
-        (path "/e63e39d7-6ac0-4ffd-8aa3-1841a4541b55"
-          (reference "#PWR048") (unit 1)
-        )
-        (path "/e63e39d7-6ac0-4ffd-8aa3-1841a4541b55/5666e7cf-6b6c-4583-8335-aa3be69ccd45"
-          (reference "#PWR075") (unit 1)
-        )
-        (path "/e63e39d7-6ac0-4ffd-8aa3-1841a4541b55/539ec63d-ac7e-42ea-858e-ff2bf33430ea"
-          (reference "#PWR074") (unit 1)
-        )
-      )
-    )
-  )
   (symbol (lib_id "74xx:74HCT04") (at 92.71 184.15 0) (unit 1)
     (in_bom yes) (on_board yes) (dnp no) (fields_autoplaced)
@@
     )
   )
-  (symbol (lib_id "Connector:TestPoint") (at 124.46 24.13 270) (unit 1)
-    (in_bom yes) (on_board yes) (dnp no)
-    (property "Reference" "INT" (at 129.54 24.13 90)
-      (effects (font (size 1.27 1.27)) (justify left))
-    )
-    (property "Value" "~" (at 133.35 22.86 90)
-      (effects (font (size 1.27 1.27)) (justify left))
-    )
-    (property "Footprint" "speciallib:TestPoint_Special_THTPad_D1.9mm_Drill1mm" (at 124.46 29.21 0)
-      (effects (font (size 1.27 1.27)) hide)
-    )
-    (property "Datasheet" "~" (at 124.46 29.21 0)
-      (effects (font (size 1.27 1.27)) hide)
-    )
-    (pin "1")
-    (instances
-      (project "qca7000"
-        (path "/e63e39d7-6ac0-4ffd-8aa3-1841a4541b55"
-          (reference "INT") (unit 1)
-        )
-        (path "/e63e39d7-6ac0-4ffd-8aa3-1841a4541b55/539ec63d-ac7e-42ea-858e-ff2bf33430ea"
-          (reference "GND2") (unit 1)
-        )
-      )
-    )
-  )
   (symbol (lib_id "power:GND") (at 238.76 144.78 0) (unit 1)
     (in_bom yes) (on_board yes) (dnp no)
@@
       (effects (font (size 1.27 1.27)) hide)
     )
-    (property "LCSC" "C236053" (at 106.68 91.44 0)
-      (effects (font (size 1.27 1.27)) hide)
-    )
-    (property "LINK" "https://jlcpcb.com/partdetail/Onsemi-NCV8402ASTT3G/C236053" (at 106.68 91.44 0)
+    (property "LCSC" "C77755" (at 106.68 91.44 0)
+      (effects (font (size 1.27 1.27)) hide)
+    )
+    (property "LINK" "https://jlcpcb.com/partdetail/C77755" (at 106.68 91.44 0)
       (effects (font (size 1.27 1.27)) hide)
     )
@@
       (effects (font (size 1.27 1.27)) hide)
     )
-    (property "LCSC" "C236053" (at 105.41 124.46 0)
-      (effects (font (size 1.27 1.27)) hide)
-    )
-    (property "LINK" "https://jlcpcb.com/partdetail/Onsemi-NCV8402ASTT3G/C236053" (at 105.41 124.46 0)
+    (property "LCSC" "C77755" (at 105.41 124.46 0)
+      (effects (font (size 1.27 1.27)) hide)
+    )
+    (property "LINK" "https://jlcpcb.com/partdetail/C77755" (at 105.41 124.46 0)
       (effects (font (size 1.27 1.27)) hide)
     )
@@
         )
       )
-    )
-  )
-  (symbol (lib_id "Connector:TestPoint") (at 124.46 21.59 270) (unit 1)
-    (in_bom yes) (on_board yes) (dnp no)
-    (property "Reference" "INT" (at 129.54 21.59 90)
-      (effects (font (size 1.27 1.27)) (justify left))
-    )
-    (property "Value" "~" (at 133.35 20.32 90)
-      (effects (font (size 1.27 1.27)) (justify left))
-    )
-    (property "Footprint" "speciallib:TestPoint_Special_THTPad_D1.9mm_Drill1mm" (at 124.46 26.67 0)
-      (effects (font (size 1.27 1.27)) hide)
-    )
-    (property "Datasheet" "~" (at 124.46 26.67 0)
-      (effects (font (size 1.27 1.27)) hide)
-    )
-    (pin "1")
-    (instances
-      (project "qca7000"
-        (path "/e63e39d7-6ac0-4ffd-8aa3-1841a4541b55"
-          (reference "INT") (unit 1)
-        )
-        (path "/e63e39d7-6ac0-4ffd-8aa3-1841a4541b55/539ec63d-ac7e-42ea-858e-ff2bf33430ea"
-          (reference "RF1") (unit 1)
-        )
-      )

Commit message: WIP: PP pull-up and divider. variant detection. ipropi connected to ADC.
Parts:
- added C61: 100nF, Capacitor_SMD:C_0805_2012Metric_Pad1.18x1.45mm_HandSolder, symbol Device:C_Small
- added R3: 47k, Resistor_SMD:R_0805_2012Metric_Pad1.20x1.40mm_HandSolder, symbol Device:R_Small
Connections:
- net GND: now also C61.1
- net at IC1.6 (IPROPI), R3.2: now also R3.2
- new net ADC_IPROPI: C61.2, R3.1
Changed lines of the file:
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@@
   (junction (at 259.08 135.89) (diameter 0) (color 0 0 0 0)
   )
+  (junction (at 140.97 139.7) (diameter 0) (color 0 0 0 0)
+  )
   (junction (at 250.19 53.34) (diameter 0) (color 0 0 0 0)
+  )
+  (junction (at 160.02 139.7) (diameter 0) (color 0 0 0 0)
   )
   (junction (at 160.02 134.62) (diameter 0) (color 0 0 0 0)
@@
     (stroke (width 0) (type default))
   )
+  (wire (pts (xy 135.89 139.7) (xy 140.97 139.7))
+    (stroke (width 0) (type default))
+  )
+  (wire (pts (xy 140.97 139.7) (xy 140.97 140.97))
+    (stroke (width 0) (type default))
+  )
   (wire (pts (xy 48.26 91.44) (xy 48.26 99.06))
     (stroke (width 0) (type default))
@@
     (stroke (width 0) (type default))
   )
+  (wire (pts (xy 140.97 139.7) (xy 147.32 139.7))
+    (stroke (width 0) (type default))
+  )
   (wire (pts (xy 44.45 91.44) (xy 48.26 91.44))
     (stroke (width 0) (type default))
@@
   )
   (wire (pts (xy 261.62 58.42) (xy 261.62 82.55))
+    (stroke (width 0) (type default))
+  )
+  (wire (pts (xy 152.4 139.7) (xy 160.02 139.7))
     (stroke (width 0) (type default))
   )
@@
   )
   (text "IPROPI is 450µA/A.\nWith 6A peak output this is 2.7mA.\nWith R=1k we get 2.7V for the 6A.\n\nOn VREF, we have 3.3V divided by 560 ohms and 2k7,\nthis results in 2.73V.\n\nThis means, the current limitation will\njump in when the output current is above 6A."
-    (at 128.27 167.64 0)
+    (at 127 171.45 0)
     (effects (font (size 1.27 1.27)) (justify left bottom))
   )
@@
     (property "Intersheetrefs" "${INTERSHEET_REFS}" (at 92.35 30.48 0)
       (effects (font (size 1.27 1.27)) (justify left) hide)
+    )
+  )
+  (global_label "ADC_IPROPI" (shape output) (at 135.89 139.7 180) (fields_autoplaced)
+    (effects (font (size 1.27 1.27)) (justify right))
+    (property "Intersheetrefs" "${INTERSHEET_REFS}" (at 122.0379 139.7 0)
+      (effects (font (size 1.27 1.27)) (justify right) hide)
     )
   )
@@
     )
   )
+  (symbol (lib_id "power:GND") (at 140.97 146.05 0) (unit 1)
+    (in_bom yes) (on_board yes) (dnp no)
+    (property "Reference" "#PWR048" (at 140.97 152.4 0)
+      (effects (font (size 1.27 1.27)) hide)
+    )
+    (property "Value" "GND" (at 143.51 149.86 0)
+      (effects (font (size 1.27 1.27)) (justify right))
+    )
+    (property "Footprint" "" (at 140.97 146.05 0)
+      (effects (font (size 1.27 1.27)) hide)
+    )
+    (property "Datasheet" "" (at 140.97 146.05 0)
+      (effects (font (size 1.27 1.27)) hide)
+    )
+    (pin "1")
+    (instances
+      (project "qca7000"
+        (path "/e63e39d7-6ac0-4ffd-8aa3-1841a4541b55"
+          (reference "#PWR048") (unit 1)
+        )
+        (path "/e63e39d7-6ac0-4ffd-8aa3-1841a4541b55/5666e7cf-6b6c-4583-8335-aa3be69ccd45"
+          (reference "#PWR069") (unit 1)
+        )
+        (path "/e63e39d7-6ac0-4ffd-8aa3-1841a4541b55/539ec63d-ac7e-42ea-858e-ff2bf33430ea"
+          (reference "#PWR0102") (unit 1)
+        )
+      )
+    )
+  )
   (symbol (lib_id "power:GND") (at 85.09 185.42 0) (unit 1)
     (in_bom yes) (on_board yes) (dnp no)
@@
         (path "/e63e39d7-6ac0-4ffd-8aa3-1841a4541b55/539ec63d-ac7e-42ea-858e-ff2bf33430ea"
           (reference "Q7") (unit 1)
+        )
+      )
+    )
+  )
+  (symbol (lib_id "Device:R_Small") (at 149.86 139.7 90) (unit 1)
+    (in_bom yes) (on_board yes) (dnp no)
+    (property "Reference" "R3" (at 152.4 143.51 0)
+      (effects (font (size 1.27 1.27)))
+    )
+    (property "Value" "47k" (at 149.86 143.51 0)
+      (effects (font (size 1.27 1.27)))
+    )
+    (property "Footprint" "Resistor_SMD:R_0805_2012Metric_Pad1.20x1.40mm_HandSolder" (at 149.86 139.7 0)
+      (effects (font (size 1.27 1.27)) hide)
+    )
+    (property "Datasheet" "https://datasheet.lcsc.com/lcsc/1811101920_UNI-ROYAL-Uniroyal-Elec-0603WAF3301T5E_C22978.pdf" (at 149.86 139.7 0)
+      (effects (font (size 1.27 1.27)) hide)
+    )
+    (property "LCSC" "C17713" (at 149.86 139.7 90)
+      (effects (font (size 1.27 1.27)) hide)
+    )
+    (property "LINK" "https://jlcpcb.com/partdetail/18401-0805W8F4702T5E/C17713" (at 149.86 139.7 0)
+      (effects (font (size 1.27 1.27)) hide)
+    )
+    (pin "1")
+    (pin "2")
+    (instances
+      (project "qca7000"
+        (path "/e63e39d7-6ac0-4ffd-8aa3-1841a4541b55"
+          (reference "R3") (unit 1)
+        )
+        (path "/e63e39d7-6ac0-4ffd-8aa3-1841a4541b55/5666e7cf-6b6c-4583-8335-aa3be69ccd45"
+          (reference "R21") (unit 1)
+        )
+        (path "/e63e39d7-6ac0-4ffd-8aa3-1841a4541b55/93c6207c-4203-4bc7-a590-e5e89c0d3d27"
+          (reference "R61") (unit 1)
+        )
+        (path "/e63e39d7-6ac0-4ffd-8aa3-1841a4541b55/539ec63d-ac7e-42ea-858e-ff2bf33430ea"
+          (reference "R63") (unit 1)
         )
       )
@@
         )
       )
+    )
+  )
+  (symbol (lib_name "C_Small_13") (lib_id "Device:C_Small") (at 140.97 143.51 180) (unit 1)
+    (in_bom yes) (on_board yes) (dnp no)
+    (property "Reference" "C61" (at 144.78 143.51 0)
+      (effects (font (size 1.27 1.27)))
+    )
+    (property "Value" "100nF" (at 146.05 146.05 0)
+      (effects (font (size 1.27 1.27)))
+    )
+    (property "Footprint" "Capacitor_SMD:C_0805_2012Metric_Pad1.18x1.45mm_HandSolder" (at 140.97 143.51 0)
+      (effects (font (size 1.27 1.27)) hide)
+    )
+    (property "Datasheet" "~" (at 140.97 143.51 0)
+      (effects (font (size 1.27 1.27)) hide)
+    )
+    (property "LCSC" "C49678" (at 140.97 143.51 90)
+      (effects (font (size 1.27 1.27)) hide)
+    )
+    (property "LINK" "https://jlcpcb.com/partdetail/Yageo-CC0805KRX7R9BB104/C49678" (at 140.97 143.51 0)
+      (effects (font (size 1.27 1.27)) hide)
+    )
+    (pin "1")
+    (pin "2")
+    (instances
+      (project "qca7000"
+        (path "/e63e39d7-6ac0-4ffd-8aa3-1841a4541b55"
+          (reference "C61") (unit 1)
+        )
+        (path "/e63e39d7-6ac0-4ffd-8aa3-1841a4541b55/5666e7cf-6b6c-4583-8335-aa3be69ccd45"
+          (reference "C68") (unit 1)
+        )
+        (path "/e63e39d7-6ac0-4ffd-8aa3-1841a4541b55/93c6207c-4203-4bc7-a590-e5e89c0d3d27"
+          (reference "C80") (unit 1)
+        )
+        (path "/e63e39d7-6ac0-4ffd-8aa3-1841a4541b55/539ec63d-ac7e-42ea-858e-ff2bf33430ea"
+          (reference "C39") (unit 1)
+        )
+      )

Commit message: feature: Added wakeup logic
Parts:
- removed Q1, Q7: DTC114E, Package_TO_SOT_SMD:SOT-23, symbol Transistor_BJT:DTC114E
- removed Q8, Q9: DTC114E, Package_TO_SOT_SMD:SOT-23, symbol Transistor_BJT:DTC113Z
- added C54, C69, C70: 22uF, Capacitor_SMD:C_1210_3225Metric_Pad1.33x2.70mm_HandSolder, symbol Device:C_Small
- added Q1, Q12, Q13, Q7, Q8: 2N7002, Package_TO_SOT_SMD:SOT-23, symbol Transistor_FET:2N7002
- added Q11: AO3401A, Package_TO_SOT_SMD:SOT-23, symbol Transistor_FET:AO3401A
- added R69: 10k, Resistor_SMD:R_0805_2012Metric_Pad1.20x1.40mm_HandSolder, symbol Device:R_Small
- renumbered C17 to C15, C17 to C18, C61 to C25, C61 to C39, C17 to C76, D10 to D14, D10 to D16, Q4 to Q5, Q4 to Q6, R3 to R25, R3 to R26, R3 to R27, R11 to R29, R11 to R30, R3 to R45, R3 to R46, R3 to R47, R3 to R48, R3 to R49, R3 to R50, R3 to R51, R3 to R58, R3 to R63
Connections:
- net 12V_P: now also C54.2, C69.2, C70.2, Q11.2 (S), R69.2
- net GND: now also C54.1, C69.1, C70.1, Q1.2 (S), Q12.2 (S), Q13.2 (S), Q7.2 (S), Q8.2 (S)
- net LED_CTL_BLUE: now also Q8.1 (G)
- net LED_CTL_GREEN: now also Q7.1 (G)
- net LED_CTL_RED: now also Q12.1 (G)
- net STATE_C_CONTROL: now also Q1.1 (G)
- net at Q4.1 (B): now also Q12.3 (D)
- net at R27.1: now also Q1.3 (D)
- net at Q5.1 (B): now also Q7.3 (D)
- net at Q6.1 (B): now also Q8.3 (D)
- new net: Q11.1 (G), Q13.3 (D), R69.1
- new net TRIGGER_WAKEUP: Q13.1 (G)
- new net WAKEUP: Q11.3 (D)
Other:
- note added: "The bulk capacitor is especially important when switching high currents, see DRV8874 data sheet."

Commit message: Moved most vias away from pads
Parts:
- Q11: LCSC (none) -> C15127
Changed lines of the file:
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@@
       (effects (font (size 1.27 1.27)) (justify left) hide)
+    )
+    (property "LCSC" "C15127" (at 201.93 44.45 0)
+      (effects (font (size 1.27 1.27)) hide)
     )
     (pin "1")

Commit message: Made relay drivers PMOS with gate drivers and free wheeling diode
Parts:
- removed Q2, Q3: NCV8402xST, Package_TO_SOT_SMD:SOT-223, symbol Driver_FET:NCV8402xST
- removed U7: 74HCT04, Package_SO:SO-14_3.9x8.65mm_P1.27mm, symbol 74xx:74HCT04
- added D17, D18: SS54B-HF, Diode_SMD:D_SMB_Handsoldering, symbol Device:D_Schottky
- added Q2, Q3: AO3401A, Package_TO_SOT_SMD:SOT-23, symbol Transistor_FET:AO3401A
- added U11, U7: UCC27517DBVR, Package_TO_SOT_SMD:SOT-23-5, symbol Driver_FET:FAN3111C
Connections:
- net 12V_P: now also Q2.2 (S), Q3.2 (S), U11.1 (VDD), U11.3 (IN+), U7.1 (VDD), U7.3 (IN+)
- net CONTACTOR1_LS: now also D18.1 (K), Q2.3 (D)
- net CONTACTOR2_LS: now also D17.1 (K), Q3.3 (D)
- net CONTACTOR_CONTROL1: now also U7.4 (~{IN-})
- net CONTACTOR_CONTROL2: now also U11.4 (~{IN-})
- net GND: now also D17.2 (A), D18.2 (A), U11.2 (GND), U7.2 (GND)
- new net: Q3.1 (G), U11.5 (OUT)
- new net: Q2.1 (G), U7.5 (OUT)
- no-connect marks 3 -> 1
Other:
- note added: "We use the driver in inverting configuration because when the output is high the PMOS is OFF"
- note removed: "HCT as level shifter from 3.3V to 5V, because the NCV needs at least 5V gate voltage. Non-inverting is important, so that a fail of the 3V3 will lead to "contactors off"."

Commit message: Using another motor driver IC for contactor control
Parts:
- removed D17, D18: SS54B-HF, Diode_SMD:D_SMB_Handsoldering, symbol Device:D_Schottky
- removed Q2, Q3: AO3401A, Package_TO_SOT_SMD:SOT-23, symbol Transistor_FET:AO3401A
- removed U11, U7: UCC27517DBVR, Package_TO_SOT_SMD:SOT-23-5, symbol Driver_FET:FAN3111C
- added C72: 22nF, Capacitor_SMD:C_0805_2012Metric_Pad1.18x1.45mm_HandSolder, symbol Device:C_Small
- added C75, C81: 100nF, Capacitor_SMD:C_0805_2012Metric_Pad1.18x1.45mm_HandSolder, symbol Device:C_Small
- added IC2: DRV8874QPWPRQ1, KiCad:SOP65P640X120-17N, symbol DRV8874QPWPRQ1:DRV8874QPWPRQ1
- R29: value 10k -> 560; LCSC C17414 -> C28636; LINK https://jlcpcb.com/partdetail/18102-0805W8F1002T5E/C17414 -> https://jlcpcb.com/partdetail/29388-0805W8F5600T5E/C28636
- R30: value 10k -> 2k7; LCSC C17414 -> C17530; LINK https://jlcpcb.com/partdetail/18102-0805W8F1002T5E/C17414 -> https://jlcpcb.com/partdetail/18218-0805W8F2701T5E/C17530
Connections:
- net 12V_P: now also C75.2, C81.1, IC2.11 (VM)
- net 3V3_uC: now also R29.2
- net CONTACTOR1_LS: now also IC2.8 (OUT1)
- net CONTACTOR2_LS: now also IC2.10 (OUT2)
- net CONTACTOR_CONTROL1: now also IC2.1 (EN/IN1); no longer R29.1
- net CONTACTOR_CONTROL2: now also IC2.2 (PH/IN2); no longer R30.2
- net DRV_FAULT: now also IC2.4 (NFAULT)
- net GND: now also R30.2, C81.2, IC2.15 (GND), IC2.17 (EP), IC2.7 (IMODE), IC2.9 (PGND); no longer R29.2, R30.1
- new net: IC2.5 (VREF), R29.1, R30.1
- new net: C75.1, IC2.12 (VCP)
- new net: C72.2, IC2.13 (CPH)
- new net: C72.1, IC2.14 (CPL)
- new net CONTACTOR_ENABLE: IC2.3 (NSLEEP)
Other:
- note added: "We reuse DRV_FAULT from the lock driver. Since software should know which device it last acted it will also know which one caused the fault"
- note removed: "4A typical at U_GS=5V and 25°C. Clamping to 42V without external circuit."
- note removed: "We use the driver in inverting configuration because when the output is high the PMOS is OFF"
- note removed: "pull down, to make sure that if the controller is in reset, the contactors are off."

Commit message: Redesigned wakeup circuit
Changed lines of the file:
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@@
     (stroke (width 0) (type default))
   )
-  (wire (pts (xy 185.42 54.61) (xy 185.42 55.88))
+  (wire (pts (xy 185.42 54.61) (xy 185.42 66.04))
     (stroke (width 0) (type default))
   )
@@
     (stroke (width 0) (type default))
   )
+  (wire (pts (xy 67.31 39.37) (xy 73.66 39.37))
+    (stroke (width 0) (type default))
+  )
   (wire (pts (xy 234.95 142.24) (xy 251.46 142.24))
     (stroke (width 0) (type default))
@@
   )
   (wire (pts (xy 74.93 109.22) (xy 74.93 106.68))
-    (stroke (width 0) (type default))
-  )
-  (wire (pts (xy 67.31 39.37) (xy 73.66 39.37))
     (stroke (width 0) (type default))
   )
@@
   (symbol (lib_id "Device:R_Small") (at 67.31 41.91 180) (unit 1)
     (in_bom yes) (on_board yes) (dnp no)
-    (property "Reference" "R27" (at 71.12 41.91 0)
-      (effects (font (size 1.27 1.27)))
-    )
-    (property "Value" "1k2" (at 71.12 44.45 0)
+    (property "Reference" "R27" (at 63.5 40.64 0)
+      (effects (font (size 1.27 1.27)))
+    )
+    (property "Value" "1k2" (at 63.5 43.18 0)
       (effects (font (size 1.27 1.27)))
     )
@@
     (in_bom yes) (on_board yes) (dnp no) (fields_autoplaced)
     (property "Reference" "Q1" (at 69.977 53.3979 0)
-      (effects (font (size 1.27 1.27)) (justify left))
+      (effects (font (size 1.27 1.27)) (justify left) hide)
     )
     (property "Value" "2N7002" (at 69.977 55.8221 0)
-      (effects (font (size 1.27 1.27)) (justify left))
+      (effects (font (size 1.27 1.27)) (justify left) hide)
     )
     (property "Footprint" "Package_TO_SOT_SMD:SOT-23" (at 69.85 56.515 0)
@@
     )
   )
-  (symbol (lib_id "power:GND") (at 185.42 55.88 0) (unit 1)
-    (in_bom yes) (on_board yes) (dnp no)
-    (property "Reference" "#PWR0103" (at 185.42 62.23 0)
-      (effects (font (size 1.27 1.27)) hide)
-    )
-    (property "Value" "GND" (at 187.96 59.69 0)
+  (symbol (lib_id "power:GND") (at 185.42 66.04 0) (unit 1)
+    (in_bom yes) (on_board yes) (dnp no)
+    (property "Reference" "#PWR0103" (at 185.42 72.39 0)
+      (effects (font (size 1.27 1.27)) hide)
+    )
+    (property "Value" "GND" (at 187.96 69.85 0)
       (effects (font (size 1.27 1.27)) (justify right))
     )
-    (property "Footprint" "" (at 185.42 55.88 0)
-      (effects (font (size 1.27 1.27)) hide)
-    )
-    (property "Datasheet" "" (at 185.42 55.88 0)
-      (effects (font (size 1.27 1.27)) hide)
-    )
+    (property "Footprint" "" (at 185.42 66.04 0)
+      (effects (font (size 1.27 1.27)) hide)
+    )
+    (property "Datasheet" "" (at 185.42 66.04 0)
+      (effects (font (size 1.27 1.27)) hide)
+    )
