File: pcb/powersupply.kicad_sch (KiCad schematic)
At the start: 23 parts, among them J3 12V_in, U3 AMS1117-3.3, U4 AMS1117-3.3, U5 TPS54302

Commit message: added sheets for inputs and outputs. layout draft.
Parts:
- removed C61: 100nF, Capacitor_SMD:C_1206_3216Metric_Pad1.33x1.80mm_HandSolder, symbol Device:C_Small
- C60, C64, C65: footprint Capacitor_SMD:C_1206_3216Metric_Pad1.33x1.80mm_HandSolder -> Capacitor_SMD:C_0805_2012Metric_Pad1.18x1.45mm_HandSolder
- JP1: footprint (none) -> Jumper:SolderJumper-2_P1.3mm_Open_TrianglePad1.0x1.5mm

Commit message: fix: divider on the stepdown. fix: non-inverted contactor drivers. fix: part number of 8MHz. add: mounting holes and spare grid. add: LIM HVDC input. docu: todo list
Parts:
- added R12: 22k, Resistor_SMD:R_1206_3216Metric_Pad1.30x1.75mm_HandSolder, symbol Device:R_Small
- R11: value 10k -> 100k
- R12: value 10k -> 33k
Connections:
- net GND: now also R12.1
- net at C69.1, R11.2, R12.2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: now also R12.2
Other:
- note added: "The combination 100k and 13.3k is recommended by the data sheet for 5V output. We use 22k || 33k, this makes 13.2k."
Changed lines of the file:
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@@
+    (stroke (width 0) (type default))
+  )
+  (wire (pts (xy 125.73 60.96) (xy 125.73 63.5))
     (stroke (width 0) (type default))
   )
@@
   (wire (pts (xy 95.25 83.82) (xy 95.25 86.36))
     (stroke (width 0) (type default))
+  )
+  (text "The combination 100k and 13.3k is\nrecommended by the data sheet for\n5V output. We use 22k || 33k, this\nmakes 13.2k."
+    (at 135.89 67.31 0)
+    (effects (font (size 1.27 1.27)) (justify left bottom))
   )
   (text "Todo: TVS" (at 35.56 57.15 0)
@@
   (symbol (lib_id "Device:R_Small") (at 129.54 50.8 0) (unit 1)
     (in_bom yes) (on_board yes) (dnp no)
-    (property "Reference" "R11" (at 132.08 48.26 0)
-      (effects (font (size 1.27 1.27)))
-    )
-    (property "Value" "10k" (at 132.08 52.07 0)
+    (property "Reference" "R11" (at 130.81 43.18 0)
+      (effects (font (size 1.27 1.27)))
+    )
+    (property "Value" "100k" (at 130.81 45.72 0)
       (effects (font (size 1.27 1.27)))
     )
@@
     )
   )
+  (symbol (lib_id "power:GND") (at 125.73 63.5 0) (unit 1)
+    (in_bom yes) (on_board yes) (dnp no)
+    (property "Reference" "#PWR056" (at 125.73 69.85 0)
+      (effects (font (size 1.27 1.27)) hide)
+    )
+    (property "Value" "GND" (at 128.27 67.31 0)
+      (effects (font (size 1.27 1.27)) (justify right))
+    )
+    (property "Footprint" "" (at 125.73 63.5 0)
+      (effects (font (size 1.27 1.27)) hide)
+    )
+    (property "Datasheet" "" (at 125.73 63.5 0)
+      (effects (font (size 1.27 1.27)) hide)
+    )
+    (pin "1")
+    (instances
+      (project "qca7000"
+        (path "/e63e39d7-6ac0-4ffd-8aa3-1841a4541b55"
+          (reference "#PWR056") (unit 1)
+        )
+        (path "/e63e39d7-6ac0-4ffd-8aa3-1841a4541b55/81db238c-e53f-4d52-98ea-36a1df697651"
+          (reference "#PWR054") (unit 1)
+        )
+      )
+    )
+  )
   (symbol (lib_name "C_Small_13") (lib_id "Device:C_Small") (at 77.47 106.68 180) (unit 1)
     (in_bom yes) (on_board yes) (dnp no)
@@
     )
   )
+  (symbol (lib_id "Device:R_Small") (at 125.73 58.42 180) (unit 1)
+    (in_bom yes) (on_board yes) (dnp no)
+    (property "Reference" "R12" (at 123.19 60.96 0)
+      (effects (font (size 1.27 1.27)))
+    )
+    (property "Value" "22k" (at 123.19 63.5 0)
+      (effects (font (size 1.27 1.27)))
+    )
+    (property "Footprint" "Resistor_SMD:R_1206_3216Metric_Pad1.30x1.75mm_HandSolder" (at 125.73 58.42 0)
+      (effects (font (size 1.27 1.27)) hide)
+    )
+    (property "Datasheet" "~" (at 125.73 58.42 0)
+      (effects (font (size 1.27 1.27)) hide)
+    )
+    (property "LCSC" "C25804" (at 125.73 58.42 0)
+      (effects (font (size 1.27 1.27)) hide)
+    )
+    (pin "1")
+    (pin "2")
+    (instances
+      (project "qca7000"
+        (path "/e63e39d7-6ac0-4ffd-8aa3-1841a4541b55"
+          (reference "R12") (unit 1)
+        )
+        (path "/e63e39d7-6ac0-4ffd-8aa3-1841a4541b55/81db238c-e53f-4d52-98ea-36a1df697651"
+          (reference "R38") (unit 1)
+        )
+      )
+    )
+  )
   (symbol (lib_id "Device:C_Polarized") (at 85.09 107.95 0) (unit 1)
     (in_bom yes) (on_board yes) (dnp no)
@@
   (symbol (lib_id "Device:R_Small") (at 129.54 58.42 180) (unit 1)
     (in_bom yes) (on_board yes) (dnp no)
-    (property "Reference" "R12" (at 132.08 57.15 0)
-      (effects (font (size 1.27 1.27)))
-    )
-    (property "Value" "10k" (at 132.08 59.69 0)
-      (effects (font (size 1.27 1.27)))
-    )
+    (property "Reference" "R12" (at 132.08 59.69 0)
+      (effects (font (size 1.27 1.27)))
+    )
+    (property "Value" "33k" (at 132.08 62.23 0)
+      (effects (font (size 1.27 1.27)))
+    )

Commit message: added TE DEUTSCH connector and housing
Parts:
- removed C60: 100nF, Capacitor_SMD:C_0805_2012Metric_Pad1.18x1.45mm_HandSolder, symbol Device:C_Small
- removed C62: 100uF, Capacitor_SMD:CP_Elec_8x10, symbol Device:C_Polarized
- removed J3: 12V_in, Connector_PinHeader_2.54mm:PinHeader_1x02_P2.54mm_Vertical, symbol Connector:Conn_01x02_Pin
- removed JP1: SolderJumper3V3together, Jumper:SolderJumper-2_P1.3mm_Open_TrianglePad1.0x1.5mm, symbol Jumper:SolderJumper_2_Open
- removed U3: AMS1117-3.3, Package_TO_SOT_SMD:SOT-223-3_TabPin2, symbol Regulator_Linear:AMS1117-3.3
- added R12: 0, Resistor_SMD:R_1206_3216Metric_Pad1.30x1.75mm_HandSolder, symbol Device:R_Small
Connections:
- net 3V3_D: now also R12.2
- net 3V3_uC: now also R12.1
Other:
- note removed: "Option to populate only one linear regulator and connect 3V3_D and 3V3_uC together."
- note removed: "Two separate linear regulators 5V to 3V3, to decouple the noise controller supply from the sensitive QCA supply"

Commit message: added RGB LED highside drivers
Parts:
- C67, C70, C71: footprint Capacitor_SMD:C_1206_3216Metric_Pad1.33x1.80mm_HandSolder -> Capacitor_SMD:C_1210_3225Metric_Pad1.33x2.70mm_HandSolder
Changed lines of the file:
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@@
       (effects (font (size 1.27 1.27)))
     )
-    (property "Footprint" "Capacitor_SMD:C_1206_3216Metric_Pad1.33x1.80mm_HandSolder" (at 78.74 49.53 0)
+    (property "Footprint" "Capacitor_SMD:C_1210_3225Metric_Pad1.33x2.70mm_HandSolder" (at 78.74 49.53 0)
       (effects (font (size 1.27 1.27)) hide)
     )
@@
       (effects (font (size 1.27 1.27)))
     )
-    (property "Footprint" "Capacitor_SMD:C_1206_3216Metric_Pad1.33x1.80mm_HandSolder" (at 135.89 49.53 0)
+    (property "Footprint" "Capacitor_SMD:C_1210_3225Metric_Pad1.33x2.70mm_HandSolder" (at 135.89 49.53 0)
       (effects (font (size 1.27 1.27)) hide)
     )
@@
       (effects (font (size 1.27 1.27)))
     )
-    (property "Footprint" "Capacitor_SMD:C_1206_3216Metric_Pad1.33x1.80mm_HandSolder" (at 144.78 49.53 0)
-      (effects (font (size 1.27 1.27)) hide)
-    )
+    (property "Footprint" "Capacitor_SMD:C_1210_3225Metric_Pad1.33x2.70mm_HandSolder" (at 144.78 49.53 0)
+      (effects (font (size 1.27 1.27)) hide)
+    )

Commit message: wired the drv8874. Added spare holes. Flash connector larger holes
Changed lines of the file:
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@@
   (junction (at 142.24 44.45) (diameter 0) (color 0 0 0 0)
+  )
+  (junction (at 95.25 83.82) (diameter 0) (color 0 0 0 0)
   )
   (junction (at 77.47 104.14) (diameter 0) (color 0 0 0 0)
@@
         )
       )
+    )
+  )
+  (symbol (lib_id "power:PWR_FLAG") (at 95.25 83.82 0) (unit 1)
+    (in_bom yes) (on_board yes) (dnp no)
+    (property "Reference" "#FLG02" (at 95.25 81.915 0)
+      (effects (font (size 1.27 1.27)) hide)
+    )
+    (property "Value" "PWR_FLAG" (at 87.63 80.01 0)
+      (effects (font (size 1.27 1.27)) (justify left))
+    )
+    (property "Footprint" "" (at 95.25 83.82 0)
+      (effects (font (size 1.27 1.27)) hide)
+    )
+    (property "Datasheet" "~" (at 95.25 83.82 0)
+      (effects (font (size 1.27 1.27)) hide)
+    )
+    (pin "1")
+    (instances
+      (project "qca7000"
+        (path "/e63e39d7-6ac0-4ffd-8aa3-1841a4541b55"
+          (reference "#FLG02") (unit 1)
+        )
+        (path "/e63e39d7-6ac0-4ffd-8aa3-1841a4541b55/81db238c-e53f-4d52-98ea-36a1df697651"
+          (reference "#FLG010") (unit 1)
+        )
+      )

Commit message: routed driver outputs for contactors and lock motor to PWM TIM3 ports. Use protected 12V for DRV.
Other:
- note added: "SS54B is rated for 5A. This is at the border, if we drive 6A in the lock/unlock motor."
- note added: "The bulk capacitor is especially important when switching high currents, see DRV8874 data sheet."
Changed lines of the file:
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@@
+    (effects (font (size 1.27 1.27)) (justify left bottom))
+  )
+  (text "The bulk capacitor is especially\nimportant when switching high\ncurrents, see DRV8874 data\nsheet."
+    (at 40.64 71.12 0)
     (effects (font (size 1.27 1.27)) (justify left bottom))
   )
@@
     (effects (font (size 1.27 1.27)) (justify left bottom))
   )
+  (text "SS54B is rated for 5A.\nThis is at the border,\nif we drive 6A in the\nlock/unlock motor."
+    (at 29.21 40.64 0)
+    (effects (font (size 1.27 1.27)) (justify left bottom))
+  )

Commit message: all 100nF now 0805. Todo list cleaned up.
Parts:
- C68: footprint Capacitor_SMD:C_1206_3216Metric_Pad1.33x1.80mm_HandSolder -> Capacitor_SMD:C_0805_2012Metric_Pad1.18x1.45mm_HandSolder
Changed lines of the file:
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@@
       (effects (font (size 1.27 1.27)))
     )
-    (property "Footprint" "Capacitor_SMD:C_1206_3216Metric_Pad1.33x1.80mm_HandSolder" (at 114.3 46.99 0)
+    (property "Footprint" "Capacitor_SMD:C_0805_2012Metric_Pad1.18x1.45mm_HandSolder" (at 114.3 46.99 0)
       (effects (font (size 1.27 1.27)) hide)
     )
