File: pcb/powersupply.kicad_sch (KiCad schematic)
At the start: 19 parts, among them U4 AMS1117-3.3, U5 TPS54302

Commit message: added some jlcpcb part numbers, adjusted some footprints and values accordingly.
Parts:
- C64, C65, C68: LCSC C14663 -> C49678; LINK (none) -> https://jlcpcb.com/partdetail/Yageo-CC0805KRX7R9BB104/C49678
- C67: value 10uF -> 10uF 25V; footprint Capacitor_SMD:C_1210_3225Metric_Pad1.33x2.70mm_HandSolder -> Capacitor_SMD:C_0805_2012Metric_Pad1.18x1.45mm_HandSolder; LCSC C14663 -> C15850; LINK (none) -> https://jlcpcb.com/partdetail/16532-CL21A106KAYNNNE/C15850
- C69: value 68pF -> 47pF; footprint Capacitor_SMD:C_1206_3216Metric_Pad1.33x1.80mm_HandSolder -> Capacitor_SMD:C_0805_2012Metric_Pad1.18x1.45mm_HandSolder; LCSC C14663 -> C14857; LINK (none) -> https://jlcpcb.com/partdetail/15529-CL21C470JBANNNC/C14857
- C70, C71: LCSC C14663 -> C12891; LINK (none) -> https://jlcpcb.com/partdetail/13537-CL31A226KAHNNNE/C12891
- L13: LCSC C162588 -> (none)
- R12: LCSC C25804 -> C17888; LINK (none) -> https://jlcpcb.com/partdetail/18576-1206W4F0000T5E/C17888
Changed lines of the file:
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@@
       (effects (font (size 1.27 1.27)))
     )
-    (property "Value" "10uF" (at 82.55 52.07 0)
-      (effects (font (size 1.27 1.27)))
-    )
-    (property "Footprint" "Capacitor_SMD:C_1210_3225Metric_Pad1.33x2.70mm_HandSolder" (at 78.74 49.53 0)
+    (property "Value" "10uF 25V" (at 82.55 52.07 0)
+      (effects (font (size 1.27 1.27)))
+    )
+    (property "Footprint" "Capacitor_SMD:C_0805_2012Metric_Pad1.18x1.45mm_HandSolder" (at 78.74 49.53 0)
       (effects (font (size 1.27 1.27)) hide)
     )
@@
       (effects (font (size 1.27 1.27)) hide)
     )
-    (property "LCSC" "C14663" (at 78.74 49.53 90)
+    (property "LCSC" "C15850" (at 78.74 49.53 90)
+      (effects (font (size 1.27 1.27)) hide)
+    )
+    (property "LINK" "https://jlcpcb.com/partdetail/16532-CL21A106KAYNNNE/C15850" (at 78.74 49.53 0)
       (effects (font (size 1.27 1.27)) hide)
     )
@@
       (effects (font (size 1.27 1.27)) hide)
     )
-    (property "LCSC" "C162588" (at 121.92 46.99 90)
+    (property "LCSC" "" (at 121.92 46.99 90)
       (effects (font (size 1.27 1.27)) hide)
     )
@@
       (effects (font (size 1.27 1.27)))
     )
-    (property "Value" "68pF" (at 121.92 54.61 0)
-      (effects (font (size 1.27 1.27)))
-    )
-    (property "Footprint" "Capacitor_SMD:C_1206_3216Metric_Pad1.33x1.80mm_HandSolder" (at 125.73 52.07 0)
+    (property "Value" "47pF" (at 121.92 54.61 0)
+      (effects (font (size 1.27 1.27)))
+    )
+    (property "Footprint" "Capacitor_SMD:C_0805_2012Metric_Pad1.18x1.45mm_HandSolder" (at 125.73 52.07 0)
       (effects (font (size 1.27 1.27)) hide)
     )
@@
       (effects (font (size 1.27 1.27)) hide)
     )
-    (property "LCSC" "C14663" (at 125.73 52.07 90)
+    (property "LCSC" "C14857" (at 125.73 52.07 90)
+      (effects (font (size 1.27 1.27)) hide)
+    )
+    (property "LINK" "https://jlcpcb.com/partdetail/15529-CL21C470JBANNNC/C14857" (at 125.73 52.07 0)
       (effects (font (size 1.27 1.27)) hide)
     )
@@
       (effects (font (size 1.27 1.27)) hide)
     )
-    (property "LCSC" "C14663" (at 135.89 49.53 90)
+    (property "LCSC" "C12891" (at 135.89 49.53 90)
+      (effects (font (size 1.27 1.27)) hide)
+    )
+    (property "LINK" "https://jlcpcb.com/partdetail/13537-CL31A226KAHNNNE/C12891" (at 135.89 49.53 0)
       (effects (font (size 1.27 1.27)) hide)
     )
@@
       (effects (font (size 1.27 1.27)) hide)
     )
-    (property "LCSC" "C14663" (at 77.47 106.68 90)
+    (property "LCSC" "C49678" (at 77.47 106.68 90)
+      (effects (font (size 1.27 1.27)) hide)
+    )
+    (property "LINK" "https://jlcpcb.com/partdetail/Yageo-CC0805KRX7R9BB104/C49678" (at 77.47 106.68 0)
       (effects (font (size 1.27 1.27)) hide)
     )
@@
       (effects (font (size 1.27 1.27)) hide)
     )
-    (property "LCSC" "C25804" (at 95.25 88.9 0)
+    (property "LCSC" "C17888" (at 95.25 88.9 0)
+      (effects (font (size 1.27 1.27)) hide)
+    )
+    (property "LINK" "https://jlcpcb.com/partdetail/18576-1206W4F0000T5E/C17888" (at 95.25 88.9 0)
       (effects (font (size 1.27 1.27)) hide)
     )
@@
       (effects (font (size 1.27 1.27)) hide)
     )
-    (property "LCSC" "C14663" (at 144.78 49.53 90)
+    (property "LCSC" "C12891" (at 144.78 49.53 90)
+      (effects (font (size 1.27 1.27)) hide)
+    )
+    (property "LINK" "https://jlcpcb.com/partdetail/13537-CL31A226KAHNNNE/C12891" (at 144.78 49.53 0)
       (effects (font (size 1.27 1.27)) hide)
     )
@@
       (effects (font (size 1.27 1.27)) hide)
     )
-    (property "LCSC" "C14663" (at 45.72 106.68 90)
+    (property "LCSC" "C49678" (at 45.72 106.68 90)
+      (effects (font (size 1.27 1.27)) hide)
+    )
+    (property "LINK" "https://jlcpcb.com/partdetail/Yageo-CC0805KRX7R9BB104/C49678" (at 45.72 106.68 0)
       (effects (font (size 1.27 1.27)) hide)
     )
@@
       (effects (font (size 1.27 1.27)) hide)
     )
-    (property "LCSC" "C14663" (at 114.3 46.99 90)
-      (effects (font (size 1.27 1.27)) hide)
-    )
+    (property "LCSC" "C49678" (at 114.3 46.99 90)
+      (effects (font (size 1.27 1.27)) hide)
+    )
+    (property "LINK" "https://jlcpcb.com/partdetail/Yageo-CC0805KRX7R9BB104/C49678" (at 114.3 46.99 0)
+      (effects (font (size 1.27 1.27)) hide)
+    )

Commit message: added more part numbers
Parts:
- C57: LCSC (none) -> C4747956; LINK (none) -> https://jlcpcb.com/partdetail/Knscha-RST470UF25V032/C4747956
- C66: LCSC (none) -> C4747956; LINK (none) -> https://jlcpcb.com/partdetail/60989-HV101M010E055ETR/C59937
- D9: LCSC (none) -> C3014033; LINK (none) -> https://jlcpcb.com/partdetail/Fosan-SS54B/C3014033
- U4: LCSC (none) -> C6186; LINK (none) -> https://jlcpcb.com/partdetail/Advanced_MonolithicSystems-AM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
- U5: LCSC (none) -> C311983; LINK (none) -> https://jlcpcb.com/partdetail/TexasInstruments-TPS54302DDCR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
Changed lines of the file:
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@@
+      (effects (font (size 1.27 1.27)) hide)
+    )
+    (property "LCSC" "C311983" (at 99.06 49.53 0)
+      (effects (font (size 1.27 1.27)) hide)
+    )
+    (property "LINK" "https://jlcpcb.com/partdetail/TexasInstruments-TPS54302DDCR/C311983" (at 99.06 49.53 0)
       (effects (font (size 1.27 1.27)) hide)
     )
@@
       (effects (font (size 1.27 1.27)) hide)
     )
+    (property "LCSC" "C4747956" (at 53.34 54.61 0)
+      (effects (font (size 1.27 1.27)) hide)
+    )
+    (property "LINK" "https://jlcpcb.com/partdetail/Knscha-RST470UF25V032/C4747956" (at 53.34 54.61 0)
+      (effects (font (size 1.27 1.27)) hide)
+    )
     (pin "1")
     (pin "2")
@@
       (effects (font (size 1.27 1.27)) hide)
     )
+    (property "LCSC" "C6186" (at 63.5 104.14 0)
+      (effects (font (size 1.27 1.27)) hide)
+    )
+    (property "LINK" "https://jlcpcb.com/partdetail/Advanced_MonolithicSystems-AMS1117_33/C6186" (at 63.5 104.14 0)
+      (effects (font (size 1.27 1.27)) hide)
+    )
     (pin "1")
     (pin "2")
@@
       (effects (font (size 1.27 1.27)) hide)
     )
+    (property "LCSC" "C3014033" (at 39.37 48.26 0)
+      (effects (font (size 1.27 1.27)) hide)
+    )
+    (property "LINK" "https://jlcpcb.com/partdetail/Fosan-SS54B/C3014033" (at 39.37 48.26 0)
+      (effects (font (size 1.27 1.27)) hide)
+    )
     (pin "1")
     (pin "2")
@@
       (effects (font (size 1.27 1.27)) hide)
     )
+    (property "LCSC" "C4747956" (at 85.09 107.95 0)
+      (effects (font (size 1.27 1.27)) hide)
+    )
+    (property "LINK" "https://jlcpcb.com/partdetail/60989-HV101M010E055ETR/C59937" (at 85.09 107.95 0)
+      (effects (font (size 1.27 1.27)) hide)
+    )

Commit message: more partnumbers assigned. split difficult values into two parts. add protection of CP_SENSE port
Parts:
- added C69: 22pF, Capacitor_SMD:C_0805_2012Metric_Pad1.18x1.45mm_HandSolder, symbol Device:C_Small
- C66: LCSC C4747956 -> C59937
- R11: footprint Resistor_SMD:R_1206_3216Metric_Pad1.30x1.75mm_HandSolder -> Resistor_SMD:R_0815_2038Metric_Pad1.20x4.05mm_HandSolder; LCSC C25804 -> C149504; LINK (none) -> https://jlcpcb.com/partdetail/160838-0805W8F1003T5E/C149504
- R12: footprint Resistor_SMD:R_1206_3216Metric_Pad1.30x1.75mm_HandSolder -> Resistor_SMD:R_0805_2012Metric_Pad1.20x1.40mm_HandSolder; LCSC C25804 -> C17560; LINK (none) -> https://jlcpcb.com/partdetail/18248-0805W8F2202T5E/C17560
- R12: footprint Resistor_SMD:R_1206_3216Metric_Pad1.30x1.75mm_HandSolder -> Resistor_SMD:R_0815_2038Metric_Pad1.20x4.05mm_HandSolder; LCSC C25804 -> C17633; LINK (none) -> https://jlcpcb.com/partdetail/18321-0805W8F3302T5E/C17633
Connections:
- net 5V: now also C69.2
- net at C69.1, R11.2, R12.2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: now also C69.1
Other:
- note added: "goal: 68pF"
- moved on the sheet: C69, C70, C71, L13, R11, R12, TP5V1

Commit message: footprint corrections. some layout adaptions for new footprints (ongoing)
Parts:
- R11, R12: footprint Resistor_SMD:R_0815_2038Metric_Pad1.20x4.05mm_HandSolder -> Resistor_SMD:R_0805_2012Metric_Pad1.20x1.40mm_HandSolder
Changed lines of the file:
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@@
       (effects (font (size 1.27 1.27)))
     )
-    (property "Footprint" "Resistor_SMD:R_0815_2038Metric_Pad1.20x4.05mm_HandSolder" (at 142.24 50.8 0)
+    (property "Footprint" "Resistor_SMD:R_0805_2012Metric_Pad1.20x1.40mm_HandSolder" (at 142.24 50.8 0)
       (effects (font (size 1.27 1.27)) hide)
     )
@@
       (effects (font (size 1.27 1.27)))
     )
-    (property "Footprint" "Resistor_SMD:R_0815_2038Metric_Pad1.20x4.05mm_HandSolder" (at 142.24 58.42 0)
-      (effects (font (size 1.27 1.27)) hide)
-    )
+    (property "Footprint" "Resistor_SMD:R_0805_2012Metric_Pad1.20x1.40mm_HandSolder" (at 142.24 58.42 0)
+      (effects (font (size 1.27 1.27)) hide)
+    )

Commit message: added part number for the big 10uH
Parts:
- L13: LCSC (none) -> C3000379; LINK (none) -> https://jlcpcb.com/partdetail/3481234-SMDRI125100MT/C3000379
Changed lines of the file:
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@@
       (effects (font (size 1.27 1.27)) hide)
     )
-    (property "Datasheet" "https://datasheet.lcsc.com/lcsc/1810231814_Murata-Electronics-LQM31PN4R7M00L_C162588.pdf" (at 124.46 46.99 0)
+    (property "Datasheet" "~" (at 124.46 46.99 0)
       (effects (font (size 1.27 1.27)) hide)
     )
-    (property "LCSC" "" (at 124.46 46.99 90)
+    (property "LCSC" "C3000379" (at 124.46 46.99 90)
       (effects (font (size 1.27 1.27)) hide)
     )
+    (property "LINK" "https://jlcpcb.com/partdetail/3481234-SMDRI125100MT/C3000379" (at 124.46 46.99 0)
+      (effects (font (size 1.27 1.27)) hide)
+    )

Commit message: added rotation attribute to get the correct footprint rotation at JLCPCB
Parts:
- U4: JLCPCB Rotation Offset (none) -> 180
Changed lines of the file:
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@@
+      (effects (font (size 1.27 1.27)) hide)
+    )
+    (property "JLCPCB Rotation Offset" "180" (at 63.5 104.14 0)
       (effects (font (size 1.27 1.27)) hide)
     )

Commit message: fix rx shortcut. add transformer. correct part number of NCV. Correct footprints of U1 and L11. add mounting holes. stepdown layout improved. added TVS at 12V
Parts:
- added U5: SMAJ18A-TR, SMA_UNI_STM, symbol TVS:SMAJ18A-TR
- L13: footprint Inductor_SMD:L_Wuerth_WE-PD-Typ-LS_Handsoldering -> Inductor_SMD:L_12x12mm_H4.5mm; LCSC C3000379 -> C5127462; LINK https://jlcpcb.com/partdetail/3481234-SMDRI125100MT/C3000379 -> https://jlcpcb.com/partdetail/LantuMicro-SMS1050100MT/C5127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
Connections:
- net 12V_P: now also U5.1 (K)
- net GND: now also U5.2 (A)
Other:
- note removed: "Todo: TVS"
- moved on the sheet: D9
Changed lines of the file:
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@@
   (junction (at 148.59 46.99) (diameter 0) (color 0 0 0 0)
+  )
+  (junction (at 31.75 34.29) (diameter 0) (color 0 0 0 0)
   )
   (junction (at 135.89 55.88) (diameter 0) (color 0 0 0 0)
@@
     (stroke (width 0) (type default))
   )
+  (wire (pts (xy 31.75 34.29) (xy 31.75 41.91))
+    (stroke (width 0) (type default))
+  )
   (wire (pts (xy 91.44 104.14) (xy 95.25 104.14))
     (stroke (width 0) (type default))
@@
     (stroke (width 0) (type default))
   )
-  (wire (pts (xy 44.45 48.26) (xy 44.45 50.8))
-    (stroke (width 0) (type default))
-  )
   (wire (pts (xy 142.24 46.99) (xy 142.24 48.26))
     (stroke (width 0) (type default))
@@
     (stroke (width 0) (type default))
   )
+  (wire (pts (xy 44.45 34.29) (xy 44.45 50.8))
+    (stroke (width 0) (type default))
+  )
   (wire (pts (xy 116.84 46.99) (xy 120.65 46.99))
     (stroke (width 0) (type default))
@@
     (stroke (width 0) (type default))
   )
-  (wire (pts (xy 43.18 48.26) (xy 44.45 48.26))
+  (wire (pts (xy 44.45 50.8) (xy 53.34 50.8))
+    (stroke (width 0) (type default))
+  )
+  (wire (pts (xy 31.75 34.29) (xy 44.45 34.29))
     (stroke (width 0) (type default))
   )
@@
   )
   (wire (pts (xy 116.84 49.53) (xy 109.22 49.53))
-    (stroke (width 0) (type default))
-  )
-  (wire (pts (xy 44.45 50.8) (xy 53.34 50.8))
     (stroke (width 0) (type default))
   )
@@
     (effects (font (size 1.27 1.27)) (justify left bottom))
   )
-  (text "Todo: TVS" (at 35.56 57.15 0)
-    (effects (font (size 1.27 1.27)) (justify left bottom))
-  )
   (text "The bulk capacitor is especially\nimportant when switching high\ncurrents, see DRV8874 data\nsheet."
-    (at 40.64 71.12 0)
+    (at 57.15 68.58 0)
     (effects (font (size 1.27 1.27)) (justify left bottom))
   )
@@
   )
   (text "SS54B is rated for 5A.\nThis is at the border,\nif we drive 6A in the\nlock/unlock motor."
-    (at 29.21 40.64 0)
+    (at 17.78 25.4 0)
     (effects (font (size 1.27 1.27)) (justify left bottom))
   )
@@
     )
   )
-  (global_label "12V" (shape input) (at 35.56 48.26 180) (fields_autoplaced)
+  (global_label "12V" (shape input) (at 24.13 34.29 180) (fields_autoplaced)
     (effects (font (size 1.27 1.27)) (justify right))
-    (property "Intersheetrefs" "${INTERSHEET_REFS}" (at 29.1466 48.26 0)
+    (property "Intersheetrefs" "${INTERSHEET_REFS}" (at 17.7166 34.29 0)
       (effects (font (size 1.27 1.27)) (justify right) hide)
     )
@@
       (effects (font (size 1.27 1.27)))
     )
-    (property "Footprint" "Inductor_SMD:L_Wuerth_WE-PD-Typ-LS_Handsoldering" (at 124.46 46.99 0)
+    (property "Footprint" "Inductor_SMD:L_12x12mm_H4.5mm" (at 124.46 46.99 0)
       (effects (font (size 1.27 1.27)) hide)
     )
@@
       (effects (font (size 1.27 1.27)) hide)
     )
-    (property "LCSC" "C3000379" (at 124.46 46.99 90)
-      (effects (font (size 1.27 1.27)) hide)
-    )
-    (property "LINK" "https://jlcpcb.com/partdetail/3481234-SMDRI125100MT/C3000379" (at 124.46 46.99 0)
+    (property "LCSC" "C5127462" (at 124.46 46.99 90)
+      (effects (font (size 1.27 1.27)) hide)
+    )
+    (property "LINK" "https://jlcpcb.com/partdetail/LantuMicro-SMS1050100MT/C5127462" (at 124.46 46.99 0)
       (effects (font (size 1.27 1.27)) hide)
     )
@@
     )
   )
-  (symbol (lib_id "Device:D_Schottky") (at 39.37 48.26 180) (unit 1)
-    (in_bom yes) (on_board yes) (dnp no) (fields_autoplaced)
-    (property "Reference" "D9" (at 39.6875 43.18 0)
-      (effects (font (size 1.27 1.27)))
-    )
-    (property "Value" "SS54B-HF" (at 39.6875 45.72 0)
-      (effects (font (size 1.27 1.27)))
-    )
-    (property "Footprint" "Diode_SMD:D_SMB_Handsoldering" (at 39.37 48.26 0)
-      (effects (font (size 1.27 1.27)) hide)
-    )
-    (property "Datasheet" "https://www.mouser.de/datasheet/2/80/20190806170503-2505092.pdf" (at 39.37 48.26 0)
-      (effects (font (size 1.27 1.27)) hide)
-    )
-    (property "LCSC" "C3014033" (at 39.37 48.26 0)
-      (effects (font (size 1.27 1.27)) hide)
-    )
-    (property "LINK" "https://jlcpcb.com/partdetail/Fosan-SS54B/C3014033" (at 39.37 48.26 0)
+  (symbol (lib_id "Device:D_Schottky") (at 27.94 34.29 180) (unit 1)
+    (in_bom yes) (on_board yes) (dnp no)
+    (property "Reference" "D9" (at 28.2575 29.21 0)
+      (effects (font (size 1.27 1.27)))
+    )
+    (property "Value" "SS54B-HF" (at 29.21 30.48 0)
+      (effects (font (size 1.27 1.27)))
+    )
+    (property "Footprint" "Diode_SMD:D_SMB_Handsoldering" (at 27.94 34.29 0)
+      (effects (font (size 1.27 1.27)) hide)
+    )
+    (property "Datasheet" "https://www.mouser.de/datasheet/2/80/20190806170503-2505092.pdf" (at 27.94 34.29 0)
+      (effects (font (size 1.27 1.27)) hide)
+    )
+    (property "LCSC" "C3014033" (at 27.94 34.29 0)
+      (effects (font (size 1.27 1.27)) hide)
+    )
+    (property "LINK" "https://jlcpcb.com/partdetail/Fosan-SS54B/C3014033" (at 27.94 34.29 0)
       (effects (font (size 1.27 1.27)) hide)
     )
@@
         )
       )
+    )
+  )
+  (symbol (lib_id "power:GND") (at 31.75 82.55 0) (unit 1)
+    (in_bom yes) (on_board yes) (dnp no)
+    (property "Reference" "#PWR040" (at 31.75 88.9 0)
+      (effects (font (size 1.27 1.27)) hide)
+    )
+    (property "Value" "GND" (at 34.29 86.36 0)
+      (effects (font (size 1.27 1.27)) (justify right))
+    )
+    (property "Footprint" "" (at 31.75 82.55 0)
+      (effects (font (size 1.27 1.27)) hide)
+    )
+    (property "Datasheet" "" (at 31.75 82.55 0)
+      (effects (font (size 1.27 1.27)) hide)
+    )
+    (pin "1")
+    (instances
+      (project "qca7000"
+        (path "/e63e39d7-6ac0-4ffd-8aa3-1841a4541b55"
+          (reference "#PWR040") (unit 1)
+        )
+        (path "/e63e39d7-6ac0-4ffd-8aa3-1841a4541b55/81db238c-e53f-4d52-98ea-36a1df697651"
+          (reference "#PWR086") (unit 1)
+        )
+      )
+    )
+  )
+  (symbol (lib_id "TVS:SMAJ18A-TR") (at 31.75 41.91 270) (unit 1)
+    (in_bom yes) (on_board yes) (dnp no) (fields_autoplaced)
+    (property "Reference" "U5" (at 38.1 61.595 90)
+      (effects (font (size 1.524 1.524)) (justify left))
+    )
+    (property "Value" "SMAJ18A-TR" (at 38.1 64.135 90)
+      (effects (font (size 1.524 1.524)) (justify left))
+    )
+    (property "Footprint" "SMA_UNI_STM" (at 31.75 41.91 0)
+      (effects (font (size 1.27 1.27) italic) hide)
+    )
+    (property "Datasheet" "SMAJ18A-TR" (at 31.75 41.91 0)
+      (effects (font (size 1.27 1.27) italic) hide)
+    )
+    (property "LCSC" "C908771" (at 31.75 41.91 90)
+      (effects (font (size 1.27 1.27)) hide)
+    )
+    (property "LINK" "https://jlcpcb.com/partdetail/Goodwork-SMAJ18A/C908771" (at 31.75 41.91 90)
+      (effects (font (size 1.27 1.27)) hide)
+    )
+    (pin "1")
+    (pin "2")
+    (instances
+      (project "qca7000"
+        (path "/e63e39d7-6ac0-4ffd-8aa3-1841a4541b55/81db238c-e53f-4d52-98ea-36a1df697651"
+          (reference "U5") (unit 1)
+        )
+      )

Commit message: fix: origin of the transformer into the middle. Fix: rotation attributes for jlcpcb
Parts:
- U5: JLCPCB Rotation Offset (none) -> -90
Changed lines of the file:
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@@
+      (effects (font (size 1.27 1.27)) hide)
+    )
+    (property "JLCPCB Rotation Offset" "-90" (at 99.06 49.53 0)
       (effects (font (size 1.27 1.27)) hide)
     )
