File: pcb/powersupply.kicad_sch (KiCad schematic)
At the start: 21 parts, among them U4 AMS1117-3.3, U5 SMAJ18A-TR, U5 TPS54302

Commit message: stepdown L and layout further optimized. fix rotation and layout
Parts:
- L13: footprint Inductor_SMD:L_12x12mm_H4.5mm -> Inductor_SMD:L_6.3x6.3_H3; LCSC C5127462 -> C408412; LINK https://jlcpcb.com/partdetail/LantuMicro-SMS1050100MT/C5127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 -> https://jlcpcb.com/partdetail/Sunlord-MWSA0503S100MT/C408412
Changed lines of the file:
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@@
       (effects (font (size 1.27 1.27)))
     )
-    (property "Footprint" "Inductor_SMD:L_12x12mm_H4.5mm" (at 124.46 46.99 0)
+    (property "Footprint" "Inductor_SMD:L_6.3x6.3_H3" (at 124.46 46.99 0)
       (effects (font (size 1.27 1.27)) hide)
     )
@@
       (effects (font (size 1.27 1.27)) hide)
     )
-    (property "LCSC" "C5127462" (at 124.46 46.99 90)
+    (property "LCSC" "C408412" (at 124.46 46.99 90)
       (effects (font (size 1.27 1.27)) hide)
     )
-    (property "LINK" "https://jlcpcb.com/partdetail/LantuMicro-SMS1050100MT/C5127462" (at 124.46 46.99 0)
+    (property "LINK" "https://jlcpcb.com/partdetail/Sunlord-MWSA0503S100MT/C408412" (at 124.46 46.99 0)
       (effects (font (size 1.27 1.27)) hide)
     )

Commit message: fix: for the big elcap, use jlc part C3445244 to avoid running into expensive standard service
Parts:
- C57: LCSC C4747956 -> C3445244; LINK https://jlcpcb.com/partdetail/Knscha-RST470UF25V032/C4747956 -> https://jlcpcb.com/parts/componentSearch?searchTxt=C3445244
Changed lines of the file:
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@@
       (effects (font (size 1.27 1.27)) hide)
     )
-    (property "LCSC" "C4747956" (at 53.34 54.61 0)
+    (property "LCSC" "C3445244" (at 53.34 54.61 0)
       (effects (font (size 1.27 1.27)) hide)
     )
-    (property "LINK" "https://jlcpcb.com/partdetail/Knscha-RST470UF25V032/C4747956" (at 53.34 54.61 0)
+    (property "LINK" "https://jlcpcb.com/parts/componentSearch?searchTxt=C3445244" (at 53.34 54.61 0)
       (effects (font (size 1.27 1.27)) hide)
     )

Commit message: feature: Added wakeup logic
Parts:
- removed C57: 470uF, Capacitor_SMD:CP_Elec_10x10, symbol Device:C_Polarized
- removed C66: 100uF, Capacitor_SMD:CP_Elec_8x10, symbol Device:C_Polarized
- added C41: 22uF, Capacitor_SMD:C_1210_3225Metric_Pad1.33x2.70mm_HandSolder, symbol Device:C_Small
- added Q10, Q9: 2N7002, Package_TO_SOT_SMD:SOT-23, symbol Transistor_FET:2N7002
- added R65, R66: 22k, Resistor_SMD:R_0805_2012Metric_Pad1.20x1.40mm_HandSolder, symbol Device:R_Small
- added R67: 100k, Resistor_SMD:R_0805_2012Metric_Pad1.20x1.40mm_HandSolder, symbol Device:R_Small
- added R68: 10k, Resistor_SMD:R_0805_2012Metric_Pad1.20x1.40mm_HandSolder, symbol Device:R_Small
- added U10: SMAJ16A-TR, tvs:SMA_UNI_STM, symbol TVS:SMAJ18A-TR
- added U9: CJ431, Package_TO_SOT_SMD:SOT-23-3, symbol Reference_Voltage:TL431DBZ
- U5: value SMAJ18A-TR -> SMAJ16A-TR; footprint SMA_UNI_STM -> tvs:SMA_UNI_STM; LCSC C908771 -> C908770
- renumbered C69 to C27, C68 to C64, C67 to C65, C70 to C66, C71 to C67, C69 to C68, C64 to C73, C65 to C74, D9 to D13, R11 to R23, R12 to R24, R12 to R38, R12 to R43, U5 to U4, U4 to U6
Connections:
- net 12V_P: now also R65.2
- net 3V3_uC: now also C41.2
- net GND: now also C41.1, Q10.2 (S), Q9.2 (S), R67.2, U10.2 (A), U9.3 (A)
- net at U4.5 (EN): now also R65.1, U9.1 (K)
- new net: Q10.3 (D), Q9.3 (D), R66.1, R67.1, U9.2 (REF)
- new net: Q10.1 (G), R68.1
- new net KEEP_POWER_ON: Q9.1 (G)
- new net PP: R66.2
- new net WAKEUP: R68.2, U10.1 (K)
- no-connect marks 1 -> 0
Other:
- note added: "The controller can inhibit turn-off by setting KEEP_POWER_ON high Likewise the controller can also be powered up externally by the WAKEUP signal"
- note added: "When PP drops below 3V EN pin is freed and power supply starts"
- note removed: "The bulk capacitor is especially important when switching high currents, see DRV8874 data sheet."
- moved on the sheet: C27, C64, C65, C66, C67, C68, C73, C74, D13, L13, R23, R24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

Commit message: Corrected pin map for CJ431 Increased variant resistor Added pull-down for Wakeup
Parts:
- added R70: 10k, Resistor_SMD:R_0805_2012Metric_Pad1.20x1.40mm_HandSolder, symbol Device:R_Small
- U9: symbol Reference_Voltage:TL431DBZ -> Reference_Voltage:CJ431DBZ
Connections:
- net GND: now also R70.1
- net at R65.1, U4.5 (EN): now also U9.2 (K); no longer U9.1 (K)
- net at Q10.3 (D), Q9.3 (D), R66.1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: now also U9.1 (REF); no longer U9.2 (REF)
- net at Q10.1 (G), R68.1: now also R70.2
Changed lines of the file:
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@@
   (junction (at 170.18 53.34) (diameter 0) (color 0 0 0 0)
   )
+  (junction (at 93.98 74.93) (diameter 0) (color 0 0 0 0)
+  )
   (junction (at 162.56 53.34) (diameter 0) (color 0 0 0 0)
   )
@@
   (junction (at 43.18 118.11) (diameter 0) (color 0 0 0 0)
   )
+  (junction (at 97.79 69.85) (diameter 0) (color 0 0 0 0)
+  )
   (junction (at 162.56 44.45) (diameter 0) (color 0 0 0 0)
   )
@@
     (stroke (width 0) (type default))
   )
+  (wire (pts (xy 93.98 69.85) (xy 97.79 69.85))
+    (stroke (width 0) (type default))
+  )
   (wire (pts (xy 49.53 31.75) (xy 49.53 48.26))
     (stroke (width 0) (type default))
@@
     (stroke (width 0) (type default))
   )
-  (wire (pts (xy 80.01 74.93) (xy 105.41 74.93))
+  (wire (pts (xy 80.01 74.93) (xy 93.98 74.93))
     (stroke (width 0) (type default))
   )
@@
   )
   (wire (pts (xy 116.84 60.96) (xy 116.84 63.5))
+    (stroke (width 0) (type default))
+  )
+  (wire (pts (xy 93.98 74.93) (xy 105.41 74.93))
     (stroke (width 0) (type default))
   )
@@
     )
   )
-  (symbol (lib_id "Reference_Voltage:TL431DBZ") (at 119.38 60.96 90) (unit 1)
+  (symbol (lib_id "Reference_Voltage:CJ431DBZ") (at 119.38 60.96 90) (unit 1)
     (in_bom yes) (on_board yes) (dnp no) (fields_autoplaced)
     (property "Reference" "U9" (at 121.158 59.7479 90)
@@
       (effects (font (size 1.27 1.27) italic) hide)
     )
-    (property "Datasheet" "http://www.ti.com/lit/ds/symlink/tl431.pdf" (at 119.38 60.96 0)
+    (property "Datasheet" "http://www.ti.com/lit/ds/symlink/tl431.pdf" (at 128.27 59.69 0)
       (effects (font (size 1.27 1.27) italic) hide)
     )
-    (property "LCSC" "C3113" (at 119.38 60.96 90)
+    (property "LCSC" "C3113" (at 119.38 40.64 90)
       (effects (font (size 1.27 1.27)) hide)
     )
@@
         )
       )
+    )
+  )
+  (symbol (lib_id "Device:R_Small") (at 93.98 72.39 180) (unit 1)
+    (in_bom yes) (on_board yes) (dnp no)
+    (property "Reference" "R70" (at 96.52 73.66 0)
+      (effects (font (size 1.27 1.27)))
+    )
+    (property "Value" "10k" (at 96.52 71.12 0)
+      (effects (font (size 1.27 1.27)))
+    )
+    (property "Footprint" "Resistor_SMD:R_0805_2012Metric_Pad1.20x1.40mm_HandSolder" (at 93.98 72.39 0)
+      (effects (font (size 1.27 1.27)) hide)
+    )
+    (property "Datasheet" "~" (at 93.98 72.39 0)
+      (effects (font (size 1.27 1.27)) hide)
+    )
+    (property "LCSC" "C17414" (at 93.98 72.39 0)
+      (effects (font (size 1.27 1.27)) hide)
+    )
+    (property "LINK" "https://jlcpcb.com/partdetail/18102-0805W8F1002T5E/C17414" (at 93.98 72.39 0)
+      (effects (font (size 1.27 1.27)) hide)
+    )
+    (pin "1")
+    (pin "2")
+    (instances
+      (project "qca7000"
+        (path "/e63e39d7-6ac0-4ffd-8aa3-1841a4541b55/81db238c-e53f-4d52-98ea-36a1df697651"
+          (reference "R70") (unit 1)
+        )
+      )

Commit message: Redesigned wakeup circuit
Parts:
- removed Q10, Q9: 2N7002, Package_TO_SOT_SMD:SOT-23, symbol Transistor_FET:2N7002
- removed R66: 22k, Resistor_SMD:R_0805_2012Metric_Pad1.20x1.40mm_HandSolder, symbol Device:R_Small
- removed R67: 100k, Resistor_SMD:R_0805_2012Metric_Pad1.20x1.40mm_HandSolder, symbol Device:R_Small
- removed R68, R70: 10k, Resistor_SMD:R_0805_2012Metric_Pad1.20x1.40mm_HandSolder, symbol Device:R_Small
- removed U9: CJ431, Package_TO_SOT_SMD:SOT-23-3, symbol Reference_Voltage:CJ431DBZ
- added C82: 10uF 25V, Capacitor_SMD:C_0805_2012Metric_Pad1.18x1.45mm_HandSolder, symbol Device:C_Small
- added C83: 100nF, Capacitor_SMD:C_0805_2012Metric_Pad1.18x1.45mm_HandSolder, symbol Device:C_Small
- added C84: 10uF, Capacitor_SMD:C_0805_2012Metric_Pad1.18x1.45mm_HandSolder, symbol Device:C_Small
- added D18, D19, D21: B5819W, Diode_SMD:D_SOD-123, symbol Diode:1N4148W
- added Q2, Q9: AO3401A, Package_TO_SOT_SMD:SOT-23, symbol Transistor_FET:AO3401A
- added Q3: 2N7002, Package_TO_SOT_SMD:SOT-23, symbol Transistor_FET:2N7002
- added R56: 100k, Resistor_SMD:R_0805_2012Metric_Pad1.20x1.40mm_HandSolder, symbol Device:R_Small
- added R64: 10k, Resistor_SMD:R_0805_2012Metric_Pad1.20x1.40mm_HandSolder, symbol Device:R_Small
- R65: value 22k -> 3.3K; LCSC C17560 -> C26010; LINK https://jlcpcb.com/partdetail/18248-0805W8F2202T5E/C17560 -> https://jlcpcb.com/partdetail/26753-0805W8F3301T5E/C26010
Connections:
- net 12V_P: now also Q2.2 (S), Q9.2 (S), R64.1; no longer R65.2
- net GND: now also C83.1, Q3.2 (S), R56.2
- net KEEP_POWER_ON: now also Q3.1 (G)
- net WAKEUP: now also D19.2 (A)
- net at U4.5 (EN): now also C82.1, D19.1 (K), Q2.3 (D), Q9.3 (D), R56.1; no longer R65.1
- new net: D21.2 (A), Q2.1 (G), Q3.3 (D), R64.2
- new net: C82.2, C83.2, R65.2
- new net: C84.1, D21.1 (K)
- new net: D18.1 (K), R65.1
- new net BUTTON: Q9.1 (G)
- new net CP: D18.2 (A)
- new net PP_WAKE: C84.2
Other:
- note added: "C82 changes the continous high level of the filtered CP signal to a one-shot pulse when the cable is plugged in. We can therefor choose to shut down the controller even with the cable still plugged in e.g. when no charge power available on solar powered systems"
- note removed: "The controller can inhibit turn-off by setting KEEP_POWER_ON high Likewise the controller can also be powered up externally by the WAKEUP signal"
- note removed: "When PP drops below 3V EN pin is freed and power supply starts"
- moved on the sheet: C27, C41, C64, C65, C66, C67, C68, C73, C74, L13, R23, R24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

Commit message: Added 1M discharge resistor for CP enable Removed momentary turn-on resitor for PP enable because always charged by uC voltage divider
Parts:
- removed C84: 10uF, Capacitor_SMD:C_0805_2012Metric_Pad1.18x1.45mm_HandSolder, symbol Device:C_Small
- added R67: 1M, Resistor_SMD:R_0805_2012Metric_Pad1.20x1.40mm_HandSolder, symbol Device:R_Small
Connections:
- net GND: now also R67.2
- net PP_WAKE: now also D21.1 (K)
- net at C82.2, C83.2, R65.2: now also R67.1
Other:
- moved on the sheet: C82
Changed lines of the file:
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@@
   (junction (at 227.33 53.34) (diameter 0) (color 0 0 0 0)
   )
+  (junction (at 152.4 59.69) (diameter 0) (color 0 0 0 0)
+  )
+  (junction (at 146.05 67.31) (diameter 0) (color 0 0 0 0)
+  )
   (junction (at 168.91 57.15) (diameter 0) (color 0 0 0 0)
   )
@@
     (stroke (width 0) (type default))
   )
-  (wire (pts (xy 95.25 85.09) (xy 97.79 85.09))
-    (stroke (width 0) (type default))
-  )
   (wire (pts (xy 168.91 59.69) (xy 168.91 77.47))
     (stroke (width 0) (type default))
@@
     (stroke (width 0) (type default))
   )
+  (wire (pts (xy 152.4 67.31) (xy 146.05 67.31))
+    (stroke (width 0) (type default))
+  )
   (wire (pts (xy 151.13 77.47) (xy 157.48 77.47))
     (stroke (width 0) (type default))
@@
     (stroke (width 0) (type default))
   )
+  (wire (pts (xy 152.4 59.69) (xy 158.75 59.69))
+    (stroke (width 0) (type default))
+  )
+  (wire (pts (xy 152.4 59.69) (xy 152.4 60.96))
+    (stroke (width 0) (type default))
+  )
   (wire (pts (xy 233.68 49.53) (xy 233.68 50.8))
     (stroke (width 0) (type default))
@@
     (stroke (width 0) (type default))
   )
-  (wire (pts (xy 87.63 85.09) (xy 90.17 85.09))
+  (wire (pts (xy 87.63 85.09) (xy 97.79 85.09))
     (stroke (width 0) (type default))
   )
@@
     (stroke (width 0) (type default))
   )
+  (wire (pts (xy 152.4 66.04) (xy 152.4 67.31))
+    (stroke (width 0) (type default))
+  )
   (wire (pts (xy 168.91 57.15) (xy 168.91 59.69))
     (stroke (width 0) (type default))
   )
-  (wire (pts (xy 153.67 59.69) (xy 168.91 59.69))
+  (wire (pts (xy 163.83 59.69) (xy 168.91 59.69))
     (stroke (width 0) (type default))
   )
@@
     (stroke (width 0) (type default))
   )
-  (wire (pts (xy 146.05 59.69) (xy 148.59 59.69))
-    (stroke (width 0) (type default))
-  )
-  (wire (pts (xy 99.06 93.98) (xy 101.6 93.98))
+  (wire (pts (xy 146.05 59.69) (xy 152.4 59.69))
+    (stroke (width 0) (type default))
+  )
+  (wire (pts (xy 95.25 93.98) (xy 101.6 93.98))
     (stroke (width 0) (type default))
   )
@@
     )
   )
-  (global_label "KEEP_POWER_ON" (shape input) (at 99.06 93.98 180) (fields_autoplaced)
+  (global_label "KEEP_POWER_ON" (shape input) (at 95.25 93.98 180) (fields_autoplaced)
     (effects (font (size 1.27 1.27)) (justify right))
-    (property "Intersheetrefs" "${INTERSHEET_REFS}" (at 80.1697 93.98 0)
+    (property "Intersheetrefs" "${INTERSHEET_REFS}" (at 76.3597 93.98 0)
       (effects (font (size 1.27 1.27)) (justify right) hide)
     )
@@
     )
   )
-  (symbol (lib_id "Device:C_Small") (at 151.13 59.69 270) (unit 1)
-    (in_bom yes) (on_board yes) (dnp no)
-    (property "Reference" "C82" (at 149.86 64.77 0)
-      (effects (font (size 1.27 1.27)))
-    )
-    (property "Value" "10uF 25V" (at 153.67 64.77 0)
-      (effects (font (size 1.27 1.27)))
-    )
-    (property "Footprint" "Capacitor_SMD:C_0805_2012Metric_Pad1.18x1.45mm_HandSolder" (at 151.13 59.69 0)
-      (effects (font (size 1.27 1.27)) hide)
-    )
-    (property "Datasheet" "https://datasheet.lcsc.com/lcsc/1811110921_Samsung-Electro-Mechanics-CL10A106MA8NRNC_C96446.pdf" (at 151.13 59.69 0)
-      (effects (font (size 1.27 1.27)) hide)
-    )
-    (property "LCSC" "C15850" (at 151.13 59.69 0)
-      (effects (font (size 1.27 1.27)) hide)
-    )
-    (property "LINK" "https://jlcpcb.com/partdetail/16532-CL21A106KAYNNNE/C15850" (at 151.13 59.69 0)
+  (symbol (lib_id "Device:C_Small") (at 161.29 59.69 270) (unit 1)
+    (in_bom yes) (on_board yes) (dnp no)
+    (property "Reference" "C82" (at 161.29 55.88 90)
+      (effects (font (size 1.27 1.27)))
+    )
+    (property "Value" "10uF 25V" (at 163.83 64.77 0)
+      (effects (font (size 1.27 1.27)))
+    )
+    (property "Footprint" "Capacitor_SMD:C_0805_2012Metric_Pad1.18x1.45mm_HandSolder" (at 161.29 59.69 0)
+      (effects (font (size 1.27 1.27)) hide)
+    )
+    (property "Datasheet" "https://datasheet.lcsc.com/lcsc/1811110921_Samsung-Electro-Mechanics-CL10A106MA8NRNC_C96446.pdf" (at 161.29 59.69 0)
+      (effects (font (size 1.27 1.27)) hide)
+    )
+    (property "LCSC" "C15850" (at 161.29 59.69 0)
+      (effects (font (size 1.27 1.27)) hide)
+    )
+    (property "LINK" "https://jlcpcb.com/partdetail/16532-CL21A106KAYNNNE/C15850" (at 161.29 59.69 0)
       (effects (font (size 1.27 1.27)) hide)
     )
@@
     )
   )
+  (symbol (lib_id "Device:R_Small") (at 152.4 63.5 0) (unit 1)
+    (in_bom yes) (on_board yes) (dnp no)
+    (property "Reference" "R67" (at 154.94 60.96 0)
+      (effects (font (size 1.27 1.27)))
+    )
+    (property "Value" "1M" (at 154.94 64.77 0)
+      (effects (font (size 1.27 1.27)))
+    )
+    (property "Footprint" "Resistor_SMD:R_0805_2012Metric_Pad1.20x1.40mm_HandSolder" (at 152.4 63.5 0)
+      (effects (font (size 1.27 1.27)) hide)
+    )
+    (property "Datasheet" "~" (at 152.4 63.5 0)
+      (effects (font (size 1.27 1.27)) hide)
+    )
+    (property "LCSC" "C22935" (at 152.4 63.5 0)
+      (effects (font (size 1.27 1.27)) hide)
+    )
+    (property "LINK" "https://jlcpcb.com/partdetail/23662-0603WAF1004T5E/C22935" (at 152.4 63.5 0)
+      (effects (font (size 1.27 1.27)) hide)
+    )
+    (pin "1")
+    (pin "2")
+    (instances
+      (project "qca7000"
+        (path "/e63e39d7-6ac0-4ffd-8aa3-1841a4541b55/81db238c-e53f-4d52-98ea-36a1df697651"
+          (reference "R67") (unit 1)
+        )
+      )
+    )
+  )
   (symbol (lib_id "power:GND") (at 227.33 60.96 0) (unit 1)
     (in_bom yes) (on_board yes) (dnp no)
@@
         )
       )
-    )
-  )
-  (symbol (lib_id "Device:C_Small") (at 92.71 85.09 270) (unit 1)
-    (in_bom yes) (on_board yes) (dnp no)
-    (property "Reference" "C84" (at 91.44 82.55 90)
-      (effects (font (size 1.27 1.27)))
-    )
-    (property "Value" "10uF" (at 91.44 88.9 90)
-      (effects (font (size 1.27 1.27)))
-    )
-    (property "Footprint" "Capacitor_SMD:C_0805_2012Metric_Pad1.18x1.45mm_HandSolder" (at 92.71 85.09 0)
-      (effects (font (size 1.27 1.27)) hide)
-    )
-    (property "Datasheet" "https://datasheet.lcsc.com/lcsc/1811110921_Samsung-Electro-Mechanics-CL10A106MA8NRNC_C96446.pdf" (at 92.71 85.09 0)
-      (effects (font (size 1.27 1.27)) hide)
-    )
-    (property "LCSC" "C15850" (at 92.71 85.09 0)
-      (effects (font (size 1.27 1.27)) hide)
-    )
-    (property "LINK" "https://jlcpcb.com/partdetail/16532-CL21A106KAYNNNE/C15850" (at 92.71 85.09 0)
-      (effects (font (size 1.27 1.27)) hide)
-    )
-    (pin "1")
-    (pin "2")
-    (instances
-      (project "qca7000"
-        (path "/e63e39d7-6ac0-4ffd-8aa3-1841a4541b55/81db238c-e53f-4d52-98ea-36a1df697651"
-          (reference "C84") (unit 1)
-        )
-      )

Commit message: BOM optimization
Parts:
- D13: value SS54B-HF -> SS54; LCSC C3014033 -> C22452; LINK https://jlcpcb.com/partdetail/Fosan-SS54B/C3014033 -> https://jlcpcb.com/partdetail/Mdd-SS54/C22452
Changed lines of the file:
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@@
       (effects (font (size 1.27 1.27)))
     )
-    (property "Value" "SS54B-HF" (at 34.29 27.94 0)
+    (property "Value" "SS54" (at 34.29 27.94 0)
       (effects (font (size 1.27 1.27)))
     )
@@
       (effects (font (size 1.27 1.27)) hide)
     )
-    (property "Datasheet" "https://www.mouser.de/datasheet/2/80/20190806170503-2505092.pdf" (at 33.02 31.75 0)
+    (property "Datasheet" "~" (at 33.02 31.75 0)
       (effects (font (size 1.27 1.27)) hide)
     )
-    (property "LCSC" "C3014033" (at 33.02 31.75 0)
+    (property "LCSC" "C22452" (at 33.02 31.75 0)
       (effects (font (size 1.27 1.27)) hide)
     )
-    (property "LINK" "https://jlcpcb.com/partdetail/Fosan-SS54B/C3014033" (at 33.02 31.75 0)
+    (property "LINK" "https://jlcpcb.com/partdetail/Mdd-SS54/C22452" (at 33.02 31.75 0)
       (effects (font (size 1.27 1.27)) hide)
     )

Commit message: Made PP standby and button pullup 1k Improved connection of TVS diode
Parts:
- R64: value 10k -> 1k; LCSC C17414 -> C17513; LINK https://jlcpcb.com/partdetail/18102-0805W8F1002T5E/C17414 -> https://jlcpcb.com/partdetail/18201-0805W8F1001T5E/C17513
Connections:
- net 12V_P: now also R64.2; no longer R64.1
- net at D21.2 (A), Q2.1 (G), Q3.3 (D): now also R64.1; no longer R64.2
Changed lines of the file:
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@@
+    )
+  )
+  (symbol (lib_id "Device:R_Small") (at 109.22 72.39 180) (unit 1)
+    (in_bom yes) (on_board yes) (dnp no)
+    (property "Reference" "R64" (at 106.68 72.39 90)
+      (effects (font (size 1.27 1.27)))
+    )
+    (property "Value" "1k" (at 111.76 72.39 90)
+      (effects (font (size 1.27 1.27)))
+    )
+    (property "Footprint" "Resistor_SMD:R_0805_2012Metric_Pad1.20x1.40mm_HandSolder" (at 109.22 72.39 0)
+      (effects (font (size 1.27 1.27)) hide)
+    )
+    (property "Datasheet" "https://datasheet.lcsc.com/lcsc/1811101920_UNI-ROYAL-Uniroyal-Elec-0603WAF3301T5E_C22978.pdf" (at 109.22 72.39 0)
+      (effects (font (size 1.27 1.27)) hide)
+    )
+    (property "LCSC" "C17513" (at 109.22 72.39 90)
+      (effects (font (size 1.27 1.27)) hide)
+    )
+    (property "LINK" "https://jlcpcb.com/partdetail/18201-0805W8F1001T5E/C17513" (at 109.22 72.39 0)
+      (effects (font (size 1.27 1.27)) hide)
+    )
+    (pin "1")
+    (pin "2")
+    (instances
+      (project "qca7000"
+        (path "/e63e39d7-6ac0-4ffd-8aa3-1841a4541b55/81db238c-e53f-4d52-98ea-36a1df697651"
+          (reference "R64") (unit 1)
+        )
+      )
     )
   )
@@
         )
       )
-    )
-  )
-  (symbol (lib_id "Device:R_Small") (at 109.22 72.39 0) (unit 1)
-    (in_bom yes) (on_board yes) (dnp no)
-    (property "Reference" "R64" (at 111.76 69.85 0)
-      (effects (font (size 1.27 1.27)))
-    )
-    (property "Value" "10k" (at 111.76 73.66 0)
-      (effects (font (size 1.27 1.27)))
-    )
-    (property "Footprint" "Resistor_SMD:R_0805_2012Metric_Pad1.20x1.40mm_HandSolder" (at 109.22 72.39 0)
-      (effects (font (size 1.27 1.27)) hide)
-    )
-    (property "Datasheet" "~" (at 109.22 72.39 0)
-      (effects (font (size 1.27 1.27)) hide)
-    )
-    (property "LCSC" "C17414" (at 109.22 72.39 0)
-      (effects (font (size 1.27 1.27)) hide)
-    )
-    (property "LINK" "https://jlcpcb.com/partdetail/18102-0805W8F1002T5E/C17414" (at 109.22 72.39 0)
-      (effects (font (size 1.27 1.27)) hide)
-    )
-    (pin "1")
-    (pin "2")
-    (instances
-      (project "qca7000"
-        (path "/e63e39d7-6ac0-4ffd-8aa3-1841a4541b55/81db238c-e53f-4d52-98ea-36a1df697651"
-          (reference "R64") (unit 1)
-        )
-      )
