File: pcb/qca7000.kicad_sch (KiCad schematic)
At the start: 84 parts, among them J1 Conn_01x04_Pin, J2 Conn_01x08_Pin, U1 25Q16, Y1 25MHz

Commit message: footprint corrections. some layout adaptions for new footprints (ongoing)
Parts:
- R1, R2: footprint Resistor_SMD:R_1206_3216Metric_Pad1.30x1.75mm_HandSolder -> Resistor_SMD:R_0805_2012Metric_Pad1.20x1.40mm_HandSolder; LCSC C17958 -> C17561; LINK https://jlcpcb.com/partdetail/18646-1206W4F220JT5E/C17958 -> https://jlcpcb.com/partdetail/18249-0805W8F220JT5E/C17561
Changed lines of the file:
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@@
       (effects (font (size 1.27 1.27)) (justify left))
     )
-    (property "Footprint" "Resistor_SMD:R_1206_3216Metric_Pad1.30x1.75mm_HandSolder" (at 26.67 24.13 0)
+    (property "Footprint" "Resistor_SMD:R_0805_2012Metric_Pad1.20x1.40mm_HandSolder" (at 26.67 24.13 0)
       (effects (font (size 1.27 1.27)) hide)
     )
@@
       (effects (font (size 1.27 1.27)) hide)
     )
-    (property "LCSC" "C17958" (at 26.67 24.13 0)
-      (effects (font (size 1.27 1.27)) hide)
-    )
-    (property "LINK" "https://jlcpcb.com/partdetail/18646-1206W4F220JT5E/C17958" (at 26.67 24.13 0)
+    (property "LCSC" "C17561" (at 26.67 24.13 0)
+      (effects (font (size 1.27 1.27)) hide)
+    )
+    (property "LINK" "https://jlcpcb.com/partdetail/18249-0805W8F220JT5E/C17561" (at 26.67 24.13 0)
       (effects (font (size 1.27 1.27)) hide)
     )
@@
       (effects (font (size 1.27 1.27)) (justify left))
     )
-    (property "Footprint" "Resistor_SMD:R_1206_3216Metric_Pad1.30x1.75mm_HandSolder" (at 26.67 39.37 0)
+    (property "Footprint" "Resistor_SMD:R_0805_2012Metric_Pad1.20x1.40mm_HandSolder" (at 26.67 39.37 0)
       (effects (font (size 1.27 1.27)) hide)
     )
@@
       (effects (font (size 1.27 1.27)) hide)
     )
-    (property "LCSC" "C17958" (at 26.67 39.37 0)
-      (effects (font (size 1.27 1.27)) hide)
-    )
-    (property "LINK" "https://jlcpcb.com/partdetail/18646-1206W4F220JT5E/C17958" (at 26.67 39.37 0)
-      (effects (font (size 1.27 1.27)) hide)
-    )
+    (property "LCSC" "C17561" (at 26.67 39.37 0)
+      (effects (font (size 1.27 1.27)) hide)
+    )
+    (property "LINK" "https://jlcpcb.com/partdetail/18249-0805W8F220JT5E/C17561" (at 26.67 39.37 0)
+      (effects (font (size 1.27 1.27)) hide)
+    )

Commit message: added alternative 1206 for the 0603 capacitors
Parts:
- added C17a1, C29a1: 6.8pF, Capacitor_SMD:C_1206_3216Metric_Pad1.33x1.80mm_HandSolder, symbol Device:C_Small
Connections:
- net GND: now also C17a1.1, C29a1.1
- net RBIAS: now reaches D8.51 (RBIAS), R9.1
- net SW_VDD_OUT: now reaches D8.10 (SW_VDD_OUT), D8.9 (SW_VDD_OUT), L11.1
- net at C17.2, D8.37 (XTAL_IN), Y1.1: now also C17a1.2
- net RSVD05: now reaches C51.2, D8.48 (RSVD02), D8.52 (RSVD05)
- net at C29.2, R5.1, Y1.3: now also C29a1.2
Other:
- note added: "alternative footprints for C17, C29"
- moved on the sheet: C29
Changed lines of the file:
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@@
   (junction (at 135.89 175.26) (diameter 0) (color 0 0 0 0)
   )
+  (junction (at 34.29 109.22) (diameter 0) (color 0 0 0 0)
+  )
   (junction (at 54.61 130.81) (diameter 0) (color 0 0 0 0)
   )
+  (junction (at 22.86 106.68) (diameter 0) (color 0 0 0 0)
+  )
   (junction (at 22.86 101.6) (diameter 0) (color 0 0 0 0)
   )
@@
   (junction (at 46.99 58.42) (diameter 0) (color 0 0 0 0)
   )
-  (junction (at 34.29 109.22) (diameter 0) (color 0 0 0 0)
+  (junction (at 22.86 90.17) (diameter 0) (color 0 0 0 0)
   )
   (junction (at 90.17 38.1) (diameter 0) (color 0 0 0 0)
@@
   (junction (at 59.69 66.04) (diameter 0) (color 0 0 0 0)
   )
+  (junction (at 34.29 106.68) (diameter 0) (color 0 0 0 0)
+  )
   (junction (at 41.91 133.35) (diameter 0) (color 0 0 0 0)
   )
@@
     (stroke (width 0) (type default))
   )
+  (wire (pts (xy 22.86 82.55) (xy 22.86 90.17))
+    (stroke (width 0) (type default))
+  )
   (wire (pts (xy 99.06 22.86) (xy 90.17 22.86))
     (stroke (width 0) (type default))
@@
     (stroke (width 0) (type default))
   )
+  (wire (pts (xy 34.29 106.68) (xy 34.29 109.22))
+    (stroke (width 0) (type default))
+  )
   (wire (pts (xy 173.99 87.63) (xy 173.99 91.44))
     (stroke (width 0) (type default))
@@
     (stroke (width 0) (type default))
   )
-  (wire (pts (xy 34.29 105.41) (xy 34.29 109.22))
+  (wire (pts (xy 34.29 105.41) (xy 34.29 106.68))
     (stroke (width 0) (type default))
   )
@@
     (stroke (width 0) (type default))
   )
+  (wire (pts (xy 30.48 111.76) (xy 34.29 111.76))
+    (stroke (width 0) (type default))
+  )
   (wire (pts (xy 34.29 44.45) (xy 41.91 44.45))
     (stroke (width 0) (type default))
@@
     (stroke (width 0) (type default))
   )
+  (wire (pts (xy 25.4 82.55) (xy 22.86 82.55))
+    (stroke (width 0) (type default))
+  )
   (wire (pts (xy 49.53 143.51) (xy 59.69 143.51))
     (stroke (width 0) (type default))
@@
     (stroke (width 0) (type default))
   )
+  (wire (pts (xy 30.48 82.55) (xy 34.29 82.55))
+    (stroke (width 0) (type default))
+  )
+  (wire (pts (xy 34.29 109.22) (xy 34.29 111.76))
+    (stroke (width 0) (type default))
+  )
   (wire (pts (xy 22.86 90.17) (xy 22.86 101.6))
     (stroke (width 0) (type default))
@@
     (stroke (width 0) (type default))
   )
-  (wire (pts (xy 34.29 109.22) (xy 30.48 109.22))
+  (wire (pts (xy 34.29 106.68) (xy 30.48 106.68))
     (stroke (width 0) (type default))
   )
@@
     (stroke (width 0) (type default))
   )
-  (wire (pts (xy 22.86 109.22) (xy 25.4 109.22))
+  (wire (pts (xy 22.86 106.68) (xy 25.4 106.68))
     (stroke (width 0) (type default))
   )
@@
     (stroke (width 0) (type default))
   )
+  (wire (pts (xy 25.4 111.76) (xy 22.86 111.76))
+    (stroke (width 0) (type default))
+  )
   (wire (pts (xy 123.19 165.1) (xy 123.19 162.56))
     (stroke (width 0) (type default))
@@
     (stroke (width 0) (type default))
   )
+  (wire (pts (xy 22.86 111.76) (xy 22.86 106.68))
+    (stroke (width 0) (type default))
+  )
   (wire (pts (xy 69.85 176.53) (xy 69.85 179.07))
     (stroke (width 0) (type default))
@@
     (stroke (width 0) (type default))
   )
+  (wire (pts (xy 34.29 82.55) (xy 34.29 90.17))
+    (stroke (width 0) (type default))
+  )
   (wire (pts (xy 227.33 87.63) (xy 226.06 87.63))
     (stroke (width 0) (type default))
@@
     (stroke (width 0) (type default))
   )
-  (wire (pts (xy 22.86 101.6) (xy 22.86 109.22))
+  (wire (pts (xy 22.86 101.6) (xy 22.86 106.68))
     (stroke (width 0) (type default))
   )
@@
     (stroke (width 0) (type default))
   )
-  (wire (pts (xy 72.39 158.75) (xy 72.39 151.13))
-    (stroke (width 0) (type default))
-  )
   (wire (pts (xy 144.78 146.05) (xy 152.4 146.05))
     (stroke (width 0) (type default))
@@
     (stroke (width 0) (type default))
   )
+  (wire (pts (xy 72.39 151.13) (xy 72.39 158.75))
+    (stroke (width 0) (type default))
+  )
   (wire (pts (xy 110.49 92.71) (xy 110.49 96.52))
     (stroke (width 0) (type default))
@@
     (effects (font (size 1.27 1.27)) (justify left bottom))
   )
+  (text "alternative footprints for C17, C29" (at 16.51 113.03 90)
+    (effects (font (size 1.27 1.27)) (justify left bottom))
+  )
   (text "3rd Order Butterworth Bandpass\nLower Cutoff Freq. = 1.900 MHz; Upper Cutoff Freq. = 31.00 MHz\nhttps://rf-tools.com/lc-filter/"
     (at 71.12 53.34 0)
@@
     (effects (font (size 1.27 1.27)) (justify left bottom))
   )
+  (label "SW_VDD_OUT" (at 148.59 128.27 0) (fields_autoplaced)
+    (effects (font (size 1.27 1.27)) (justify left bottom))
+  )
+  (label "RSVD05" (at 80.01 175.26 0) (fields_autoplaced)
+    (effects (font (size 1.27 1.27)) (justify left bottom))
+  )
+  (label "RBIAS" (at 72.39 151.13 0) (fields_autoplaced)
+    (effects (font (size 1.27 1.27)) (justify left bottom))
+  )
   (global_label "RX_N" (shape input) (at 24.13 29.21 180) (fields_autoplaced)
     (effects (font (size 1.27 1.27)) (justify right))
@@
     )
   )
-  (symbol (lib_id "Device:C_Small") (at 27.94 109.22 90) (unit 1)
+  (symbol (lib_id "Device:C_Small") (at 27.94 106.68 90) (unit 1)
     (in_bom yes) (on_board yes) (dnp no)
-    (property "Reference" "C29" (at 27.94 105.41 90)
+    (property "Reference" "C29" (at 25.4 105.41 90)
       (effects (font (size 1.27 1.27)))
     )
-    (property "Value" "6.8pF" (at 27.94 113.03 90)
+    (property "Value" "6.8pF" (at 31.75 107.95 90)
       (effects (font (size 1.27 1.27)))
     )
-    (property "Footprint" "Capacitor_SMD:C_0603_1608Metric_Pad1.08x0.95mm_HandSolder" (at 27.94 109.22 0)
+    (property "Footprint" "Capacitor_SMD:C_0603_1608Metric_Pad1.08x0.95mm_HandSolder" (at 27.94 106.68 0)
       (effects (font (size 1.27 1.27)) hide)
     )
-    (property "Datasheet" "https://datasheet.lcsc.com/lcsc/1811061822_FH-Guangdong-Fenghua-Advanced-Tech-0603CG6R8C500NT_C1679.pdf" (at 27.94 109.22 0)
+    (property "Datasheet" "https://datasheet.lcsc.com/lcsc/1811061822_FH-Guangdong-Fenghua-Advanced-Tech-0603CG6R8C500NT_C1679.pdf" (at 27.94 106.68 0)
       (effects (font (size 1.27 1.27)) hide)
     )
-    (property "LCSC" "C1679" (at 27.94 109.22 0)
+    (property "LCSC" "C1679" (at 27.94 106.68 0)
       (effects (font (size 1.27 1.27)) hide)
     )
-    (property "LINK" "https://jlcpcb.com/partdetail/2031-0603CG6R8C500NT/C1679" (at 27.94 109.22 0)
+    (property "LINK" "https://jlcpcb.com/partdetail/2031-0603CG6R8C500NT/C1679" (at 27.94 106.68 0)
       (effects (font (size 1.27 1.27)) hide)
     )
@@
     )
   )
+  (symbol (lib_id "Device:C_Small") (at 27.94 111.76 90) (unit 1)
+    (in_bom yes) (on_board yes) (dnp no)
+    (property "Reference" "C29a1" (at 20.32 111.76 90)
+      (effects (font (size 1.27 1.27)))
+    )
+    (property "Value" "6.8pF" (at 22.86 109.22 90)
+      (effects (font (size 1.27 1.27)))
+    )
+    (property "Footprint" "Capacitor_SMD:C_1206_3216Metric_Pad1.33x1.80mm_HandSolder" (at 27.94 111.76 0)
+      (effects (font (size 1.27 1.27)) hide)
+    )
+    (property "Datasheet" "" (at 27.94 111.76 0)
+      (effects (font (size 1.27 1.27)) hide)
+    )
+    (property "LCSC" "" (at 27.94 111.76 0)
+      (effects (font (size 1.27 1.27)) hide)
+    )
+    (property "LINK" "" (at 27.94 111.76 0)
+      (effects (font (size 1.27 1.27)) hide)
+    )
+    (pin "1")
+    (pin "2")
+    (instances
+      (project "qca7000"
+        (path "/e63e39d7-6ac0-4ffd-8aa3-1841a4541b55"
+          (reference "C29a1") (unit 1)
+        )
+      )
+    )
+  )
   (symbol (lib_name "C_Small_22") (lib_id "Device:C_Small") (at 57.15 101.6 270) (unit 1)
     (in_bom yes) (on_board yes) (dnp no)
@@
     )
   )
+  (symbol (lib_id "Device:C_Small") (at 27.94 82.55 90) (unit 1)
+    (in_bom yes) (on_board yes) (dnp no)
+    (property "Reference" "C17a1" (at 27.94 78.74 90)
+      (effects (font (size 1.27 1.27)))
+    )
+    (property "Value" "6.8pF" (at 22.86 80.01 90)
+      (effects (font (size 1.27 1.27)))
+    )
+    (property "Footprint" "Capacitor_SMD:C_1206_3216Metric_Pad1.33x1.80mm_HandSolder" (at 27.94 82.55 0)
+      (effects (font (size 1.27 1.27)) hide)
+    )
+    (property "Datasheet" "" (at 27.94 82.55 0)
+      (effects (font (size 1.27 1.27)) hide)
+    )
+    (property "LCSC" "" (at 27.94 82.55 0)
+      (effects (font (size 1.27 1.27)) hide)
+    )
+    (property "LINK" "" (at 27.94 82.55 0)
+      (effects (font (size 1.27 1.27)) hide)
+    )
+    (pin "1")
+    (pin "2")
+    (instances
+      (project "qca7000"
+        (path "/e63e39d7-6ac0-4ffd-8aa3-1841a4541b55"
+          (reference "C17a1") (unit 1)
+        )
+      )
+    )
+  )
   (symbol (lib_id "power:GND") (at 81.28 66.04 90) (unit 1)
     (in_bom yes) (on_board yes) (dnp no)
@@
   (symbol (lib_id "Device:L") (at 154.94 129.54 90) (unit 1)
     (in_bom yes) (on_board yes) (dnp no)
-    (property "Reference" "L11" (at 154.94 127 90)
+    (property "Reference" "L11" (at 153.67 130.81 90)
       (effects (font (size 1.27 1.27)))
     )
-    (property "Value" "4.7uH" (at 154.94 130.81 90)
+    (property "Value" "4.7uH" (at 158.75 130.81 90)
       (effects (font (size 1.27 1.27)))
     )

Commit message: BOM consolidation: XTAL options and back to 8MHz. Replace internal connectors by testpoints. Use T with integrated R for CP switching. Fix: Footprint Q7-Q9 corrected.
Parts:
- removed J1: Conn_01x04_Pin, Connector_PinHeader_2.54mm:PinHeader_1x04_P2.54mm_Vertical, symbol Connector:Conn_01x04_Pin
- removed J2: Conn_01x08_Pin, Connector_PinHeader_2.54mm:PinHeader_1x08_P2.54mm_Vertical, symbol Connector:Conn_01x08_Pin
- added 3V3, CLK1, CS1, GND1, INT1, MISO1, MOSI1, RES1: ~, speciallib:TestPoint_Special_THTPad_D1.9mm_Drill1mm, symbol Connector:TestPoint
- added RX_N1, RX_P1, TX_N1, TX_P1: ~, TestPoint:TestPoint_THTPad_D1.0mm_Drill0.5mm, symbol Connector:TestPoint
Connections:
- net 3V3_D: now also 3V3.1
- net GND: now also GND1.1
- net RESET#: now also RES1.1
- net RX_N: now also RX_N1.1
- net RX_P: now also RX_P1.1
- net SERIAL_IO_0_INT: now also INT1.1
- net SERIAL_IO_1_CLK: now also CLK1.1
- net SERIAL_IO_2_CS: now also CS1.1
- net SERIAL_IO_3_MISO: now also MISO1.1
- net SERIAL_IO_4_MOSI: now also MOSI1.1
- net TX_N: now also TX_N1.1
- net TX_P: now also TX_P1.1

Commit message: added rotation attribute to get the correct footprint rotation at JLCPCB
Parts:
- U1: JLCPCB Rotation Offset (none) -> -90
Changed lines of the file:
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@@
+      (effects (font (size 1.27 1.27)) hide)
+    )
+    (property "JLCPCB Rotation Offset" "-90" (at 243.84 146.05 0)
       (effects (font (size 1.27 1.27)) hide)
     )

Commit message: fix rx shortcut. add transformer. correct part number of NCV. Correct footprints of U1 and L11. add mounting holes. stepdown layout improved. added TVS at 12V
Parts:
- removed RX_N1, RX_P1, TX_N1, TX_P1: ~, TestPoint:TestPoint_THTPad_D1.0mm_Drill0.5mm, symbol Connector:TestPoint
- added C32, C33: 1.5nF, Capacitor_SMD:C_0805_2012Metric_Pad1.18x1.45mm_HandSolder, symbol Device:C_Small
- added T1: ~, transformerCL4532A-201:transformerCL4532A-201, symbol transformerCL4532A-201:transformer
- L11: footprint Inductor_SMD:L_1812_4532Metric_Pad1.30x3.40mm_HandSolder -> Inductor_SMD:L_1206_3216Metric_Pad1.22x1.90mm_HandSolder
- U1: footprint Package_SO:SOP-8_5.28x5.23mm_P1.27mm -> Package_SO:SOIC-8_3.9x4.9mm_P1.27mm
Connections:
- net GND: now also T1.2
- net RXIN_N: now also C32.1; no longer C3.1, D2.3 (K), L1.2, L5.1
- net RXIN_P: now also C33.1; no longer C7.2, D1.3 (K), L7.2, L8.2
- net RX_N: now also T1.7
- net RX_P: now also T1.8
- net TX_N: now also T1.5
- net TX_P: now also T1.6
- new net: C3.1, C32.2, D2.3 (K), L1.2, L5.1
- new net: C33.2, C7.2, D1.3 (K), L7.2, L8.2
- new net MODEM_RF: T1.1
- no-connect marks 9 -> 11
Other:
- note added: "The RF transformer. The polarity of the windings does not matter in this application. Goal is to have a conversion between unsymmetrical (on CP line) and symmetrical (on QCA side) signals, in a freq range of 2 to 30 MHz."
- moved on the sheet: L3

Commit message: fix: origin of the transformer into the middle. Fix: rotation attributes for jlcpcb
Parts:
- D1, D2: JLCPCB Rotation Offset (none) -> 180
Changed lines of the file:
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@@
+      (effects (font (size 1.27 1.27)) hide)
+    )
+    (property "JLCPCB Rotation Offset" "180" (at 80.01 30.48 90)
       (effects (font (size 1.27 1.27)) hide)
     )
@@
       (effects (font (size 1.27 1.27)) hide)
     )
+    (property "JLCPCB Rotation Offset" "180" (at 90.17 30.48 90)
+      (effects (font (size 1.27 1.27)) hide)
+    )

Commit message: Redesigned wakeup circuit
Parts:
- R59: LCSC C17630 -> C23138
Changed lines of the file:
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@@
       (effects (font (size 1.27 1.27)) hide)
     )
-    (property "LCSC" "C17630" (at 72.39 167.64 0)
+    (property "LCSC" "C23138" (at 72.39 167.64 0)
       (effects (font (size 1.27 1.27)) hide)
     )
