File: pcb/qca7000.kicad_sch (KiCad schematic)
At the start: 95 parts, among them U1 25Q16, Y1 25MHz

Commit message: BOM optimization
Parts:
- R6: LCSC C17767 -> C4260
- renumbered D8 to U7
Changed lines of the file:
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@@
   (symbol (lib_id "QualcommAtheros:QCA 7000") (at 109.22 130.81 180) (unit 1)
     (in_bom yes) (on_board yes) (dnp no)
-    (property "Reference" "D8" (at 107.95 130.81 0)
+    (property "Reference" "U7" (at 107.95 130.81 0)
       (effects (font (size 1.27 1.27)))
     )
@@
       (project "qca7000"
         (path "/e63e39d7-6ac0-4ffd-8aa3-1841a4541b55"
-          (reference "D8") (unit 1)
+          (reference "U7") (unit 1)
         )
       )
@@
       (effects (font (size 1.27 1.27)) hide)
     )
-    (property "LCSC" "C17767" (at 34.29 123.19 0)
+    (property "LCSC" "C4260" (at 34.29 123.19 0)
       (effects (font (size 1.27 1.27)) hide)
     )

Commit message: Re-assigned pins to be able to make one loom to the charge port and one to the car
Parts:
- U7: LCSC (none) -> C9900078626

Commit message: Forgot to save
Parts:
- removed TP2: FL_MOSI, speciallib:TestPoint_Special_THTPad_D1.9mm_Drill1mm, symbol Connector:TestPoint
- removed TP3: FL_CLK, speciallib:TestPoint_Special_THTPad_D1.9mm_Drill1mm, symbol Connector:TestPoint
- removed TP39: FL_GND, speciallib:TestPoint_Special_THTPad_D1.9mm_Drill1mm, symbol Connector:TestPoint
- removed TP4: FL_CS, speciallib:TestPoint_Special_THTPad_D1.9mm_Drill1mm, symbol Connector:TestPoint
- removed TP40: FL_RES, speciallib:TestPoint_Special_THTPad_D1.9mm_Drill1mm, symbol Connector:TestPoint
- removed TP5: FL_MISO, speciallib:TestPoint_Special_THTPad_D1.9mm_Drill1mm, symbol Connector:TestPoint
- added J1: Conn_01x06, Connector_PinHeader_2.54mm:PinHeader_1x06_P2.54mm_Vertical, symbol Connector_Generic:Conn_01x06
Connections:
- net GND: now also J1.5 (Pin_5)
- net RESET#: now also J1.6 (Pin_6)
- net SPI_CLK: now also J1.4 (Pin_4)
- net SPI_CS_L: now also J1.2 (Pin_2)
- net SPI_DI: now also J1.1 (Pin_1)
- net SPI_DO: now also J1.3 (Pin_3)

Commit message: More re-assignment
Connections:
- net GND: now also J1.6 (Pin_6); no longer J1.5 (Pin_5)
- net RESET#: now also J1.5 (Pin_5); no longer J1.6 (Pin_6)
Changed lines of the file:
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@@
 	)
 	(junction
-		(at 185.42 162.56)
-		(diameter 0)
-		(color 0 0 0 0)
-	)
-	(junction
 		(at 149.86 129.54)
 		(diameter 0)
@@
 	)
 	(junction
-		(at 243.84 158.75)
+		(at 69.85 176.53)
 		(diameter 0)
 		(color 0 0 0 0)
 	)
 	(junction
-		(at 69.85 176.53)
+		(at 69.85 19.05)
 		(diameter 0)
 		(color 0 0 0 0)
 	)
 	(junction
-		(at 69.85 19.05)
+		(at 243.84 129.54)
 		(diameter 0)
 		(color 0 0 0 0)
 	)
 	(junction
-		(at 243.84 129.54)
+		(at 243.84 158.75)
 		(diameter 0)
 		(color 0 0 0 0)
@@
 	)
 	(junction
+		(at 185.42 160.02)
+		(diameter 0)
+		(color 0 0 0 0)
+	)
+	(junction
 		(at 212.09 143.51)
 		(diameter 0)
@@
 	(wire
 		(pts
-			(xy 217.17 167.64) (xy 185.42 167.64)
+			(xy 148.59 125.73) (xy 144.78 125.73)
 		)
 		(stroke
@@
 	(wire
 		(pts
-			(xy 148.59 125.73) (xy 144.78 125.73)
+			(xy 34.29 106.68) (xy 34.29 109.22)
 		)
 		(stroke
@@
 	(wire
 		(pts
-			(xy 34.29 106.68) (xy 34.29 109.22)
+			(xy 173.99 87.63) (xy 173.99 91.44)
 		)
 		(stroke
@@
 	(wire
 		(pts
-			(xy 173.99 87.63) (xy 173.99 91.44)
+			(xy 217.17 162.56) (xy 240.03 162.56)
 		)
 		(stroke
@@
 	(wire
 		(pts
+			(xy 219.71 160.02) (xy 185.42 160.02)
+		)
+		(stroke
+			(width 0)
+			(type default)
+		)
+	)
+	(wire
+		(pts
 			(xy 95.25 19.05) (xy 96.52 19.05)
 		)
@@
 	(wire
 		(pts
-			(xy 185.42 162.56) (xy 185.42 157.48)
+			(xy 185.42 162.56) (xy 185.42 160.02)
 		)
 		(stroke
@@
 	(wire
 		(pts
-			(xy 219.71 158.75) (xy 243.84 158.75)
-		)
-		(stroke
-			(width 0)
-			(type default)
-		)
-	)
-	(wire
-		(pts
 			(xy 64.77 95.25) (xy 92.71 95.25)
 		)
@@
 	(wire
 		(pts
-			(xy 219.71 167.64) (xy 219.71 158.75)
-		)
-		(stroke
-			(width 0)
-			(type default)
-		)
-	)
-	(wire
-		(pts
 			(xy 243.84 129.54) (xy 248.92 129.54)
 		)
@@
 	(wire
 		(pts
+			(xy 185.42 160.02) (xy 185.42 157.48)
+		)
+		(stroke
+			(width 0)
+			(type default)
+		)
+	)
+	(wire
+		(pts
 			(xy 39.37 116.84) (xy 39.37 120.65)
 		)
@@
 	(wire
 		(pts
+			(xy 217.17 167.64) (xy 217.17 162.56)
+		)
+		(stroke
+			(width 0)
+			(type default)
+		)
+	)
+	(wire
+		(pts
 			(xy 144.78 167.64) (xy 149.86 167.64)
 		)
@@
 	(wire
 		(pts
-			(xy 90.17 39.37) (xy 90.17 38.1)
+			(xy 240.03 162.56) (xy 240.03 158.75)
 		)
 		(stroke
@@
 	(wire
 		(pts
-			(xy 186.69 101.6) (xy 186.69 99.06)
+			(xy 90.17 39.37) (xy 90.17 38.1)
 		)
 		(stroke
@@
 	(wire
 		(pts
-			(xy 25.4 111.76) (xy 22.86 111.76)
+			(xy 186.69 101.6) (xy 186.69 99.06)
 		)
 		(stroke
@@
 	(wire
 		(pts
-			(xy 123.19 165.1) (xy 123.19 162.56)
+			(xy 25.4 111.76) (xy 22.86 111.76)
 		)
 		(stroke
@@
 	(wire
 		(pts
-			(xy 34.29 90.17) (xy 43.18 90.17)
+			(xy 123.19 165.1) (xy 123.19 162.56)
 		)
 		(stroke
@@
 	(wire
 		(pts
-			(xy 185.42 167.64) (xy 185.42 162.56)
+			(xy 34.29 90.17) (xy 43.18 90.17)
 		)
 		(stroke
@@
 	(wire
 		(pts
+			(xy 219.71 167.64) (xy 219.71 160.02)
+		)
+		(stroke
+			(width 0)
+			(type default)
+		)
+	)
+	(wire
+		(pts
 			(xy 62.23 22.86) (xy 62.23 19.05)
 		)
@@
 		)
 		(stroke
+			(width 0)
+			(type default)
+		)
+	)
+	(wire
+		(pts
+			(xy 240.03 158.75) (xy 243.84 158.75)
+		)
+		(stroke

Commit message: added diode D8, corrected resistors, corrected rotations. V5.1
Parts:
- removed C17a1, C29a1: 6.8pF, Capacitor_SMD:C_1206_3216Metric_Pad1.33x1.80mm_HandSolder, symbol Device:C_Small

Commit message: 5.2pre: transformerless RF path. TVS. Demo placement for alternative connectors.
Parts:
- removed C12: 100nF, Capacitor_SMD:C_0805_2012Metric_Pad1.18x1.45mm_HandSolder, symbol Device:C_Small
- removed C6, C7: 220pF, Capacitor_SMD:C_0805_2012Metric_Pad1.18x1.45mm_HandSolder, symbol Device:C_Small
- removed C8: 1.5nF, Capacitor_SMD:C_0805_2012Metric_Pad1.18x1.45mm_HandSolder, symbol Device:C_Small
- removed D1: BAV99, Package_TO_SOT_SMD:SOT-23, symbol Diode:BAV99
- removed D6, D7: B5819W, Diode_SMD:D_SOD-123, symbol Diode:1N5819
- removed L6, L7: 1.8uH, Inductor_SMD:L_0603_1608Metric_Pad1.05x0.95mm_HandSolder, symbol Device:L
- removed L8: 270nH, Inductor_SMD:L_0805_2012Metric_Pad1.05x1.20mm_HandSolder, symbol Device:L
- removed R2: 22, Resistor_SMD:R_0805_2012Metric_Pad1.20x1.40mm_HandSolder, symbol Device:R_Small
- removed R44: 100, Resistor_SMD:R_0805_2012Metric_Pad1.20x1.40mm_HandSolder, symbol Device:R_Small
- removed T1: ~, transformerCL4532A-201:transformerCL4532A-201, symbol transformerCL4532A-201:transformer
- added C76: 1nF, Capacitor_SMD:C_0805_2012Metric_Pad1.18x1.45mm_HandSolder, symbol Device:C_Small
- added R25: 100, Resistor_SMD:R_0805_2012Metric_Pad1.20x1.40mm_HandSolder, symbol Device:R_Small
- added TP2: TXOUTP, TestPoint:TestPoint_Pad_D1.0mm, symbol Connector:TestPoint
- added U9: DESD3V3S1BL-7B, X1-DFN1006-2_RH_DIO, symbol DESD3V3S1BL_7B:DESD3V3S1BL-7B
Connections:
- net TX_N is gone; now on net RF_protected: R8.2
- net GND: now also C10.2, C33.2, U9.2
- net RX_N renamed RF_protected
- net RF_protected: now also R25.1, U9.1
- net TXOUT_P: no longer names the net of U7.33 (TXOUT_P)
- net TXOUT_P: now also TP2.1
- new net: C76.2, R25.2
- new net CP: C76.1
- no-connect marks 11 -> 10
Other:
- note added: "1N5819HW 2pcs"
- note added: "With 3.3V TVS and input divider R25 we allow >12Vpp on CP line without saturation."
- note removed: "1N5819HW 4pcs"
- note removed: "The RF transformer. The polarity of the windings does not matter in this application. Goal is to have a conversion between unsymmetrical (on CP line) and symmetrical (on QCA side) signals, in a freq range of 2 to 30 MHz."
- note removed: "alternative footprints for C17, C29"
- moved on the sheet: C10, C11, C13, C16, C17, C19, C2, C22, C24, C26, C28, C29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

Commit message: corrected some rotations for JLC. Version 5.2p7
Parts:
- D2: JLCPCB Rotation Offset 180 -> 0
- U1: JLCPCB Rotation Offset -90 -> 0
Changed lines of the file:
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@@
 			)
 		)
-		(property "JLCPCB Rotation Offset" "-90"
+		(property "JLCPCB Rotation Offset" "0"
 			(at 245.11 158.75 0)
 			(effects
@@
 			)
 		)
-		(property "JLCPCB Rotation Offset" "180"
+		(property "JLCPCB Rotation Offset" "0"
 			(at 90.17 30.48 90)
 			(effects

Commit message: Changed RF dampening resistors from 100 to 22 Ohms
Parts:
- R25, R8: value 100 -> 22; LCSC C17408 -> C17561
Changed lines of the file:
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@@
 (kicad_sch
-	(version 20231120)
+	(version 20250114)
 	(generator "eeschema")
-	(generator_version "8.0")
+	(generator_version "9.0")
 	(paper "A3")
 	(title_block
@@
 		(comment 2 "Reused by uhi22 (https://github.com/uhi22/foccci)")
 	)
+	(text "2k5"
+		(exclude_from_sim no)
+		(at 73.66 167.64 0)
+		(effects
+			(font
+				(size 1.27 1.27)
+			)
+			(justify left bottom)
+		)
+	)
+	(text "With 3.3V TVS and input divider R25 we\nallow >12Vpp on CP line without\nsaturation."
+		(exclude_from_sim no)
+		(at 15.494 57.658 0)
+		(effects
+			(font
+				(size 1.27 1.27)
+			)
+			(justify left bottom)
+		)
+	)
+	(text "1N5819HW 2pcs\n"
+		(exclude_from_sim no)
+		(at 55.118 70.612 0)
+		(effects
+			(font
+				(size 1.27 1.27)
+			)
+			(justify left bottom)
+		)
+	)
+	(text "Atmel AT26DF161-SU 100 MHz 16-Mbits Not for new designs \nAtmel  	    AT26DF161A-SU  	70 MHz  16-Mbits\nNumonyx   	M25P80-VMW6TP   75 MHz  8-Mbits\nNumonyx 	M25P16-VMW6TP 	75MHz 16-Mbits\nMacronix  	MX25L8005  	    70 MHz  8-Mbits\nMacronix  	MX25L1605  	    86 MHz  16-Mbits\n"
+		(exclude_from_sim no)
+		(at 218.44 137.16 0)
+		(effects
+			(font
+				(size 1.27 1.27)
+			)
+			(justify left bottom)
+		)
+	)
+	(text "GPIO_2 selects burst mode (3V3)"
+		(exclude_from_sim no)
+		(at 215.9 76.2 0)
+		(effects
+			(font
+				(size 1.27 1.27)
+			)
+			(justify left bottom)
+		)
+	)
+	(text "ARM926"
+		(exclude_from_sim no)
+		(at 106.68 148.59 0)
+		(effects
+			(font
+				(size 1.27 1.27)
+			)
+			(justify left bottom)
+		)
+	)
+	(text "3rd Order Butterworth Bandpass\nLower Cutoff Freq. = 1.900 MHz; Upper Cutoff Freq. = 31.00 MHz\nhttps://rf-tools.com/lc-filter/"
+		(exclude_from_sim no)
+		(at 18.542 40.64 0)
+		(effects
+			(font
+				(size 1.27 1.27)
+			)
+			(justify left bottom)
+		)
+	)
+	(text "M25P16"
+		(exclude_from_sim no)
+		(at 238.76 121.92 0)
+		(effects
+			(font
+				(size 1.27 1.27)
+			)
+			(justify left bottom)
+		)
+	)
+	(text "GPIO_1 must be pulled down."
+		(exclude_from_sim no)
+		(at 218.44 60.96 0)
+		(effects
+			(font
+				(size 1.27 1.27)
+			)
+			(justify left bottom)
+		)
+	)
+	(text "25q16"
+		(exclude_from_sim no)
+		(at 250.19 121.92 0)
+		(effects
+			(font
+				(size 1.27 1.27)
+			)
+			(justify left bottom)
+		)
+	)
 	(junction
 		(at 148.59 175.26)
@@
 		)
 	)
-	(text "2k5"
-		(exclude_from_sim no)
-		(at 73.66 167.64 0)
-		(effects
-			(font
-				(size 1.27 1.27)
-			)
-			(justify left bottom)
-		)
-	)
-	(text "With 3.3V TVS and input divider R25 we\nallow >12Vpp on CP line without\nsaturation."
-		(exclude_from_sim no)
-		(at 15.494 57.658 0)
-		(effects
-			(font
-				(size 1.27 1.27)
-			)
-			(justify left bottom)
-		)
-	)
-	(text "1N5819HW 2pcs\n"
-		(exclude_from_sim no)
-		(at 55.118 70.612 0)
-		(effects
-			(font
-				(size 1.27 1.27)
-			)
-			(justify left bottom)
-		)
-	)
-	(text "Atmel AT26DF161-SU 100 MHz 16-Mbits Not for new designs \nAtmel  	    AT26DF161A-SU  	70 MHz  16-Mbits\nNumonyx   	M25P80-VMW6TP   75 MHz  8-Mbits\nNumonyx 	M25P16-VMW6TP 	75MHz 16-Mbits\nMacronix  	MX25L8005  	    70 MHz  8-Mbits\nMacronix  	MX25L1605  	    86 MHz  16-Mbits\n"
-		(exclude_from_sim no)
-		(at 218.44 137.16 0)
-		(effects
-			(font
-				(size 1.27 1.27)
-			)
-			(justify left bottom)
-		)
-	)
-	(text "GPIO_2 selects burst mode (3V3)"
-		(exclude_from_sim no)
-		(at 215.9 76.2 0)
-		(effects
-			(font
-				(size 1.27 1.27)
-			)
-			(justify left bottom)
-		)
-	)
-	(text "ARM926"
-		(exclude_from_sim no)
-		(at 106.68 148.59 0)
-		(effects
-			(font
-				(size 1.27 1.27)
-			)
-			(justify left bottom)
-		)
-	)
-	(text "3rd Order Butterworth Bandpass\nLower Cutoff Freq. = 1.900 MHz; Upper Cutoff Freq. = 31.00 MHz\nhttps://rf-tools.com/lc-filter/"
-		(exclude_from_sim no)
-		(at 18.542 40.64 0)
-		(effects
-			(font
-				(size 1.27 1.27)
-			)
-			(justify left bottom)
-		)
-	)
-	(text "M25P16"
-		(exclude_from_sim no)
-		(at 238.76 121.92 0)
-		(effects
-			(font
-				(size 1.27 1.27)
-			)
-			(justify left bottom)
-		)
-	)
-	(text "GPIO_1 must be pulled down."
-		(exclude_from_sim no)
-		(at 218.44 60.96 0)
-		(effects
-			(font
-				(size 1.27 1.27)
-			)
-			(justify left bottom)
-		)
-	)
-	(text "25q16"
-		(exclude_from_sim no)
-		(at 250.19 121.92 0)
-		(effects
-			(font
-				(size 1.27 1.27)
-			)
-			(justify left bottom)
-		)
-	)
 	(label "SW_VDD_OUT"
 		(at 149.86 140.97 0)
-		(fields_autoplaced yes)
 		(effects
 			(font
@@
 	(label "RSVD05"
 		(at 81.28 187.96 0)
-		(fields_autoplaced yes)
 		(effects
 			(font
@@
 	(label "RBIAS"
 		(at 73.66 163.83 0)
-		(fields_autoplaced yes)
 		(effects
 			(font
@@
 			)
 		)
-		(property "Value" "100"
+		(property "Value" "22"
 			(at 33.274 47.752 90)
 			(effects
@@
 			)
 		)
-		(property "LCSC" "C17408"
+		(property "LCSC" "C17561"
 			(at 33.02 45.72 0)
 			(effects
@@
 			)
 		)
-		(property "Value" "100"
+		(property "Value" "22"
 			(at 36.83 69.85 90)
 			(effects
@@
 			)
 		)
-		(property "LCSC" "C17408"
+		(property "LCSC" "C17561"
 			(at 36.83 72.39 0)
 			(effects
@@
 		(at 323.85 229.87)
 		(size 27.94 20.32)
+		(exclude_from_sim no)
+		(in_bom yes)
+		(on_board yes)
+		(dnp no)
 		(fields_autoplaced yes)
 		(stroke
@@
 		(at 270.51 198.12)
 		(size 49.53 20.32)
+		(exclude_from_sim no)
+		(in_bom yes)
+		(on_board yes)
+		(dnp no)
 		(fields_autoplaced yes)
 		(stroke
@@
 		(at 220.98 198.12)
 		(size 39.37 20.32)
+		(exclude_from_sim no)
+		(in_bom yes)
+		(on_board yes)
+		(dnp no)
 		(fields_autoplaced yes)
 		(stroke
@@
 		(at 220.98 229.87)
 		(size 40.64 21.59)
+		(exclude_from_sim no)
+		(in_bom yes)
+		(on_board yes)
+		(dnp no)
 		(fields_autoplaced yes)
 		(stroke
@@
 		(at 270.51 229.87)
 		(size 49.53 20.32)
+		(exclude_from_sim no)
+		(in_bom yes)
+		(on_board yes)
+		(dnp no)
 		(fields_autoplaced yes)
 		(stroke
@@
 		(at 323.85 198.12)
 		(size 27.94 20.32)
+		(exclude_from_sim no)
+		(in_bom yes)
+		(on_board yes)
+		(dnp no)
 		(fields_autoplaced yes)
 		(stroke
@@
 		)
 	)
+	(embedded_fonts no)
 )
