File: pcb/Inputs.kicad_sch (KiCad schematic)
At the start: 10 parts, among them J9 Temps

Commit message: fix: divider on the stepdown. fix: non-inverted contactor drivers. fix: part number of 8MHz. add: mounting holes and spare grid. add: LIM HVDC input. docu: todo list
Parts:
- added C61 (x2): 100nF, Capacitor_SMD:C_1206_3216Metric_Pad1.33x1.80mm_HandSolder, symbol Device:C_Small
- added J17: IN_U_HV, Connector_PinHeader_2.54mm:PinHeader_1x01_P2.54mm_Vertical, symbol Connector:Conn_01x01_Pin
- added R3: 22k, Resistor_SMD:R_1206_3216Metric_Pad1.30x1.75mm_HandSolder, symbol Device:R_Small
- added R3 (x2): 240, Resistor_SMD:R_1206_3216Metric_Pad1.30x1.75mm_HandSolder, symbol Device:R_Small
- added R3: 47k, Resistor_SMD:R_1206_3216Metric_Pad1.30x1.75mm_HandSolder, symbol Device:R_Small
Connections:
- net GND: now also C61.1, C61.1, R3.1, R3.1
- new net: R3.1, R3.2
- new net: C61.2, J17.1 (Pin_1), R3.2, R3.2
- new net ADC_U_HVDC: C61.2, R3.1, R3.2
Other:
- note added: "Analog inputs, e.g. for use with NTCs to ground for temperature measurement or analog feedback contacts or switches."
- note added: "Current input for HV DC voltage measurement as done in LIM, see https://openinverter.org/forum/viewtopic.php?p=58839#p58839"

Commit message: added TE DEUTSCH connector and housing
Parts:
- removed J17: IN_U_HV, Connector_PinHeader_2.54mm:PinHeader_1x01_P2.54mm_Vertical, symbol Connector:Conn_01x01_Pin
- removed J9: Temps, Connector_PinHeader_2.54mm:PinHeader_1x04_P2.54mm_Vertical, symbol Connector:Conn_01x04_Pin
- C61: value 100nF -> 1nF
Connections:
- net IN_U_HV: now reaches C61.2, R3.2, R3.2
- net TEMP3: now reaches R11.1, R11.2
- net TEMP2: now reaches R11.1, R11.2
- net TEMP1: now reaches R11.1, R11.2
Changed lines of the file:
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@@
     (stroke (width 0) (type default))
   )
-  (wire (pts (xy 43.18 39.37) (xy 43.18 31.75))
+  (wire (pts (xy 52.07 53.34) (xy 68.58 53.34))
     (stroke (width 0) (type default))
   )
@@
     (stroke (width 0) (type default))
   )
-  (wire (pts (xy 43.18 41.91) (xy 55.88 41.91))
-    (stroke (width 0) (type default))
-  )
-  (wire (pts (xy 43.18 31.75) (xy 68.58 31.75))
+  (wire (pts (xy 50.8 31.75) (xy 68.58 31.75))
     (stroke (width 0) (type default))
   )
@@
     (stroke (width 0) (type default))
   )
-  (wire (pts (xy 55.88 53.34) (xy 68.58 53.34))
-    (stroke (width 0) (type default))
-  )
   (wire (pts (xy 68.58 62.23) (xy 68.58 64.77))
     (stroke (width 0) (type default))
   )
-  (wire (pts (xy 43.18 44.45) (xy 52.07 44.45))
-    (stroke (width 0) (type default))
-  )
   (wire (pts (xy 66.04 44.45) (xy 68.58 44.45))
     (stroke (width 0) (type default))
@@
   )
   (wire (pts (xy 68.58 24.13) (xy 66.04 24.13))
-    (stroke (width 0) (type default))
-  )
-  (wire (pts (xy 52.07 44.45) (xy 52.07 72.39))
-    (stroke (width 0) (type default))
-  )
-  (wire (pts (xy 55.88 41.91) (xy 55.88 53.34))
     (stroke (width 0) (type default))
   )
@@
     )
   )
+  (global_label "IN_U_HV" (shape input) (at 66.04 128.27 180) (fields_autoplaced)
+    (effects (font (size 1.27 1.27)) (justify right))
+    (property "Intersheetrefs" "${INTERSHEET_REFS}" (at 55.5141 128.27 0)
+      (effects (font (size 1.27 1.27)) (justify right) hide)
+    )
+  )
+  (global_label "TEMP3" (shape input) (at 52.07 72.39 180) (fields_autoplaced)
+    (effects (font (size 1.27 1.27)) (justify right))
+    (property "Intersheetrefs" "${INTERSHEET_REFS}" (at 43.1167 72.39 0)
+      (effects (font (size 1.27 1.27)) (justify right) hide)
+    )
+  )
+  (global_label "TEMP2" (shape input) (at 52.07 53.34 180) (fields_autoplaced)
+    (effects (font (size 1.27 1.27)) (justify right))
+    (property "Intersheetrefs" "${INTERSHEET_REFS}" (at 43.1167 53.34 0)
+      (effects (font (size 1.27 1.27)) (justify right) hide)
+    )
+  )
+  (global_label "TEMP1" (shape input) (at 50.8 31.75 180) (fields_autoplaced)
+    (effects (font (size 1.27 1.27)) (justify right))
+    (property "Intersheetrefs" "${INTERSHEET_REFS}" (at 41.8467 31.75 0)
+      (effects (font (size 1.27 1.27)) (justify right) hide)
+    )
+  )
   (global_label "3V3_uC" (shape input) (at 66.04 24.13 180) (fields_autoplaced)
     (effects (font (size 1.27 1.27)) (justify right))
@@
     )
   )
-  (symbol (lib_id "power:GND") (at 43.18 46.99 0) (unit 1)
-    (in_bom yes) (on_board yes) (dnp no)
-    (property "Reference" "#PWR048" (at 43.18 53.34 0)
-      (effects (font (size 1.27 1.27)) hide)
-    )
-    (property "Value" "GND" (at 45.72 50.8 0)
-      (effects (font (size 1.27 1.27)) (justify right))
-    )
-    (property "Footprint" "" (at 43.18 46.99 0)
-      (effects (font (size 1.27 1.27)) hide)
-    )
-    (property "Datasheet" "" (at 43.18 46.99 0)
-      (effects (font (size 1.27 1.27)) hide)
-    )
-    (pin "1")
-    (instances
-      (project "qca7000"
-        (path "/e63e39d7-6ac0-4ffd-8aa3-1841a4541b55"
-          (reference "#PWR048") (unit 1)
-        )
-        (path "/e63e39d7-6ac0-4ffd-8aa3-1841a4541b55/5666e7cf-6b6c-4583-8335-aa3be69ccd45"
-          (reference "#PWR056") (unit 1)
-        )
-        (path "/e63e39d7-6ac0-4ffd-8aa3-1841a4541b55/93c6207c-4203-4bc7-a590-e5e89c0d3d27"
-          (reference "#PWR083") (unit 1)
-        )
-      )
-    )
-  )
   (symbol (lib_id "Device:R_Small") (at 80.01 130.81 180) (unit 1)
     (in_bom yes) (on_board yes) (dnp no)
@@
         (path "/e63e39d7-6ac0-4ffd-8aa3-1841a4541b55/93c6207c-4203-4bc7-a590-e5e89c0d3d27"
           (reference "R36") (unit 1)
-        )
-      )
-    )
-  )
-  (symbol (lib_id "Connector:Conn_01x01_Pin") (at 60.96 128.27 0) (unit 1)
-    (in_bom yes) (on_board yes) (dnp no)
-    (property "Reference" "J17" (at 58.42 124.46 0)
-      (effects (font (size 1.27 1.27)))
-    )
-    (property "Value" "IN_U_HV" (at 57.15 127 0)
-      (effects (font (size 1.27 1.27)))
-    )
-    (property "Footprint" "Connector_PinHeader_2.54mm:PinHeader_1x01_P2.54mm_Vertical" (at 60.96 128.27 0)
-      (effects (font (size 1.27 1.27)) hide)
-    )
-    (property "Datasheet" "~" (at 60.96 128.27 0)
-      (effects (font (size 1.27 1.27)) hide)
-    )
-    (pin "1")
-    (instances
-      (project "qca7000"
-        (path "/e63e39d7-6ac0-4ffd-8aa3-1841a4541b55/5666e7cf-6b6c-4583-8335-aa3be69ccd45"
-          (reference "J17") (unit 1)
-        )
-        (path "/e63e39d7-6ac0-4ffd-8aa3-1841a4541b55/93c6207c-4203-4bc7-a590-e5e89c0d3d27"
-          (reference "J19") (unit 1)
         )
       )
@@
       (effects (font (size 1.27 1.27)))
     )
-    (property "Value" "100nF" (at 74.93 134.62 0)
+    (property "Value" "1nF" (at 74.93 134.62 0)
       (effects (font (size 1.27 1.27)))
     )
@@
         )
       )
-    )
-  )
-  (symbol (lib_id "Connector:Conn_01x04_Pin") (at 38.1 41.91 0) (unit 1)
-    (in_bom yes) (on_board yes) (dnp no)
-    (property "Reference" "J9" (at 33.02 41.91 0)
-      (effects (font (size 1.27 1.27)))
-    )
-    (property "Value" "Temps" (at 33.02 44.45 0)
-      (effects (font (size 1.27 1.27)))
-    )
-    (property "Footprint" "Connector_PinHeader_2.54mm:PinHeader_1x04_P2.54mm_Vertical" (at 38.1 41.91 0)
-      (effects (font (size 1.27 1.27)) hide)
-    )
-    (property "Datasheet" "~" (at 38.1 41.91 0)
-      (effects (font (size 1.27 1.27)) hide)
-    )
-    (pin "1")
-    (pin "2")
-    (pin "3")
-    (pin "4")
-    (instances
-      (project "qca7000"
-        (path "/e63e39d7-6ac0-4ffd-8aa3-1841a4541b55/93c6207c-4203-4bc7-a590-e5e89c0d3d27"
-          (reference "J9") (unit 1)
-        )
-      )

Commit message: changed to 4 layers. Added button, PP and lock feedback. New testpoints to avoid courtyard warnings.
Parts:
- added C61 (x3): 100nF, Capacitor_SMD:C_0805_2012Metric_Pad1.18x1.45mm_HandSolder, symbol Device:C_Small
- added R11 (x3): 47k, Resistor_SMD:R_1206_3216Metric_Pad1.30x1.75mm_HandSolder, symbol Device:R_Small
- added R11: 1k, Resistor_SMD:R_1206_3216Metric_Pad1.30x1.75mm_HandSolder, symbol Device:R_Small
- added R11 (x2): 10k, Resistor_SMD:R_1206_3216Metric_Pad1.30x1.75mm_HandSolder, symbol Device:R_Small
Connections:
- net 3V3_uC: now also R11.1, R11.1, R11.1
- net GND: now also C61.1, C61.1, C61.1
- new net ADC_BUTTON: C61.2, R11.2
- new net ADC_CONN_LOCK_FEEDBACK: C61.2, R11.2
- new net ADC_PP: C61.2, R11.2
- new net BUTTON: R11.1, R11.2
- new net CONN_LOCK_FEEDBACK: R11.1, R11.2
- new net PP: R11.1, R11.2
Other:
- note added: "PlugPresent: - 1k5 to ground for CCS2 - 100 ohm to 1k5 for AC (current limit of the cable) - 150 ohm (button idle) or 480 ohm (button pressed) for CCS1"

Commit message: all 100nF now 0805. Todo list cleaned up.
Parts:
- C61: footprint Capacitor_SMD:C_1206_3216Metric_Pad1.33x1.80mm_HandSolder -> Capacitor_SMD:C_0805_2012Metric_Pad1.18x1.45mm_HandSolder
Changed lines of the file:
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@@
       (effects (font (size 1.27 1.27)))
     )
-    (property "Footprint" "Capacitor_SMD:C_1206_3216Metric_Pad1.33x1.80mm_HandSolder" (at 78.74 55.88 0)
+    (property "Footprint" "Capacitor_SMD:C_0805_2012Metric_Pad1.18x1.45mm_HandSolder" (at 78.74 55.88 0)
       (effects (font (size 1.27 1.27)) hide)
     )
@@
       (effects (font (size 1.27 1.27)))
     )
-    (property "Footprint" "Capacitor_SMD:C_1206_3216Metric_Pad1.33x1.80mm_HandSolder" (at 78.74 34.29 0)
+    (property "Footprint" "Capacitor_SMD:C_0805_2012Metric_Pad1.18x1.45mm_HandSolder" (at 78.74 34.29 0)
       (effects (font (size 1.27 1.27)) hide)
     )
@@
       (effects (font (size 1.27 1.27)))
     )
-    (property "Footprint" "Capacitor_SMD:C_1206_3216Metric_Pad1.33x1.80mm_HandSolder" (at 80.01 77.47 0)
+    (property "Footprint" "Capacitor_SMD:C_0805_2012Metric_Pad1.18x1.45mm_HandSolder" (at 80.01 77.47 0)
       (effects (font (size 1.27 1.27)) hide)
     )
@@
       (effects (font (size 1.27 1.27)))
     )
-    (property "Footprint" "Capacitor_SMD:C_1206_3216Metric_Pad1.33x1.80mm_HandSolder" (at 102.87 137.16 0)
-      (effects (font (size 1.27 1.27)) hide)
-    )
+    (property "Footprint" "Capacitor_SMD:C_0805_2012Metric_Pad1.18x1.45mm_HandSolder" (at 102.87 137.16 0)
+      (effects (font (size 1.27 1.27)) hide)
+    )

Commit message: added some jlcpcb part numbers, adjusted some footprints and values accordingly.
Parts:
- C61: LCSC C14663 -> C49678; LINK (none) -> https://jlcpcb.com/partdetail/Yageo-CC0805KRX7R9BB104/C49678
- C61: footprint Capacitor_SMD:C_1206_3216Metric_Pad1.33x1.80mm_HandSolder -> Capacitor_SMD:C_0805_2012Metric_Pad1.18x1.45mm_HandSolder; LCSC C14663 -> C46653; LINK (none) -> https://jlcpcb.com/partdetail/47657-CL21B102KBCNNNC/C46653
Changed lines of the file:
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@@
       (effects (font (size 1.27 1.27)) hide)
     )
-    (property "LCSC" "C14663" (at 78.74 55.88 90)
+    (property "LCSC" "C49678" (at 78.74 55.88 90)
+      (effects (font (size 1.27 1.27)) hide)
+    )
+    (property "LINK" "https://jlcpcb.com/partdetail/Yageo-CC0805KRX7R9BB104/C49678" (at 78.74 55.88 0)
       (effects (font (size 1.27 1.27)) hide)
     )
@@
       (effects (font (size 1.27 1.27)) hide)
     )
-    (property "LCSC" "C14663" (at 179.07 62.23 90)
+    (property "LCSC" "C49678" (at 179.07 62.23 90)
+      (effects (font (size 1.27 1.27)) hide)
+    )
+    (property "LINK" "https://jlcpcb.com/partdetail/Yageo-CC0805KRX7R9BB104/C49678" (at 179.07 62.23 0)
       (effects (font (size 1.27 1.27)) hide)
     )
@@
       (effects (font (size 1.27 1.27)) hide)
     )
-    (property "LCSC" "C14663" (at 78.74 34.29 90)
+    (property "LCSC" "C49678" (at 78.74 34.29 90)
+      (effects (font (size 1.27 1.27)) hide)
+    )
+    (property "LINK" "https://jlcpcb.com/partdetail/Yageo-CC0805KRX7R9BB104/C49678" (at 78.74 34.29 0)
       (effects (font (size 1.27 1.27)) hide)
     )
@@
       (effects (font (size 1.27 1.27)) hide)
     )
-    (property "LCSC" "C14663" (at 80.01 77.47 90)
+    (property "LCSC" "C49678" (at 80.01 77.47 90)
+      (effects (font (size 1.27 1.27)) hide)
+    )
+    (property "LINK" "https://jlcpcb.com/partdetail/Yageo-CC0805KRX7R9BB104/C49678" (at 80.01 77.47 0)
       (effects (font (size 1.27 1.27)) hide)
     )
@@
       (effects (font (size 1.27 1.27)) hide)
     )
-    (property "LCSC" "C14663" (at 179.07 83.82 90)
+    (property "LCSC" "C49678" (at 179.07 83.82 90)
+      (effects (font (size 1.27 1.27)) hide)
+    )
+    (property "LINK" "https://jlcpcb.com/partdetail/Yageo-CC0805KRX7R9BB104/C49678" (at 179.07 83.82 0)
       (effects (font (size 1.27 1.27)) hide)
     )
@@
       (effects (font (size 1.27 1.27)) hide)
     )
-    (property "LCSC" "C14663" (at 175.26 40.64 90)
+    (property "LCSC" "C49678" (at 175.26 40.64 90)
+      (effects (font (size 1.27 1.27)) hide)
+    )
+    (property "LINK" "https://jlcpcb.com/partdetail/Yageo-CC0805KRX7R9BB104/C49678" (at 175.26 40.64 0)
       (effects (font (size 1.27 1.27)) hide)
     )
@@
       (effects (font (size 1.27 1.27)))
     )
-    (property "Footprint" "Capacitor_SMD:C_1206_3216Metric_Pad1.33x1.80mm_HandSolder" (at 71.12 132.08 0)
+    (property "Footprint" "Capacitor_SMD:C_0805_2012Metric_Pad1.18x1.45mm_HandSolder" (at 71.12 132.08 0)
       (effects (font (size 1.27 1.27)) hide)
     )
@@
       (effects (font (size 1.27 1.27)) hide)
     )
-    (property "LCSC" "C14663" (at 71.12 132.08 90)
+    (property "LCSC" "C46653" (at 71.12 132.08 90)
+      (effects (font (size 1.27 1.27)) hide)
+    )
+    (property "LINK" "https://jlcpcb.com/partdetail/47657-CL21B102KBCNNNC/C46653" (at 71.12 132.08 0)
       (effects (font (size 1.27 1.27)) hide)
     )
@@
       (effects (font (size 1.27 1.27)) hide)
     )
-    (property "LCSC" "C14663" (at 102.87 137.16 90)
-      (effects (font (size 1.27 1.27)) hide)
-    )
+    (property "LCSC" "C49678" (at 102.87 137.16 90)
+      (effects (font (size 1.27 1.27)) hide)
+    )
+    (property "LINK" "https://jlcpcb.com/partdetail/Yageo-CC0805KRX7R9BB104/C49678" (at 102.87 137.16 0)
+      (effects (font (size 1.27 1.27)) hide)
+    )

Commit message: more partnumbers assigned. split difficult values into two parts. add protection of CP_SENSE port
Parts:
- R11: footprint Resistor_SMD:R_1206_3216Metric_Pad1.30x1.75mm_HandSolder -> Resistor_SMD:R_0805_2012Metric_Pad1.20x1.40mm_HandSolder; LCSC C25804 -> C17713; LINK (none) -> https://jlcpcb.com/partdetail/18401-0805W8F4702T5E/C17713
- R11: footprint Resistor_SMD:R_1206_3216Metric_Pad1.30x1.75mm_HandSolder -> Resistor_SMD:R_0805_2012Metric_Pad1.20x1.40mm_HandSolder; LCSC todo -> C17513; LINK (none) -> https://jlcpcb.com/partdetail/18201-0805W8F1001T5E/C17513
- R11: footprint Resistor_SMD:R_1206_3216Metric_Pad1.30x1.75mm_HandSolder -> Resistor_SMD:R_0805_2012Metric_Pad1.20x1.40mm_HandSolder; LCSC C25804 -> C17414; LINK (none) -> https://jlcpcb.com/partdetail/18102-0805W8F1002T5E/C17414
- R3: footprint Resistor_SMD:R_1206_3216Metric_Pad1.30x1.75mm_HandSolder -> Resistor_SMD:R_0805_2012Metric_Pad1.20x1.40mm_HandSolder; LCSC tbd -> C17560; LINK (none) -> https://jlcpcb.com/partdetail/18248-0805W8F2202T5E/C17560
- R3: footprint Resistor_SMD:R_1206_3216Metric_Pad1.30x1.75mm_HandSolder -> Resistor_SMD:R_0805_2012Metric_Pad1.20x1.40mm_HandSolder; LCSC C22978 -> C17572; LINK (none) -> https://jlcpcb.com/partdetail/18260-0805W8F2400T5E/C17572
- R3: footprint Resistor_SMD:R_1206_3216Metric_Pad1.30x1.75mm_HandSolder -> Resistor_SMD:R_0805_2012Metric_Pad1.20x1.40mm_HandSolder; LCSC tbd -> C17572; LINK (none) -> https://jlcpcb.com/partdetail/18260-0805W8F2400T5E/C17572
- R3: footprint Resistor_SMD:R_1206_3216Metric_Pad1.30x1.75mm_HandSolder -> Resistor_SMD:R_0805_2012Metric_Pad1.20x1.40mm_HandSolder; LCSC tbd -> C17713; LINK (none) -> https://jlcpcb.com/partdetail/18401-0805W8F4702T5E/C17713

Commit message: WIP: PP pull-up and divider. variant detection. ipropi connected to ADC.
Parts:
- added JP2: PP_PULLDOWN, Jumper:SolderJumper-2_P1.3mm_Open_TrianglePad1.0x1.5mm, symbol Jumper:SolderJumper_2_Open
- added R11, R3: 47k, Resistor_SMD:R_0805_2012Metric_Pad1.20x1.40mm_HandSolder, symbol Device:R_Small
- added R11: 3k0, Resistor_SMD:R_0805_2012Metric_Pad1.20x1.40mm_HandSolder, symbol Device:R_Small
- added R11: 10k, Resistor_SMD:R_0805_2012Metric_Pad1.20x1.40mm_HandSolder, symbol Device:R_Small
- R11: value 1k -> 330; LCSC C17513 -> C17634; LINK https://jlcpcb.com/partdetail/18201-0805W8F1001T5E/C17513 -> https://jlcpcb.com/partdetail/18318-0805W8F3300T5E/C17630
Connections:
- net 3V3_uC: now also R3.2; no longer R11.1
- net ADC_PP: now also R11.1
- net GND: now also R11.2, R11.2, R11.2
- net PP: now also JP2.1 (A)
- new net: JP2.2 (B), R11.1
- new net 5V: R11.1
- new net ADC_HWVARIANT: R11.1, R3.1
Other:
- note added: "330 ohms to 5V is the "offical" spec"
- note added: "Divider 2:1 to be able to measure up to 5V with the 3.3V ADC ref."
- note added: "Hardware variant detection: R62 can be increased with each hardware version 10k: Foccci 4.2"
- note added: "PlugPresent: - 1k5 to ground for CCS2 - 100 ohm to 1k5 for AC (current limit of the cable) - 150 ohm (button idle) or 480 ohm (button pressed) for CCS1 Some inlets may contain 2k7 or 3k0 to ground. The optional R60 can be used if no external pull down is present. Discussion here: https://openinverter.org/forum/viewtopic.php?p=66305#p66305"
- note removed: "PlugPresent: - 1k5 to ground for CCS2 - 100 ohm to 1k5 for AC (current limit of the cable) - 150 ohm (button idle) or 480 ohm (button pressed) for CCS1"
- moved on the sheet: R11
