File: pcb/Inputs.kicad_sch (KiCad schematic)
At the start: 29 parts

Commit message: feature: Added wakeup logic
Parts:
- added JP4: PP_PULL5V, Jumper:SolderJumper-2_P1.3mm_Open_TrianglePad1.0x1.5mm, symbol Jumper:SolderJumper_2_Open
- added JP5: PP_PULL12V, Jumper:SolderJumper-2_P1.3mm_Open_TrianglePad1.0x1.5mm, symbol Jumper:SolderJumper_2_Open
- added R64: 6k2, Resistor_SMD:R_0805_2012Metric_Pad1.20x1.40mm_HandSolder, symbol Device:R_Small
- R28: renamed from R11; value 47k -> 33k; LCSC C17713 -> (none)
- R57: renamed from R11; value 47k -> 100k
- renumbered C61 to C20, C61 to C21, C61 to C23, C61 to C71, C61 to C77, C61 to C78, C61 to C79, C61 to C80, JP2 to JP3, R11 to R31, R11 to R32, R11 to R33, R11 to R34, R11 to R35, R11 to R36, R3 to R39, R3 to R40, R3 to R41, R3 to R42, R11 to R52, R11 to R53, R11 to R54, R11 to R55, R11 to R56, R11 to R60, R3 to R61, R11 to R62
Connections:
- net PP: now also JP4.1 (A), JP5.1 (A); no longer R56.2
- new net: JP5.2 (B), R64.2
- new net: JP4.2 (B), R56.2
- new net 12V_P: R64.1
Other:
- note added: "Divider 4:1 to be able to measure up to 13.3V with the 3.3V ADC ref."
- note added: "Pull-up to 12V is needed if we want PP to enable the controller. Threshold is 2.5V"
- note removed: "Divider 2:1 to be able to measure up to 5V with the 3.3V ADC ref."
- moved on the sheet: R56

Commit message: Corrected pin map for CJ431 Increased variant resistor Added pull-down for Wakeup
Parts:
- R62: value 10k -> 12k; LCSC C17414 -> C22790
Other:
- note added: "Hardware variant detection: R62 can be increased with each hardware version 10k: Foccci 4.2 12k: Foccci 4.3"
- note removed: "Hardware variant detection: R62 can be increased with each hardware version 10k: Foccci 4.2"
Changed lines of the file:
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@@
     (effects (font (size 1.27 1.27)) (justify left bottom))
   )
-  (text "Hardware variant detection: R62 can be increased with each hardware version\n10k: Foccci 4.2"
+  (text "Hardware variant detection: R62 can be increased with each hardware version\n10k: Foccci 4.2\n12k: Foccci 4.3"
     (at 73.66 166.37 0)
     (effects (font (size 1.27 1.27)) (justify left bottom))
@@
       (effects (font (size 1.27 1.27)))
     )
-    (property "Value" "10k" (at 66.04 168.91 0)
+    (property "Value" "12k" (at 66.04 168.91 0)
       (effects (font (size 1.27 1.27)))
     )
@@
       (effects (font (size 1.27 1.27)) hide)
     )
-    (property "LCSC" "C17414" (at 63.5 167.64 0)
-      (effects (font (size 1.27 1.27)) hide)
-    )
+    (property "LCSC" "C22790" (at 63.5 167.64 0)
+      (effects (font (size 1.27 1.27)) hide)
+    )

Commit message: Made relay drivers PMOS with gate drivers and free wheeling diode
Parts:
- R62: value 12k -> 15k; LCSC C22790 -> C22809
Other:
- note added: "Hardware variant detection: R62 can be increased with each hardware version 10k: Foccci 4.2 12k: Foccci 4.3 15k: Foccci 4.4"
- note removed: "Hardware variant detection: R62 can be increased with each hardware version 10k: Foccci 4.2 12k: Foccci 4.3"
Changed lines of the file:
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@@
     (effects (font (size 1.27 1.27)) (justify left bottom))
   )
-  (text "Hardware variant detection: R62 can be increased with each hardware version\n10k: Foccci 4.2\n12k: Foccci 4.3"
+  (text "Hardware variant detection: R62 can be increased with each hardware version\n10k: Foccci 4.2\n12k: Foccci 4.3\n15k: Foccci 4.4"
     (at 73.66 166.37 0)
     (effects (font (size 1.27 1.27)) (justify left bottom))
@@
       (effects (font (size 1.27 1.27)))
     )
-    (property "Value" "12k" (at 66.04 168.91 0)
+    (property "Value" "15k" (at 66.04 168.91 0)
       (effects (font (size 1.27 1.27)))
     )
@@
       (effects (font (size 1.27 1.27)) hide)
     )
-    (property "LCSC" "C22790" (at 63.5 167.64 0)
-      (effects (font (size 1.27 1.27)) hide)
-    )
+    (property "LCSC" "C22809" (at 63.5 167.64 0)
+      (effects (font (size 1.27 1.27)) hide)
+    )

Commit message: Using another motor driver IC for contactor control
Other:
- note added: "Hardware variant detection: R62 can be increased with each hardware version Table here: https://openinverter.org/wiki/Fully_Open_CCS_Charge_Controller_(FOCCCI) 10k: Foccci 4.2 12k: Foccci 4.3 15k: Foccci 4.4"
- note added: "Pull-up to 12V is needed if we want PP to enable the controller. Threshold is 3V"
- note removed: "Hardware variant detection: R62 can be increased with each hardware version 10k: Foccci 4.2 12k: Foccci 4.3 15k: Foccci 4.4"
- note removed: "Pull-up to 12V is needed if we want PP to enable the controller. Threshold is 2.5V"
Changed lines of the file:
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@@
     (effects (font (size 1.27 1.27)) (justify left bottom))
   )
-  (text "Hardware variant detection: R62 can be increased with each hardware version\n10k: Foccci 4.2\n12k: Foccci 4.3\n15k: Foccci 4.4"
+  (text "Hardware variant detection: R62 can be increased with each hardware version\nTable here: https://openinverter.org/wiki/Fully_Open_CCS_Charge_Controller_(FOCCCI)\n10k: Foccci 4.2\n12k: Foccci 4.3\n15k: Foccci 4.4"
     (at 73.66 166.37 0)
     (effects (font (size 1.27 1.27)) (justify left bottom))
@@
     (effects (font (size 1.27 1.27)) (justify left bottom) (href "https://openinverter.org/forum/viewtopic.php?p=58839#p58839"))
   )
-  (text "Pull-up to 12V is needed if we want PP \nto enable the controller. Threshold is 2.5V"
+  (text "Pull-up to 12V is needed if we want PP \nto enable the controller. Threshold is 3V"
     (at 135.89 64.77 0)
     (effects (font (size 1.27 1.27)) (justify left bottom))

Commit message: Redesigned wakeup circuit
Parts:
- removed JP3: PP_PULLDOWN, Jumper:SolderJumper-2_P1.3mm_Open_TrianglePad1.0x1.5mm, symbol Jumper:SolderJumper_2_Open
- removed JP4: PP_PULL5V, Jumper:SolderJumper-2_P1.3mm_Open_TrianglePad1.0x1.5mm, symbol Jumper:SolderJumper_2_Open
- removed JP5: PP_PULL12V, Jumper:SolderJumper-2_P1.3mm_Open_TrianglePad1.0x1.5mm, symbol Jumper:SolderJumper_2_Open
- removed R56: 330, Resistor_SMD:R_0805_2012Metric_Pad1.20x1.40mm_HandSolder, symbol Device:R_Small
- removed R64: 6k2, Resistor_SMD:R_0805_2012Metric_Pad1.20x1.40mm_HandSolder, symbol Device:R_Small
- added D20: B5819W, Diode_SMD:D_SOD-123, symbol Diode:1N4148W
- added D22, D23: BAV99, Package_TO_SOT_SMD:SOT-23, symbol Diode:BAV99
- added JP3: SolderJumper_3_Open, Jumper:SolderJumper-3_P1.3mm_Open_RoundedPad1.0x1.5mm, symbol Jumper:SolderJumper_3_Open
- added R66: 100k, Resistor_SMD:R_0805_2012Metric_Pad1.20x1.40mm_HandSolder, symbol Device:R_Small
- added R71: 330, Resistor_SMD:R_0805_2012Metric_Pad1.20x1.40mm_HandSolder, symbol Device:R_Small
- R28: value 33k -> 47k
- R53: value 47k -> 22k; LCSC C17713 -> C17560; LINK https://jlcpcb.com/partdetail/18401-0805W8F4702T5E/C17713 -> https://jlcpcb.com/partdetail/18248-0805W8F2202T5E/C17560
- R57: value 100k -> 47k
Connections:
- net 12V_P: now also R52.1, D22.2 (A), D23.2 (A)
- net 3V3_uC: no longer R52.1
- net 5V: now also D20.2 (A)
- net ADC_BUTTON: now also R66.2
- net BUTTON: now also D23.3 (K), R66.1; no longer R53.1
- net GND: now also R53.1, D22.1 (K), D23.1 (K)
- net PP: now also D22.3 (K), JP3.2 (C), R71.2
- net at R60.1: now also JP3.3 (B)
- new net: D20.1 (K), R71.1
- new net PP_WAKE: JP3.1 (A)
Other:
- note added: "Divider 2:1 to be able to measure up to 6.6V with the 3.3V ADC ref."
- note added: "PlugPresent: - 1k5 to ground for CCS2 - 100 ohm to 1k5 for AC (current limit of the cable) - 150 ohm (button idle) or 480 ohm (button pressed) for CCS1 Some inlets may contain 2k7 or 3k0 to ground. The optional R60 can be used if no external pull down is present. Discussion here: https://openinverter.org/forum/viewtopic.php?p=66305#p66305 Wakeup via PP only works without any pull-down resistor"
- note removed: "Divider 4:1 to be able to measure up to 13.3V with the 3.3V ADC ref."
- note removed: "PlugPresent: - 1k5 to ground for CCS2 - 100 ohm to 1k5 for AC (current limit of the cable) - 150 ohm (button idle) or 480 ohm (button pressed) for CCS1 Some inlets may contain 2k7 or 3k0 to ground. The optional R60 can be used if no external pull down is present. Discussion here: https://openinverter.org/forum/viewtopic.php?p=66305#p66305"
- moved on the sheet: R52, R60

Commit message: Added 1M discharge resistor for CP enable Removed momentary turn-on resitor for PP enable because always charged by uC voltage divider
Parts:
- R60: value 3k0 -> 3.3K; LCSC C17661 -> C26010; LINK https://jlcpcb.com/partdetail/18349-0805W8F3001T5E/C17661 -> https://jlcpcb.com/partdetail/26753-0805W8F3301T5E/C26010
- R62: value 15k -> 18k; LCSC C22809 -> C25810; LINK https://jlcpcb.com/partdetail/18102-0805W8F1002T5E/C17414 -> https://jlcpcb.com/partdetail/26553-0603WAF1802T5E/C25810
Other:
- note added: "Hardware variant detection: R62 can be increased with each hardware version Table here: https://openinverter.org/wiki/Fully_Open_CCS_Charge_Controller_(FOCCCI) 10k: Foccci 4.2 12k: Foccci 4.3 15k: Foccci 4.4 18k: Foccci 4.5"
- note removed: "Hardware variant detection: R62 can be increased with each hardware version Table here: https://openinverter.org/wiki/Fully_Open_CCS_Charge_Controller_(FOCCCI) 10k: Foccci 4.2 12k: Foccci 4.3 15k: Foccci 4.4"
Changed lines of the file:
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@@
     (effects (font (size 1.27 1.27)) (justify left bottom))
   )
-  (text "Hardware variant detection: R62 can be increased with each hardware version\nTable here: https://openinverter.org/wiki/Fully_Open_CCS_Charge_Controller_(FOCCCI)\n10k: Foccci 4.2\n12k: Foccci 4.3\n15k: Foccci 4.4"
+  (text "Hardware variant detection: R62 can be increased with each hardware version\nTable here: https://openinverter.org/wiki/Fully_Open_CCS_Charge_Controller_(FOCCCI)\n10k: Foccci 4.2\n12k: Foccci 4.3\n15k: Foccci 4.4\n18k: Foccci 4.5"
     (at 73.66 166.37 0)
     (effects (font (size 1.27 1.27)) (justify left bottom))
@@
     )
   )
+  (symbol (lib_id "Device:R_Small") (at 166.37 93.98 90) (unit 1)
+    (in_bom yes) (on_board yes) (dnp no)
+    (property "Reference" "R60" (at 166.37 91.44 90)
+      (effects (font (size 1.27 1.27)))
+    )
+    (property "Value" "3.3K" (at 166.37 96.52 90)
+      (effects (font (size 1.27 1.27)))
+    )
+    (property "Footprint" "Resistor_SMD:R_0805_2012Metric_Pad1.20x1.40mm_HandSolder" (at 166.37 93.98 0)
+      (effects (font (size 1.27 1.27)) hide)
+    )
+    (property "Datasheet" "https://datasheet.lcsc.com/lcsc/1811101920_UNI-ROYAL-Uniroyal-Elec-0603WAF3301T5E_C22978.pdf" (at 166.37 93.98 0)
+      (effects (font (size 1.27 1.27)) hide)
+    )
+    (property "LCSC" "C26010" (at 166.37 93.98 90)
+      (effects (font (size 1.27 1.27)) hide)
+    )
+    (property "LINK" "https://jlcpcb.com/partdetail/26753-0805W8F3301T5E/C26010" (at 166.37 93.98 0)
+      (effects (font (size 1.27 1.27)) hide)
+    )
+    (pin "1")
+    (pin "2")
+    (instances
+      (project "qca7000"
+        (path "/e63e39d7-6ac0-4ffd-8aa3-1841a4541b55/93c6207c-4203-4bc7-a590-e5e89c0d3d27"
+          (reference "R60") (unit 1)
+        )
+      )
+    )
+  )
   (symbol (lib_id "Device:R_Small") (at 73.66 53.34 90) (unit 1)
     (in_bom yes) (on_board yes) (dnp no)
@@
         (path "/e63e39d7-6ac0-4ffd-8aa3-1841a4541b55/93c6207c-4203-4bc7-a590-e5e89c0d3d27"
           (reference "C23") (unit 1)
-        )
-      )
-    )
-  )
-  (symbol (lib_id "Device:R_Small") (at 166.37 93.98 90) (unit 1)
-    (in_bom yes) (on_board yes) (dnp no)
-    (property "Reference" "R60" (at 166.37 91.44 90)
-      (effects (font (size 1.27 1.27)))
-    )
-    (property "Value" "3k0" (at 166.37 96.52 90)
-      (effects (font (size 1.27 1.27)))
-    )
-    (property "Footprint" "Resistor_SMD:R_0805_2012Metric_Pad1.20x1.40mm_HandSolder" (at 166.37 93.98 0)
-      (effects (font (size 1.27 1.27)) hide)
-    )
-    (property "Datasheet" "~" (at 166.37 93.98 0)
-      (effects (font (size 1.27 1.27)) hide)
-    )
-    (property "LCSC" "C17661" (at 166.37 93.98 0)
-      (effects (font (size 1.27 1.27)) hide)
-    )
-    (property "LINK" "https://jlcpcb.com/partdetail/18349-0805W8F3001T5E/C17661" (at 166.37 93.98 0)
-      (effects (font (size 1.27 1.27)) hide)
-    )
-    (pin "1")
-    (pin "2")
-    (instances
-      (project "qca7000"
-        (path "/e63e39d7-6ac0-4ffd-8aa3-1841a4541b55/93c6207c-4203-4bc7-a590-e5e89c0d3d27"
-          (reference "R60") (unit 1)
         )
       )
@@
       (effects (font (size 1.27 1.27)))
     )
-    (property "Value" "15k" (at 66.04 168.91 0)
+    (property "Value" "18k" (at 66.04 168.91 0)
       (effects (font (size 1.27 1.27)))
     )
@@
       (effects (font (size 1.27 1.27)) hide)
     )
-    (property "LCSC" "C22809" (at 63.5 167.64 0)
-      (effects (font (size 1.27 1.27)) hide)
-    )
-    (property "LINK" "https://jlcpcb.com/partdetail/18102-0805W8F1002T5E/C17414" (at 63.5 167.64 0)
+    (property "LCSC" "C25810" (at 63.5 167.64 0)
+      (effects (font (size 1.27 1.27)) hide)
+    )
+    (property "LINK" "https://jlcpcb.com/partdetail/26553-0603WAF1802T5E/C25810" (at 63.5 167.64 0)
       (effects (font (size 1.27 1.27)) hide)
     )
@@
   (symbol (lib_id "Jumper:SolderJumper_3_Open") (at 158.75 88.9 270) (unit 1)
     (in_bom yes) (on_board yes) (dnp no)
-    (property "Reference" "JP3" (at 160.401 92.7679 90)
+    (property "Reference" "JP3" (at 160.02 88.9 90)
       (effects (font (size 1.27 1.27)) (justify left))
     )

Commit message: BOM optimization
Parts:
- R28: LCSC (none) -> C17713
Changed lines of the file:
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@@
+      (effects (font (size 1.27 1.27)) hide)
+    )
+    (property "LCSC" "C17713" (at 190.5 85.09 0)
       (effects (font (size 1.27 1.27)) hide)
     )

Commit message: Made PP standby and button pullup 1k Improved connection of TVS diode
Parts:
- R52: value 10k -> 1k; LCSC C17414 -> C17513; LINK https://jlcpcb.com/partdetail/18102-0805W8F1002T5E/C17414 -> https://jlcpcb.com/partdetail/18201-0805W8F1001T5E/C17513
Connections:
- net 12V_P: now also R52.2; no longer R52.1
- net BUTTON: now also R52.1; no longer R52.2
Other:
- note removed: "Pull-up to 12V is needed if we want PP to enable the controller. Threshold is 3V"
Changed lines of the file:
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@@
     (effects (font (size 1.27 1.27)) (justify left bottom) (href "https://openinverter.org/forum/viewtopic.php?p=58839#p58839"))
-  )
-  (text "Pull-up to 12V is needed if we want PP \nto enable the controller. Threshold is 3V"
-    (at 135.89 64.77 0)
-    (effects (font (size 1.27 1.27)) (justify left bottom))
   )
   (text "330 ohms to 5V is the \"offical\" spec" (at 114.3 78.74 0)
@@
     )
   )
-  (symbol (lib_id "Device:R_Small") (at 151.13 33.02 0) (unit 1)
-    (in_bom yes) (on_board yes) (dnp no)
-    (property "Reference" "R52" (at 153.67 30.48 0)
-      (effects (font (size 1.27 1.27)))
-    )
-    (property "Value" "10k" (at 153.67 34.29 0)
-      (effects (font (size 1.27 1.27)))
-    )
-    (property "Footprint" "Resistor_SMD:R_0805_2012Metric_Pad1.20x1.40mm_HandSolder" (at 151.13 33.02 0)
-      (effects (font (size 1.27 1.27)) hide)
-    )
-    (property "Datasheet" "~" (at 151.13 33.02 0)
-      (effects (font (size 1.27 1.27)) hide)
-    )
-    (property "LCSC" "C17414" (at 151.13 33.02 0)
-      (effects (font (size 1.27 1.27)) hide)
-    )
-    (property "LINK" "https://jlcpcb.com/partdetail/18102-0805W8F1002T5E/C17414" (at 151.13 33.02 0)
-      (effects (font (size 1.27 1.27)) hide)
-    )
-    (pin "1")
-    (pin "2")
-    (instances
-      (project "qca7000"
-        (path "/e63e39d7-6ac0-4ffd-8aa3-1841a4541b55/93c6207c-4203-4bc7-a590-e5e89c0d3d27"
-          (reference "R52") (unit 1)
-        )
-      )
-    )
-  )
   (symbol (lib_id "power:GND") (at 170.18 93.98 0) (unit 1)
     (in_bom yes) (on_board yes) (dnp no)
@@
         )
       )
+    )
+  )
+  (symbol (lib_id "Device:R_Small") (at 151.13 33.02 180) (unit 1)
+    (in_bom yes) (on_board yes) (dnp no)
+    (property "Reference" "R52" (at 148.59 33.02 90)
+      (effects (font (size 1.27 1.27)))
+    )
+    (property "Value" "1k" (at 153.67 33.02 90)
+      (effects (font (size 1.27 1.27)))
+    )
+    (property "Footprint" "Resistor_SMD:R_0805_2012Metric_Pad1.20x1.40mm_HandSolder" (at 151.13 33.02 0)
+      (effects (font (size 1.27 1.27)) hide)
+    )
+    (property "Datasheet" "https://datasheet.lcsc.com/lcsc/1811101920_UNI-ROYAL-Uniroyal-Elec-0603WAF3301T5E_C22978.pdf" (at 151.13 33.02 0)
+      (effects (font (size 1.27 1.27)) hide)
+    )
+    (property "LCSC" "C17513" (at 151.13 33.02 90)
+      (effects (font (size 1.27 1.27)) hide)
+    )
+    (property "LINK" "https://jlcpcb.com/partdetail/18201-0805W8F1001T5E/C17513" (at 151.13 33.02 0)
+      (effects (font (size 1.27 1.27)) hide)
+    )
+    (pin "1")
+    (pin "2")
+    (instances
+      (project "qca7000"
+        (path "/e63e39d7-6ac0-4ffd-8aa3-1841a4541b55/93c6207c-4203-4bc7-a590-e5e89c0d3d27"
+          (reference "R52") (unit 1)
+        )
+      )
