File: pcb/Inputs.kicad_sch (KiCad schematic)
At the start: 33 parts

Commit message: version 5
Other:
- note added: "Hardware variant detection: R62 can be increased with each hardware version Table here: https://openinverter.org/wiki/Fully_Open_CCS_Charge_Controller_(FOCCCI) 10k: Foccci 4.2 12k: Foccci 4.3 15k: Foccci 4.4 18k: Foccci 4.5, 4.5b and 5"
- note removed: "Hardware variant detection: R62 can be increased with each hardware version Table here: https://openinverter.org/wiki/Fully_Open_CCS_Charge_Controller_(FOCCCI) 10k: Foccci 4.2 12k: Foccci 4.3 15k: Foccci 4.4 18k: Foccci 4.5"
Changed lines of the file:
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@@
 		)
 	)
-	(text "Hardware variant detection: R62 can be increased with each hardware version\nTable here: https://openinverter.org/wiki/Fully_Open_CCS_Charge_Controller_(FOCCCI)\n10k: Foccci 4.2\n12k: Foccci 4.3\n15k: Foccci 4.4\n18k: Foccci 4.5"
+	(text "Hardware variant detection: R62 can be increased with each hardware version\nTable here: https://openinverter.org/wiki/Fully_Open_CCS_Charge_Controller_(FOCCCI)\n10k: Foccci 4.2\n12k: Foccci 4.3\n15k: Foccci 4.4\n18k: Foccci 4.5, 4.5b and 5"
 		(exclude_from_sim no)
 		(at 73.66 166.37 0)

Commit message: corrected some rotations for JLC. Version 5.2p7
Parts:
- D22, D23: JLCPCB Rotation Offset 180 -> 0
Changed lines of the file:
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@@
 			)
 		)
-		(property "JLCPCB Rotation Offset" "180"
+		(property "JLCPCB Rotation Offset" "0"
 			(at 138.43 27.94 90)
 			(effects
@@
 			)
 		)
-		(property "JLCPCB Rotation Offset" "180"
+		(property "JLCPCB Rotation Offset" "0"
 			(at 106.68 95.25 90)
 			(effects
