File: pcb/connectors.kicad_sch (KiCad schematic)
At the start: 2 parts, among them J20 DTM1312PA12PBR008, U8 EEC-325X4B

Commit message: added RGB LED highside drivers
Parts:
- added H1: MountingHole, MountingHole:MountingHole_3.2mm_M3, symbol Mechanical:MountingHole
Changed lines of the file:
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@@
+    )
+  )
+  (symbol (lib_id "Mechanical:MountingHole") (at 44.45 111.76 0) (unit 1)
+    (in_bom yes) (on_board yes) (dnp no) (fields_autoplaced)
+    (property "Reference" "H1" (at 46.99 111.125 0)
+      (effects (font (size 1.27 1.27)) (justify left))
+    )
+    (property "Value" "MountingHole" (at 46.99 113.665 0)
+      (effects (font (size 1.27 1.27)) (justify left))
+    )
+    (property "Footprint" "MountingHole:MountingHole_3.2mm_M3" (at 44.45 111.76 0)
+      (effects (font (size 1.27 1.27)) hide)
+    )
+    (property "Datasheet" "~" (at 44.45 111.76 0)
+      (effects (font (size 1.27 1.27)) hide)
+    )
+    (instances
+      (project "qca7000"
+        (path "/e63e39d7-6ac0-4ffd-8aa3-1841a4541b55/23ec3d7a-4d8b-4fb1-94c6-debe6172b9c6"
+          (reference "H1") (unit 1)
+        )
+      )
     )
   )

Commit message: first draft with the DRV8874 hbridge driver. Added 3D models.
Connections:
- net CONN_LOCK_MOT1: now also J20.A9
Changed lines of the file:
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@@
+    (stroke (width 0) (type default))
+  )
+  (wire (pts (xy 44.45 64.77) (xy 53.34 64.77))
     (stroke (width 0) (type default))
   )

Commit message: wired the drv8874. Added spare holes. Flash connector larger holes
Connections:
- net BUTTON: now also J20.B12
- net CONN_LOCK_FEEDBACK: now also J20.A4
- no-connect marks 0 -> 4
Changed lines of the file:
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@@
 (kicad_sch (version 20230121) (generator eeschema)
   (paper "A4")
+  (no_connect (at 78.74 49.53))
+  (no_connect (at 78.74 59.69))
+  (no_connect (at 78.74 52.07))
+  (no_connect (at 53.34 69.85))
+  (wire (pts (xy 52.07 52.07) (xy 53.34 52.07))
+    (stroke (width 0) (type default))
+  )
   (wire (pts (xy 53.34 43.18) (xy 53.34 44.45))
+    (stroke (width 0) (type default))
+  )
+  (wire (pts (xy 78.74 72.39) (xy 85.09 72.39))
     (stroke (width 0) (type default))
   )
@@
     )
   )
-  (global_label "BUTTON" (shape output) (at 106.68 77.47 0) (fields_autoplaced)
+  (global_label "BUTTON" (shape output) (at 85.09 72.39 0) (fields_autoplaced)
     (effects (font (size 1.27 1.27)) (justify left))
-    (property "Intersheetrefs" "${INTERSHEET_REFS}" (at 116.7825 77.47 0)
+    (property "Intersheetrefs" "${INTERSHEET_REFS}" (at 95.1925 72.39 0)
       (effects (font (size 1.27 1.27)) (justify left) hide)
     )
@@
     )
   )
-  (global_label "CONN_LOCK_FEEDBACK" (shape output) (at 106.68 74.93 0) (fields_autoplaced)
-    (effects (font (size 1.27 1.27)) (justify left))
-    (property "Intersheetrefs" "${INTERSHEET_REFS}" (at 131.2363 74.93 0)
-      (effects (font (size 1.27 1.27)) (justify left) hide)
+  (global_label "CONN_LOCK_FEEDBACK" (shape output) (at 52.07 52.07 180) (fields_autoplaced)
+    (effects (font (size 1.27 1.27)) (justify right))
+    (property "Intersheetrefs" "${INTERSHEET_REFS}" (at 27.5137 52.07 0)
+      (effects (font (size 1.27 1.27)) (justify right) hide)
     )
   )

Commit message: changed to 4 layers. Added button, PP and lock feedback. New testpoints to avoid courtyard warnings.
Parts:
- J20: footprint TE_DTM1312PA12PBR008 -> DTM1312PA12PBR008:TE_DTM1312PA12PBR008
- U8: footprint TE_EEC-325X4B -> EEC-325X4B:TE_EEC-325X4B
Changed lines of the file:
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@@
       (effects (font (size 1.27 1.27)))
     )
-    (property "Footprint" "TE_DTM1312PA12PBR008" (at 66.04 57.15 0)
+    (property "Footprint" "DTM1312PA12PBR008:TE_DTM1312PA12PBR008" (at 66.04 57.15 0)
       (effects (font (size 1.27 1.27)) (justify left bottom) hide)
     )
@@
       (effects (font (size 1.27 1.27)) (justify left))
     )
-    (property "Footprint" "TE_EEC-325X4B" (at 63.5 93.98 0)
+    (property "Footprint" "EEC-325X4B:TE_EEC-325X4B" (at 63.5 93.98 0)
       (effects (font (size 1.27 1.27)) (justify left bottom) hide)
     )

Commit message: added CP sensing. Added 5V on the connector. Created gerber and pdf
Connections:
- net 5V: now reaches J20.A11
- no-connect marks 4 -> 3
Other:
- note added: "5V for the high-voltage measurement module."
Changed lines of the file:
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@@
   (no_connect (at 78.74 59.69))
   (no_connect (at 78.74 52.07))
-  (no_connect (at 53.34 69.85))
   (wire (pts (xy 52.07 52.07) (xy 53.34 52.07))
     (stroke (width 0) (type default))
@@
     (stroke (width 0) (type default))
   )
+  (wire (pts (xy 49.53 69.85) (xy 53.34 69.85))
+    (stroke (width 0) (type default))
+  )
   (wire (pts (xy 78.74 44.45) (xy 81.28 44.45))
     (stroke (width 0) (type default))
@@
     (effects (font (size 1.27 1.27)) (justify left bottom))
   )
+  (text "5V for the high-voltage\nmeasurement module." (at 24.13 74.93 0)
+    (effects (font (size 1.27 1.27)) (justify left bottom))
+  )
   (text "The connector, 2 x 12 pins,\nhttps://www.te.com/usa-en/product-DTM1312PA12PBR008.html"
     (at 73.66 35.56 0)
     (effects (font (size 1.27 1.27)) (justify left bottom))
   )
+  (global_label "5V" (shape input) (at 49.53 69.85 180) (fields_autoplaced)
+    (effects (font (size 1.27 1.27)) (justify right))
+    (property "Intersheetrefs" "${INTERSHEET_REFS}" (at 44.3261 69.85 0)
+      (effects (font (size 1.27 1.27)) (justify right) hide)
+    )
+  )
   (global_label "CONTACTOR2_LS" (shape input) (at 43.18 59.69 180) (fields_autoplaced)

Commit message: fix rx shortcut. add transformer. correct part number of NCV. Correct footprints of U1 and L11. add mounting holes. stepdown layout improved. added TVS at 12V
Parts:
- added H2, H3, H4, H5: MountingHole, MountingHole:MountingHole_3.2mm_M3, symbol Mechanical:MountingHole
Changed lines of the file:
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@@
+    )
+  )
+  (symbol (lib_id "Mechanical:MountingHole") (at 30.48 142.24 0) (unit 1)
+    (in_bom yes) (on_board yes) (dnp no) (fields_autoplaced)
+    (property "Reference" "H5" (at 33.02 141.605 0)
+      (effects (font (size 1.27 1.27)) (justify left))
+    )
+    (property "Value" "MountingHole" (at 33.02 144.145 0)
+      (effects (font (size 1.27 1.27)) (justify left))
+    )
+    (property "Footprint" "MountingHole:MountingHole_3.2mm_M3" (at 30.48 142.24 0)
+      (effects (font (size 1.27 1.27)) hide)
+    )
+    (property "Datasheet" "~" (at 30.48 142.24 0)
+      (effects (font (size 1.27 1.27)) hide)
+    )
+    (instances
+      (project "qca7000"
+        (path "/e63e39d7-6ac0-4ffd-8aa3-1841a4541b55/23ec3d7a-4d8b-4fb1-94c6-debe6172b9c6"
+          (reference "H5") (unit 1)
+        )
+      )
     )
   )
@@
         (path "/e63e39d7-6ac0-4ffd-8aa3-1841a4541b55/23ec3d7a-4d8b-4fb1-94c6-debe6172b9c6"
           (reference "#PWR093") (unit 1)
+        )
+      )
+    )
+  )
+  (symbol (lib_id "Mechanical:MountingHole") (at 30.48 128.27 0) (unit 1)
+    (in_bom yes) (on_board yes) (dnp no) (fields_autoplaced)
+    (property "Reference" "H3" (at 33.02 127.635 0)
+      (effects (font (size 1.27 1.27)) (justify left))
+    )
+    (property "Value" "MountingHole" (at 33.02 130.175 0)
+      (effects (font (size 1.27 1.27)) (justify left))
+    )
+    (property "Footprint" "MountingHole:MountingHole_3.2mm_M3" (at 30.48 128.27 0)
+      (effects (font (size 1.27 1.27)) hide)
+    )
+    (property "Datasheet" "~" (at 30.48 128.27 0)
+      (effects (font (size 1.27 1.27)) hide)
+    )
+    (instances
+      (project "qca7000"
+        (path "/e63e39d7-6ac0-4ffd-8aa3-1841a4541b55/23ec3d7a-4d8b-4fb1-94c6-debe6172b9c6"
+          (reference "H3") (unit 1)
         )
       )
@@
         )
       )
+    )
+  )
+  (symbol (lib_id "Mechanical:MountingHole") (at 30.48 121.92 0) (unit 1)
+    (in_bom yes) (on_board yes) (dnp no) (fields_autoplaced)
+    (property "Reference" "H2" (at 33.02 121.285 0)
+      (effects (font (size 1.27 1.27)) (justify left))
+    )
+    (property "Value" "MountingHole" (at 33.02 123.825 0)
+      (effects (font (size 1.27 1.27)) (justify left))
+    )
+    (property "Footprint" "MountingHole:MountingHole_3.2mm_M3" (at 30.48 121.92 0)
+      (effects (font (size 1.27 1.27)) hide)
+    )
+    (property "Datasheet" "~" (at 30.48 121.92 0)
+      (effects (font (size 1.27 1.27)) hide)
+    )
+    (instances
+      (project "qca7000"
+        (path "/e63e39d7-6ac0-4ffd-8aa3-1841a4541b55/23ec3d7a-4d8b-4fb1-94c6-debe6172b9c6"
+          (reference "H2") (unit 1)
+        )
+      )
+    )
+  )
+  (symbol (lib_id "Mechanical:MountingHole") (at 30.48 134.62 0) (unit 1)
+    (in_bom yes) (on_board yes) (dnp no) (fields_autoplaced)
+    (property "Reference" "H4" (at 33.02 133.985 0)
+      (effects (font (size 1.27 1.27)) (justify left))
+    )
+    (property "Value" "MountingHole" (at 33.02 136.525 0)
+      (effects (font (size 1.27 1.27)) (justify left))
+    )
+    (property "Footprint" "MountingHole:MountingHole_3.2mm_M3" (at 30.48 134.62 0)
+      (effects (font (size 1.27 1.27)) hide)
+    )
+    (property "Datasheet" "~" (at 30.48 134.62 0)
+      (effects (font (size 1.27 1.27)) hide)
+    )
+    (instances
+      (project "qca7000"
+        (path "/e63e39d7-6ac0-4ffd-8aa3-1841a4541b55/23ec3d7a-4d8b-4fb1-94c6-debe6172b9c6"
+          (reference "H4") (unit 1)
+        )
+      )

Commit message: feature: Added wakeup logic
Connections:
- net WAKEUP: now reaches J20.B7
- no-connect marks 3 -> 2
Changed lines of the file:
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@@
   (paper "A4")
   (no_connect (at 78.74 49.53))
-  (no_connect (at 78.74 59.69))
   (no_connect (at 78.74 52.07))
   (wire (pts (xy 52.07 52.07) (xy 53.34 52.07))
@@
   )
   (wire (pts (xy 45.72 43.18) (xy 53.34 43.18))
+    (stroke (width 0) (type default))
+  )
+  (wire (pts (xy 78.74 59.69) (xy 82.55 59.69))
     (stroke (width 0) (type default))
   )
@@
     )
   )
+  (global_label "WAKEUP" (shape bidirectional) (at 82.55 59.69 0) (fields_autoplaced)
+    (effects (font (size 1.27 1.27)) (justify left))
+    (property "Intersheetrefs" "${INTERSHEET_REFS}" (at 94.206 59.69 0)
+      (effects (font (size 1.27 1.27)) (justify left) hide)
+    )
+  )
   (global_label "LED_RED" (shape input) (at 83.82 64.77 0) (fields_autoplaced)
     (effects (font (size 1.27 1.27)) (justify left))
@@
   (symbol (lib_id "power:GND") (at 49.53 74.93 0) (unit 1)
     (in_bom yes) (on_board yes) (dnp no)
-    (property "Reference" "#PWR048" (at 49.53 81.28 0)
+    (property "Reference" "#PWR093" (at 49.53 81.28 0)
       (effects (font (size 1.27 1.27)) hide)
     )
@@
     (instances
       (project "qca7000"
-        (path "/e63e39d7-6ac0-4ffd-8aa3-1841a4541b55"
-          (reference "#PWR048") (unit 1)
-        )
-        (path "/e63e39d7-6ac0-4ffd-8aa3-1841a4541b55/5666e7cf-6b6c-4583-8335-aa3be69ccd45"
-          (reference "#PWR056") (unit 1)
-        )
-        (path "/e63e39d7-6ac0-4ffd-8aa3-1841a4541b55/93c6207c-4203-4bc7-a590-e5e89c0d3d27"
-          (reference "#PWR068") (unit 1)
-        )
         (path "/e63e39d7-6ac0-4ffd-8aa3-1841a4541b55/23ec3d7a-4d8b-4fb1-94c6-debe6172b9c6"
           (reference "#PWR093") (unit 1)
@@
   (symbol (lib_id "power:GND") (at 105.41 55.88 0) (unit 1)
     (in_bom yes) (on_board yes) (dnp no)
-    (property "Reference" "#PWR048" (at 105.41 62.23 0)
+    (property "Reference" "#PWR083" (at 105.41 62.23 0)
       (effects (font (size 1.27 1.27)) hide)
     )
@@
     (instances
       (project "qca7000"
-        (path "/e63e39d7-6ac0-4ffd-8aa3-1841a4541b55"
-          (reference "#PWR048") (unit 1)
-        )
-        (path "/e63e39d7-6ac0-4ffd-8aa3-1841a4541b55/5666e7cf-6b6c-4583-8335-aa3be69ccd45"
-          (reference "#PWR056") (unit 1)
-        )
-        (path "/e63e39d7-6ac0-4ffd-8aa3-1841a4541b55/93c6207c-4203-4bc7-a590-e5e89c0d3d27"
-          (reference "#PWR068") (unit 1)
-        )
         (path "/e63e39d7-6ac0-4ffd-8aa3-1841a4541b55/23ec3d7a-4d8b-4fb1-94c6-debe6172b9c6"
           (reference "#PWR083") (unit 1)

Commit message: Using another motor driver IC for contactor control
Parts:
- removed H3, H5: MountingHole, MountingHole:MountingHole_3.2mm_M3, symbol Mechanical:MountingHole
Changed lines of the file:
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@@
-    )
-  )
-  (symbol (lib_id "Mechanical:MountingHole") (at 30.48 142.24 0) (unit 1)
-    (in_bom yes) (on_board yes) (dnp no) (fields_autoplaced)
-    (property "Reference" "H5" (at 33.02 141.605 0)
-      (effects (font (size 1.27 1.27)) (justify left))
-    )
-    (property "Value" "MountingHole" (at 33.02 144.145 0)
-      (effects (font (size 1.27 1.27)) (justify left))
-    )
-    (property "Footprint" "MountingHole:MountingHole_3.2mm_M3" (at 30.48 142.24 0)
-      (effects (font (size 1.27 1.27)) hide)
-    )
-    (property "Datasheet" "~" (at 30.48 142.24 0)
-      (effects (font (size 1.27 1.27)) hide)
-    )
-    (instances
-      (project "qca7000"
-        (path "/e63e39d7-6ac0-4ffd-8aa3-1841a4541b55/23ec3d7a-4d8b-4fb1-94c6-debe6172b9c6"
-          (reference "H5") (unit 1)
-        )
-      )
     )
   )
@@
         )
       )
-    )
-  )
-  (symbol (lib_id "Mechanical:MountingHole") (at 30.48 128.27 0) (unit 1)
-    (in_bom yes) (on_board yes) (dnp no) (fields_autoplaced)
-    (property "Reference" "H3" (at 33.02 127.635 0)
-      (effects (font (size 1.27 1.27)) (justify left))
-    )
-    (property "Value" "MountingHole" (at 33.02 130.175 0)
-      (effects (font (size 1.27 1.27)) (justify left))
-    )
-    (property "Footprint" "MountingHole:MountingHole_3.2mm_M3" (at 30.48 128.27 0)
-      (effects (font (size 1.27 1.27)) hide)
-    )
-    (property "Datasheet" "~" (at 30.48 128.27 0)
-      (effects (font (size 1.27 1.27)) hide)
-    )
-    (instances
-      (project "qca7000"
-        (path "/e63e39d7-6ac0-4ffd-8aa3-1841a4541b55/23ec3d7a-4d8b-4fb1-94c6-debe6172b9c6"
-          (reference "H3") (unit 1)
-        )
-      )
