File: pcb/spareArea.kicad_sch (KiCad schematic)
At the start: 4 parts, among them J11 spare

Commit message: added TE DEUTSCH connector and housing
Parts:
- removed J11 (x4): spare, Connector_PinHeader_2.54mm:PinHeader_1x06_P2.54mm_Vertical, symbol Connector:Conn_01x06_Pin
Connections:
- no-connect marks 24 -> 0
Changed lines of the file:
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@@
 (kicad_sch (version 20230121) (generator eeschema)
   (paper "A4")
-  (no_connect (at 59.69 33.02))
-  (no_connect (at 72.39 38.1))
-  (no_connect (at 85.09 35.56))
-  (no_connect (at 59.69 45.72))
-  (no_connect (at 85.09 45.72))
-  (no_connect (at 59.69 43.18))
-  (no_connect (at 45.72 35.56))
-  (no_connect (at 85.09 33.02))
-  (no_connect (at 85.09 43.18))
-  (no_connect (at 45.72 45.72))
-  (no_connect (at 72.39 43.18))
-  (no_connect (at 72.39 40.64))
-  (no_connect (at 45.72 43.18))
-  (no_connect (at 85.09 40.64))
-  (no_connect (at 45.72 38.1))
-  (no_connect (at 72.39 45.72))
-  (no_connect (at 72.39 35.56))
-  (no_connect (at 59.69 35.56))
-  (no_connect (at 45.72 33.02))
-  (no_connect (at 72.39 33.02))
-  (no_connect (at 59.69 38.1))
-  (no_connect (at 59.69 40.64))
-  (no_connect (at 85.09 38.1))
-  (no_connect (at 45.72 40.64))
-  (symbol (lib_id "Connector:Conn_01x06_Pin") (at 40.64 38.1 0) (unit 1)
-    (in_bom yes) (on_board yes) (dnp no) (fields_autoplaced)
-    (property "Reference" "J11" (at 41.275 29.21 0)
-      (effects (font (size 1.27 1.27)))
-    )
-    (property "Value" "spare" (at 41.275 31.75 0)
-      (effects (font (size 1.27 1.27)))
-    )
-    (property "Footprint" "Connector_PinHeader_2.54mm:PinHeader_1x06_P2.54mm_Vertical" (at 40.64 38.1 0)
-      (effects (font (size 1.27 1.27)) hide)
-    )
-    (property "Datasheet" "~" (at 40.64 38.1 0)
-      (effects (font (size 1.27 1.27)) hide)
-    )
-    (pin "1")
-    (pin "2")
-    (pin "3")
-    (pin "4")
-    (pin "5")
-    (pin "6")
-    (instances
-      (project "qca7000"
-        (path "/e63e39d7-6ac0-4ffd-8aa3-1841a4541b55"
-          (reference "J11") (unit 1)
-        )
-        (path "/e63e39d7-6ac0-4ffd-8aa3-1841a4541b55/97d456cc-2984-45c2-9f4f-55359f773ff4"
-          (reference "J12") (unit 1)
-        )
-      )
-    )
-  )
-  (symbol (lib_id "Connector:Conn_01x06_Pin") (at 67.31 38.1 0) (unit 1)
-    (in_bom yes) (on_board yes) (dnp no) (fields_autoplaced)
-    (property "Reference" "J11" (at 67.945 29.21 0)
-      (effects (font (size 1.27 1.27)))
-    )
-    (property "Value" "spare" (at 67.945 31.75 0)
-      (effects (font (size 1.27 1.27)))
-    )
-    (property "Footprint" "Connector_PinHeader_2.54mm:PinHeader_1x06_P2.54mm_Vertical" (at 67.31 38.1 0)
-      (effects (font (size 1.27 1.27)) hide)
-    )
-    (property "Datasheet" "~" (at 67.31 38.1 0)
-      (effects (font (size 1.27 1.27)) hide)
-    )
-    (pin "1")
-    (pin "2")
-    (pin "3")
-    (pin "4")
-    (pin "5")
-    (pin "6")
-    (instances
-      (project "qca7000"
-        (path "/e63e39d7-6ac0-4ffd-8aa3-1841a4541b55"
-          (reference "J11") (unit 1)
-        )
-        (path "/e63e39d7-6ac0-4ffd-8aa3-1841a4541b55/97d456cc-2984-45c2-9f4f-55359f773ff4"
-          (reference "J14") (unit 1)
-        )
-      )
-    )
-  )
-  (symbol (lib_id "Connector:Conn_01x06_Pin") (at 54.61 38.1 0) (unit 1)
-    (in_bom yes) (on_board yes) (dnp no) (fields_autoplaced)
-    (property "Reference" "J11" (at 55.245 29.21 0)
-      (effects (font (size 1.27 1.27)))
-    )
-    (property "Value" "spare" (at 55.245 31.75 0)
-      (effects (font (size 1.27 1.27)))
-    )
-    (property "Footprint" "Connector_PinHeader_2.54mm:PinHeader_1x06_P2.54mm_Vertical" (at 54.61 38.1 0)
-      (effects (font (size 1.27 1.27)) hide)
-    )
-    (property "Datasheet" "~" (at 54.61 38.1 0)
-      (effects (font (size 1.27 1.27)) hide)
-    )
-    (pin "1")
-    (pin "2")
-    (pin "3")
-    (pin "4")
-    (pin "5")
-    (pin "6")
-    (instances
-      (project "qca7000"
-        (path "/e63e39d7-6ac0-4ffd-8aa3-1841a4541b55"
-          (reference "J11") (unit 1)
-        )
-        (path "/e63e39d7-6ac0-4ffd-8aa3-1841a4541b55/97d456cc-2984-45c2-9f4f-55359f773ff4"
-          (reference "J13") (unit 1)
-        )
-      )
-    )
-  )
-  (symbol (lib_id "Connector:Conn_01x06_Pin") (at 80.01 38.1 0) (unit 1)
-    (in_bom yes) (on_board yes) (dnp no) (fields_autoplaced)
-    (property "Reference" "J11" (at 80.645 29.21 0)
-      (effects (font (size 1.27 1.27)))
-    )
-    (property "Value" "spare" (at 80.645 31.75 0)
-      (effects (font (size 1.27 1.27)))
-    )
-    (property "Footprint" "Connector_PinHeader_2.54mm:PinHeader_1x06_P2.54mm_Vertical" (at 80.01 38.1 0)
-      (effects (font (size 1.27 1.27)) hide)
-    )
-    (property "Datasheet" "~" (at 80.01 38.1 0)
-      (effects (font (size 1.27 1.27)) hide)
-    )
-    (pin "1")
-    (pin "2")
-    (pin "3")
-    (pin "4")
-    (pin "5")
-    (pin "6")
-    (instances
-      (project "qca7000"
-        (path "/e63e39d7-6ac0-4ffd-8aa3-1841a4541b55"
-          (reference "J11") (unit 1)
-        )
-        (path "/e63e39d7-6ac0-4ffd-8aa3-1841a4541b55/97d456cc-2984-45c2-9f4f-55359f773ff4"
-          (reference "J15") (unit 1)
-        )
-      )
-    )
-  )
 )

Commit message: wired the drv8874. Added spare holes. Flash connector larger holes
Parts:
- added TP15, TP25, TP32, TP33, TP34, TP35, TP36, TP37, TP41, TP42, TP43, TP44, TP45, TP46, TP47, TP48, TP49, TP50, TP51, TP52, TP53, TP54, TP55, TP57, TP58, TP59, TP6, TP60: TestPoint, TestPoint:TestPoint_THTPad_D1.5mm_Drill0.7mm, symbol Connector:TestPoint
- added TP56: TestPoint, TestPoint:TestPoint_THTPad_D2.0mm_Drill1.0mm, symbol Connector:TestPoint
Connections:
- no-connect marks 0 -> 29

Commit message: changed to 4 layers. Added button, PP and lock feedback. New testpoints to avoid courtyard warnings.
Parts:
- TP15, TP25, TP32, TP33, TP34, TP35, TP36, TP37, TP41, TP42, TP43, TP44, TP45, TP46, TP47, TP48, TP49, TP50, TP51, TP52, TP53, TP54, TP55, TP57, TP58, TP59, TP6, TP60: footprint TestPoint:TestPoint_THTPad_D1.5mm_Drill0.7mm -> speciallib:TestPoint_Special_THTPad_D1.9mm_Drill1mm
- TP56: footprint TestPoint:TestPoint_THTPad_D2.0mm_Drill1.0mm -> speciallib:TestPoint_Special_THTPad_D1.9mm_Drill1mm
Changed lines of the file:
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@@
       (effects (font (size 1.27 1.27)) (justify left))
     )
-    (property "Footprint" "TestPoint:TestPoint_THTPad_D1.5mm_Drill0.7mm" (at 52.07 63.5 0)
+    (property "Footprint" "speciallib:TestPoint_Special_THTPad_D1.9mm_Drill1mm" (at 52.07 63.5 0)
       (effects (font (size 1.27 1.27)) hide)
     )
@@
       (effects (font (size 1.27 1.27)) (justify left))
     )
-    (property "Footprint" "TestPoint:TestPoint_THTPad_D1.5mm_Drill0.7mm" (at 72.39 69.85 0)
+    (property "Footprint" "speciallib:TestPoint_Special_THTPad_D1.9mm_Drill1mm" (at 72.39 69.85 0)
       (effects (font (size 1.27 1.27)) hide)
     )
@@
       (effects (font (size 1.27 1.27)) (justify left))
     )
-    (property "Footprint" "TestPoint:TestPoint_THTPad_D1.5mm_Drill0.7mm" (at 52.07 73.66 0)
+    (property "Footprint" "speciallib:TestPoint_Special_THTPad_D1.9mm_Drill1mm" (at 52.07 73.66 0)
       (effects (font (size 1.27 1.27)) hide)
     )
@@
       (effects (font (size 1.27 1.27)) (justify left))
     )
-    (property "Footprint" "TestPoint:TestPoint_THTPad_D1.5mm_Drill0.7mm" (at 50.8 101.6 0)
+    (property "Footprint" "speciallib:TestPoint_Special_THTPad_D1.9mm_Drill1mm" (at 50.8 101.6 0)
       (effects (font (size 1.27 1.27)) hide)
     )
@@
       (effects (font (size 1.27 1.27)) (justify left))
     )
-    (property "Footprint" "TestPoint:TestPoint_THTPad_D1.5mm_Drill0.7mm" (at 52.07 54.61 0)
+    (property "Footprint" "speciallib:TestPoint_Special_THTPad_D1.9mm_Drill1mm" (at 52.07 54.61 0)
       (effects (font (size 1.27 1.27)) hide)
     )
@@
       (effects (font (size 1.27 1.27)) (justify left))
     )
-    (property "Footprint" "TestPoint:TestPoint_THTPad_D1.5mm_Drill0.7mm" (at 52.07 27.94 0)
+    (property "Footprint" "speciallib:TestPoint_Special_THTPad_D1.9mm_Drill1mm" (at 52.07 27.94 0)
       (effects (font (size 1.27 1.27)) hide)
     )
@@
       (effects (font (size 1.27 1.27)) (justify left))
     )
-    (property "Footprint" "TestPoint:TestPoint_THTPad_D1.5mm_Drill0.7mm" (at 83.82 109.22 0)
+    (property "Footprint" "speciallib:TestPoint_Special_THTPad_D1.9mm_Drill1mm" (at 83.82 109.22 0)
       (effects (font (size 1.27 1.27)) hide)
     )
@@
       (effects (font (size 1.27 1.27)) (justify left))
     )
-    (property "Footprint" "TestPoint:TestPoint_THTPad_D1.5mm_Drill0.7mm" (at 31.75 49.53 0)
+    (property "Footprint" "speciallib:TestPoint_Special_THTPad_D1.9mm_Drill1mm" (at 31.75 49.53 0)
       (effects (font (size 1.27 1.27)) hide)
     )
@@
       (effects (font (size 1.27 1.27)) (justify left))
     )
-    (property "Footprint" "TestPoint:TestPoint_THTPad_D1.5mm_Drill0.7mm" (at 52.07 35.56 0)
+    (property "Footprint" "speciallib:TestPoint_Special_THTPad_D1.9mm_Drill1mm" (at 52.07 35.56 0)
       (effects (font (size 1.27 1.27)) hide)
     )
@@
       (effects (font (size 1.27 1.27)) (justify left))
     )
-    (property "Footprint" "TestPoint:TestPoint_THTPad_D1.5mm_Drill0.7mm" (at 31.75 40.64 0)
+    (property "Footprint" "speciallib:TestPoint_Special_THTPad_D1.9mm_Drill1mm" (at 31.75 40.64 0)
       (effects (font (size 1.27 1.27)) hide)
     )
@@
       (effects (font (size 1.27 1.27)) (justify left))
     )
-    (property "Footprint" "TestPoint:TestPoint_THTPad_D1.5mm_Drill0.7mm" (at 72.39 26.67 0)
+    (property "Footprint" "speciallib:TestPoint_Special_THTPad_D1.9mm_Drill1mm" (at 72.39 26.67 0)
       (effects (font (size 1.27 1.27)) hide)
     )
@@
       (effects (font (size 1.27 1.27)) (justify left))
     )
-    (property "Footprint" "TestPoint:TestPoint_THTPad_D1.5mm_Drill0.7mm" (at 72.39 59.69 0)
+    (property "Footprint" "speciallib:TestPoint_Special_THTPad_D1.9mm_Drill1mm" (at 72.39 59.69 0)
       (effects (font (size 1.27 1.27)) hide)
     )
@@
       (effects (font (size 1.27 1.27)) (justify left))
     )
-    (property "Footprint" "TestPoint:TestPoint_THTPad_D1.5mm_Drill0.7mm" (at 35.56 102.87 0)
+    (property "Footprint" "speciallib:TestPoint_Special_THTPad_D1.9mm_Drill1mm" (at 35.56 102.87 0)
       (effects (font (size 1.27 1.27)) hide)
     )
@@
       (effects (font (size 1.27 1.27)) (justify left))
     )
-    (property "Footprint" "TestPoint:TestPoint_THTPad_D1.5mm_Drill0.7mm" (at 72.39 36.83 0)
+    (property "Footprint" "speciallib:TestPoint_Special_THTPad_D1.9mm_Drill1mm" (at 72.39 36.83 0)
       (effects (font (size 1.27 1.27)) hide)
     )
@@
       (effects (font (size 1.27 1.27)) (justify left))
     )
-    (property "Footprint" "TestPoint:TestPoint_THTPad_D1.5mm_Drill0.7mm" (at 67.31 101.6 0)
+    (property "Footprint" "speciallib:TestPoint_Special_THTPad_D1.9mm_Drill1mm" (at 67.31 101.6 0)
       (effects (font (size 1.27 1.27)) hide)
     )
@@
       (effects (font (size 1.27 1.27)) (justify left))
     )
-    (property "Footprint" "TestPoint:TestPoint_THTPad_D1.5mm_Drill0.7mm" (at 72.39 46.99 0)
+    (property "Footprint" "speciallib:TestPoint_Special_THTPad_D1.9mm_Drill1mm" (at 72.39 46.99 0)
       (effects (font (size 1.27 1.27)) hide)
     )
@@
       (effects (font (size 1.27 1.27)) (justify left))
     )
-    (property "Footprint" "TestPoint:TestPoint_THTPad_D1.5mm_Drill0.7mm" (at 52.07 110.49 0)
+    (property "Footprint" "speciallib:TestPoint_Special_THTPad_D1.9mm_Drill1mm" (at 52.07 110.49 0)
       (effects (font (size 1.27 1.27)) hide)
     )
@@
       (effects (font (size 1.27 1.27)) (justify left))
     )
-    (property "Footprint" "TestPoint:TestPoint_THTPad_D1.5mm_Drill0.7mm" (at 31.75 69.85 0)
+    (property "Footprint" "speciallib:TestPoint_Special_THTPad_D1.9mm_Drill1mm" (at 31.75 69.85 0)
       (effects (font (size 1.27 1.27)) hide)
     )
@@
       (effects (font (size 1.27 1.27)) (justify left))
     )
-    (property "Footprint" "TestPoint:TestPoint_THTPad_D1.5mm_Drill0.7mm" (at 67.31 110.49 0)
+    (property "Footprint" "speciallib:TestPoint_Special_THTPad_D1.9mm_Drill1mm" (at 67.31 110.49 0)
       (effects (font (size 1.27 1.27)) hide)
     )
@@
       (effects (font (size 1.27 1.27)) (justify left))
     )
-    (property "Footprint" "TestPoint:TestPoint_THTPad_D1.5mm_Drill0.7mm" (at 72.39 81.28 0)
+    (property "Footprint" "speciallib:TestPoint_Special_THTPad_D1.9mm_Drill1mm" (at 72.39 81.28 0)
       (effects (font (size 1.27 1.27)) hide)
     )
@@
       (effects (font (size 1.27 1.27)) (justify left))
     )
-    (property "Footprint" "TestPoint:TestPoint_THTPad_D1.5mm_Drill0.7mm" (at 31.75 80.01 0)
+    (property "Footprint" "speciallib:TestPoint_Special_THTPad_D1.9mm_Drill1mm" (at 31.75 80.01 0)
       (effects (font (size 1.27 1.27)) hide)
     )
@@
       (effects (font (size 1.27 1.27)) (justify left))
     )
-    (property "Footprint" "TestPoint:TestPoint_THTPad_D1.5mm_Drill0.7mm" (at 52.07 45.72 0)
+    (property "Footprint" "speciallib:TestPoint_Special_THTPad_D1.9mm_Drill1mm" (at 52.07 45.72 0)
       (effects (font (size 1.27 1.27)) hide)
     )
@@
       (effects (font (size 1.27 1.27)) (justify left))
     )
-    (property "Footprint" "TestPoint:TestPoint_THTPad_D1.5mm_Drill0.7mm" (at 36.83 110.49 0)
+    (property "Footprint" "speciallib:TestPoint_Special_THTPad_D1.9mm_Drill1mm" (at 36.83 110.49 0)
       (effects (font (size 1.27 1.27)) hide)
     )
@@
       (effects (font (size 1.27 1.27)) (justify left))
     )
-    (property "Footprint" "TestPoint:TestPoint_THTPad_D1.5mm_Drill0.7mm" (at 73.66 93.98 0)
+    (property "Footprint" "speciallib:TestPoint_Special_THTPad_D1.9mm_Drill1mm" (at 73.66 93.98 0)
       (effects (font (size 1.27 1.27)) hide)
     )
@@
       (effects (font (size 1.27 1.27)) (justify left))
     )
-    (property "Footprint" "TestPoint:TestPoint_THTPad_D1.5mm_Drill0.7mm" (at 31.75 27.94 0)
+    (property "Footprint" "speciallib:TestPoint_Special_THTPad_D1.9mm_Drill1mm" (at 31.75 27.94 0)
       (effects (font (size 1.27 1.27)) hide)
     )
@@
       (effects (font (size 1.27 1.27)) (justify left))
     )
-    (property "Footprint" "TestPoint:TestPoint_THTPad_D1.5mm_Drill0.7mm" (at 31.75 34.29 0)
+    (property "Footprint" "speciallib:TestPoint_Special_THTPad_D1.9mm_Drill1mm" (at 31.75 34.29 0)
       (effects (font (size 1.27 1.27)) hide)
     )
@@
       (effects (font (size 1.27 1.27)) (justify left))
     )
-    (property "Footprint" "TestPoint:TestPoint_THTPad_D2.0mm_Drill1.0mm" (at 82.55 101.6 0)
+    (property "Footprint" "speciallib:TestPoint_Special_THTPad_D1.9mm_Drill1mm" (at 82.55 101.6 0)
       (effects (font (size 1.27 1.27)) hide)
     )
@@
       (effects (font (size 1.27 1.27)) (justify left))
     )
-    (property "Footprint" "TestPoint:TestPoint_THTPad_D1.5mm_Drill0.7mm" (at 52.07 85.09 0)
+    (property "Footprint" "speciallib:TestPoint_Special_THTPad_D1.9mm_Drill1mm" (at 52.07 85.09 0)
       (effects (font (size 1.27 1.27)) hide)
     )
@@
       (effects (font (size 1.27 1.27)) (justify left))
     )
-    (property "Footprint" "TestPoint:TestPoint_THTPad_D1.5mm_Drill0.7mm" (at 31.8846 59.2374 0)
-      (effects (font (size 1.27 1.27)) hide)
-    )
+    (property "Footprint" "speciallib:TestPoint_Special_THTPad_D1.9mm_Drill1mm" (at 31.8846 59.2374 0)
+      (effects (font (size 1.27 1.27)) hide)
+    )

Commit message: v4.2 layout finished. release files and readme
Parts:
- added TP10, TP16, TP17, TP18, TP19, TP20, TP21, TP22, TP61, TP62, TP63, TP64, TP7, TP9: TestPoint, speciallib:TestPoint_Special_THTPad_D1.9mm_Drill1mm, symbol Connector:TestPoint
Connections:
- no-connect marks 29 -> 43

Commit message: Routed new parts
Parts:
- removed TP19: TestPoint, speciallib:TestPoint_Special_THTPad_D1.9mm_Drill1mm, symbol Connector:TestPoint
Connections:
- no-connect marks 43 -> 42
Changed lines of the file:
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@@
   (no_connect (at 67.31 59.69))
   (no_connect (at 113.03 107.95))
-  (no_connect (at 96.52 116.84))
   (no_connect (at 30.48 102.87))
   (no_connect (at 67.31 36.83))
@@
         )
       )
-    )
-  )
-  (symbol (lib_id "Connector:TestPoint") (at 96.52 116.84 0) (unit 1)
-    (in_bom yes) (on_board yes) (dnp no) (fields_autoplaced)
-    (property "Reference" "TP19" (at 99.06 112.903 0)
-      (effects (font (size 1.27 1.27)) (justify left))
-    )
-    (property "Value" "TestPoint" (at 99.06 115.443 0)
-      (effects (font (size 1.27 1.27)) (justify left))
-    )
-    (property "Footprint" "speciallib:TestPoint_Special_THTPad_D1.9mm_Drill1mm" (at 101.6 116.84 0)
-      (effects (font (size 1.27 1.27)) hide)
-    )
-    (property "Datasheet" "~" (at 101.6 116.84 0)
-      (effects (font (size 1.27 1.27)) hide)
-    )
-    (pin "1")
-    (instances
-      (project "qca7000"
-        (path "/e63e39d7-6ac0-4ffd-8aa3-1841a4541b55/97d456cc-2984-45c2-9f4f-55359f773ff4"
-          (reference "TP19") (unit 1)
-        )
-      )
